File: hardware/mainboard/FanControl.kicad_sch (KiCad schematic)
At the start: 25 parts, among them Q2 DMT6018LDR-7, Q3 DMT6018LDR-7, Q4 DMT6018LDR-7, Q5 DMT6018LDR-7

Commit message: sync
Parts:
- removed D17, D20, D21: 60V/0.5/3A, Diode_SMD:D_SOD-123, symbol Device:D_Schottky_Small
- removed Q4, Q5: DMT6018LDR-7, Samacsys:DMT6018LDR7, symbol Samacsys_kicad_sym:DMT6018LDR-7
- removed R62, R63, R66: 100, Resistor_SMD:R_0603_1608Metric, symbol Device:R_Small
- removed R64, R65, R67: 10k, Resistor_SMD:R_0603_1608Metric, symbol Device:R_Small
Connections:
- no-connect marks 3 -> 0
Other:
- note removed: "NMOS 5"
- note removed: "NMOS 6"
- note removed: "NMOS 7"
- note removed: "UNUSED"
- moved on the sheet: D13, D18, D19, D8, Q2A, Q2B, Q3A, Q3B, R30, R5, R56, R57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

Commit message: schematic?
Connections:
- net +12V renamed +24V
