File: hardware/mainboard/PUTM_EV_AMS_MASTER_2025.kicad_pcb (KiCad board)
At the start: 4 copper layers, 60 x 100 mm, 257 parts, among them IC1 3.3V/0.5A, IC11 ISO6760, IC2 TPS54202HDDCR, IC3 BQ79600PWRQ1, IC4 ADC 24bit, IC5 LTC1799, IC6 LTC6820IMS, IC7 ISO6760, IC8 3.3V/0.5A, J1 M80-5100642, J10 M300-MV10345M1, J12 M80-51034XX, J2 USB_C_Receptacle_USB2.0_14P, J3 M80-51014XX, J4 FTSH-107-01-L-D-K, J5 M80-51004XX, J7 M300-MV10345M1, J8 M80-51004XX, K1 IMB03ITS, Q1 DMT6018LDR-7, Q2 DMT6018LDR-7, Q3 DMT6018LDR-7, Q4 DMT6018LDR-7, Q5 DMT6018LDR-7, Q6 2N7002, Q7 DMT6018LDR-7, Q8 2N7002, Q9 2N7002, T1 >100kHz, U10 STM32H573RITx, U12 LMR33640DDDA, U13 LM397, U2 LM397, U3 74AUP1G32, U4 UCC12040DVE, U5 LM397, U6 MCP2542FD-E/MF, U7 MCP2542FD-E/MF, U8 LM397, U9 LM397, Y1 50MHz

Commit message: schematic?
Parts:
- removed C1, C2: 8pF/.1pF, Capacitor_SMD:C_0603_1608Metric
- removed C35, C60, C71, C73, C75, C82: 100nF, Capacitor_SMD:C_0603_1608Metric
- removed C41: 220nF, Capacitor_SMD:C_0603_1608Metric
- removed C66, C72, C74: TBD, Capacitor_SMD:C_0603_1608Metric
- removed D17: 60V/0.5/3A, Diode_SMD:D_SOD-123
- removed F3: 12V/4A, Fuse:Fuse_1206_3216Metric
- removed F6, F7: 5V/0.5A, Fuse:Fuse_0805_2012Metric
- removed IC11: ISO6760, Package_SO:SOIC-16W_7.5x10.3mm_P1.27mm
- removed IC5: LTC1799, Package_TO_SOT_SMD:SOT-23-5
- removed J12: M80-51034XX, Samacsys:M80-51034YY
- removed L2: 6.8uF/3.5A, Inductor_SMD:L_TDK_VLS6045EX_VLS6045AF
- removed Q5: DMT6018LDR-7, Samacsys:DMT6018LDR7
- removed R1, R2: 1M/700V/.1%, Resistor_SMD:R_1206_3216Metric
- removed R106, R107, R69, R75, R76, R82, R83: TBD, Resistor_SMD:R_0603_1608Metric
- removed R15: 100, Resistor_SMD:R_0603_1608Metric
- removed R18: 8.2k, Resistor_SMD:R_0603_1608Metric
- removed R19: 1k, Resistor_SMD:R_0603_1608Metric
- removed R4, R94: 10k, Resistor_SMD:R_0603_1608Metric
- removed R6: 100/.1%, Resistor_SMD:R_1206_3216Metric
- removed R91, R92: 5.1k, Resistor_SMD:R_0603_1608Metric
- removed R95: 100k, Resistor_SMD:R_0603_1608Metric
- removed REF** (x2): Symbol_HighVoltage_Triangle_6x6mm_Copper, Symbol:Symbol_HighVoltage_Triangle_6x6mm_Copper
- removed TP10, TP5, TP6, TP7, TP8: TestPoint_Small, TestPoint:TestPoint_THTPad_D1.0mm_Drill0.5mm
- removed U5, U8, U9: LM397, Package_TO_SOT_SMD:SOT-23-5
- removed Y1: 50MHz, Crystal:Crystal_SMD_3225-4Pin_3.2x2.5mm
- added C101: 10nF, Capacitor_SMD:C_0603_1608Metric, B.Cu at (130.2, 101.0)
- added C102: 10nF, Capacitor_SMD:C_0603_1608Metric, B.Cu at (130.2, 97.0)
- added C103: 10nF, Capacitor_SMD:C_0603_1608Metric, B.Cu at (134.0, 101.0)
- added C104: 10nF, Capacitor_SMD:C_0603_1608Metric, B.Cu at (134.0, 97.0)
- added C105: 10nF, Capacitor_SMD:C_0603_1608Metric, B.Cu at (137.8, 101.0)
- added C88: 1nF, Capacitor_SMD:C_0603_1608Metric, F.Cu at (138.5, 83.0)
- added C89: 10nF, Capacitor_SMD:C_0603_1608Metric, F.Cu at (136.5, 80.2)
- added C90: 10nF, Capacitor_SMD:C_0603_1608Metric, F.Cu at (133.0, 80.2)
- added C91: 1n, Capacitor_SMD:C_0603_1608Metric, B.Cu at (140.0, 60.0)
- added C92: 1n, Capacitor_SMD:C_0603_1608Metric, B.Cu at (125.0, 60.0)
- added C93: 1n, Capacitor_SMD:C_0603_1608Metric, F.Cu at (176.7, 56.3)
- added C94: 1n, Capacitor_SMD:C_0603_1608Metric, F.Cu at (176.7, 58.8)
- added C95: 1n, Capacitor_SMD:C_0603_1608Metric, F.Cu at (180.7, 46.2)
- added C96: 1n, Capacitor_SMD:C_0603_1608Metric, F.Cu at (180.7, 48.8)
- added C97: 1n, Capacitor_SMD:C_0603_1608Metric, F.Cu at (180.7, 51.3)
- added C98: 1n, Capacitor_SMD:C_0603_1608Metric, F.Cu at (180.7, 53.8)
- added C99: 100nF, Capacitor_SMD:C_0603_1608Metric, F.Cu at (180.7, 56.3)
- added D12: 5.3V/400W, Package_TO_SOT_SMD:SOT-23-3, F.Cu at (147.0, 108.5)
- added D23: 5.3V/400W, Package_TO_SOT_SMD:SOT-23-3, F.Cu at (140.5, 78.5)
- added FB1: 100@100Mhz, Inductor_SMD:L_0603_1608Metric, F.Cu at (179.0, 83.7)
- added FB2: 100@100Mhz, Inductor_SMD:L_0603_1608Metric, F.Cu at (181.6, 83.7)
- added IC9: LTC1799, Package_TO_SOT_SMD:SOT-23-5, F.Cu at (140.5, 87.0)
- added L1: 10uH, Inductor_SMD:L_1008_2520Metric, F.Cu at (114.0, 122.5)
- added R33: 20k/.1%, Resistor_SMD:R_0603_1608Metric, F.Cu at (141.0, 82.0)
- added R43: 10k/.1%, Resistor_SMD:R_0603_1608Metric, F.Cu at (141.0, 84.0)
- added R49: 100k, Resistor_SMD:R_0603_1608Metric, F.Cu at (130.2, 103.2)
- added R50: 1k/.1%, Resistor_SMD:R_0603_1608Metric, F.Cu at (137.2, 78.0)
- added R51: 1k/.1%, Resistor_SMD:R_0603_1608Metric, F.Cu at (135.8, 78.0)
- added R52: 1k/.1%, Resistor_SMD:R_0603_1608Metric, F.Cu at (133.8, 78.0)
- added TP1: TestPoint_Small, TestPoint:TestPoint_Pad_D1.0mm, F.Cu at (139.0, 128.5)
- added U14: LM393, Package_SO:VSSOP-8_3x3mm_P0.65mm, F.Cu at (137.8, 99.0)
- C10, C18: value 100nF -> 1uF
- C16: value 22uF -> 1uF; footprint Capacitor_SMD:C_0805_2012Metric -> Capacitor_SMD:C_0603_1608Metric
- C19, C20: value 22uF -> 2.2uF; footprint Capacitor_SMD:C_0805_2012Metric -> Capacitor_SMD:C_0603_1608Metric; moved to F.Cu
- C30: value 1nF -> 22uF; footprint Capacitor_SMD:C_0603_1608Metric -> Capacitor_SMD:C_0805_2012Metric
- C31: value 100nF -> 22uF; footprint Capacitor_SMD:C_0603_1608Metric -> Capacitor_SMD:C_0805_2012Metric; moved to F.Cu
- C34: value 10nF -> 100nF
- C4: value 220nF -> 2.2uF; moved to F.Cu
- C40, C52, C54, C55, C59, C77: value 22uF -> 100nF; footprint Capacitor_SMD:C_0805_2012Metric -> Capacitor_SMD:C_0603_1608Metric
- C46: value 100nF -> 10nF
- C48: value 100nF -> 220nF
- C5: value TBD -> 2.2uF; moved to F.Cu
- C67: value 1nF -> 100nF
- C76, F5, F8: moved to F.Cu
- C79, C80: value 100p -> 100pF
- C81: value TBD -> 100pF
- C86, C87: value 2.2nF -> 2.2uF
- D11: value ESDA5V3SC5 -> 5.3V/400W; footprint Package_TO_SOT_SMD:SOT-23-6 -> Package_TO_SOT_SMD:SOT-23-3
- D20: value 60V/0.5/3A -> 8V
- D21: value 60V/0.5/3A -> 3.6V/400W; footprint Diode_SMD:D_SOD-123 -> Package_TO_SOT_SMD:SOT-23-6
- D22: value ESDA5V3SC5 -> 3.6V/400W
- D4: value 60V/0.5/3A -> 5.3V/400W; footprint Diode_SMD:D_SOD-123 -> Package_TO_SOT_SMD:SOT-23-3; moved to F.Cu
- D5: value 60V/0.5/3A -> 10V; moved to F.Cu
- IC4: value ADC 24bit -> TLV61046ADBVT; footprint Package_DFN_QFN:WQFN-20-1EP_3x3mm_P0.4mm_EP1.7x1.7mm -> Package_TO_SOT_SMD:SOT-23-6
- IC6: value LTC6820IMS -> AMC3330DWER; footprint Package_SO:MSOP-16_3x4.039mm_P0.5mm -> Package_SO:SOIC-16W_7.5x10.3mm_P1.27mm
- IC7: value ISO6760 -> AMC3330DWER
- IC8: value 3.3V/0.5A -> ADC 24bit; footprint Package_TO_SOT_SMD:SOT-23-5 -> Package_DFN_QFN:WQFN-20-1EP_3x3mm_P0.4mm_EP1.7x1.7mm
- J2: value USB_C_Receptacle_USB2.0_14P -> M80-5102042; footprint Connector_USB:USB_C_Receptacle_JAE_DX07S024WJ3R400 -> Samacsys:M80-51020YY
- J3: value M80-51014XX -> M80-5100842; footprint Samacsys:M80-51014YY -> Samacsys:M80-51008YY
- K1: value IMB03ITS -> IM07DTS; footprint Samacsys:IMB03ITS -> Samacsys:IM23TS
- Q4: value DMT6018LDR-7 -> SI2347DS-T1-GE3; footprint Samacsys:DMT6018LDR7 -> Package_TO_SOT_SMD:SOT-23-3
- R10: value 10k -> 100k; footprint Resistor_SMD:R_0603_1608Metric -> Resistor_SMD:R_0603_1608Metric_Pad0.98x0.95mm_HandSolder
- R16: value 1k -> 20k
- R17: value 10k -> 20k
- R20: value 120 -> 10k; moved to B.Cu
- R22: value 200 -> 10k
- R24: value 9.09k -> 25k/.1%
- R25: value 100k -> 10k
- R32: value 100 -> 10k; moved to F.Cu
- R35, R68: value TBD -> 100k; moved to F.Cu
- R38: value TBD -> 1k
- R39: value 33 -> 100k
- R40: value 33 -> 400
- R41: value 100 -> 10k
- R53: value 1M/700V/.1% -> 100k; footprint Resistor_SMD:R_1206_3216Metric -> Resistor_SMD:R_0603_1608Metric; moved to F.Cu
- R54: value 1M/700V/.1% -> 1k/.1%; footprint Resistor_SMD:R_1206_3216Metric -> Resistor_SMD:R_0603_1608Metric; moved to F.Cu
- R55: value 100/.1% -> 649k; footprint Resistor_SMD:R_1206_3216Metric -> Resistor_SMD:R_0603_1608Metric
- R62: value 100 -> 71.5k
- R63: value 100 -> 100k; moved to F.Cu
- R64: value 10k -> 1M/700V/.1%; footprint Resistor_SMD:R_0603_1608Metric -> Resistor_SMD:R_1206_3216Metric
- R65, R67: value 10k -> 1k/.1%; footprint Resistor_SMD:R_0603_1608Metric -> Resistor_SMD:R_1206_3216Metric
- R66: value 100 -> 1M/700V/.1%; footprint Resistor_SMD:R_0603_1608Metric -> Resistor_SMD:R_1206_3216Metric
- R7, R8: value 33 -> 27; moved to F.Cu
- R70: value 10k -> 100k; moved to F.Cu
- R9: value 10k -> 0
- T1: value >100kHz -> SM91502ALE; footprint Samacsys:SOP254P914X350-4N -> Samacsys:SOP254P927X572-6N
- TP4: footprint TestPoint:TestPoint_THTPad_D1.0mm_Drill0.5mm -> TestPoint:TestPoint_Pad_D1.0mm
- U12: value LMR33640DDDA -> LM393; footprint Package_SO:Texas_HSOP-8-1EP_3.9x4.9mm_P1.27mm -> Package_SO:VSSOP-8_3x3mm_P0.65mm
- U13: value LM397 -> LM393; footprint Package_TO_SOT_SMD:SOT-23-5 -> Package_SO:VSSOP-8_3x3mm_P0.65mm
- U2: value LM397 -> FT230XS; footprint Package_TO_SOT_SMD:SOT-23-5 -> Package_SO:SSOP-16_3.9x4.9mm_P0.635mm
- U4: value UCC12040DVE -> TPS2113PWR; footprint Package_SO:SOIC-16W_7.5x10.3mm_P1.27mm -> Package_SO:TSSOP-8_4.4x3mm_P0.65mm
- moved C54 115.3 mm to (186.0, 43.0)
- moved C55 110.0 mm to (188.5, 43.0)
- moved C10 108.2 mm to (178.5, 43.0)
- moved C9 105.8 mm to (176.0, 43.0)
- moved C16 103.4 mm to (181.0, 43.0)
- moved G*** 86.8 mm to (204.5, 58.5)
- moved R64 75.1 mm to (140.5, 56.0)
- moved R65 74.9 mm to (146.5, 56.0), turned to -90 degrees
- moved C20 73.6 mm to (176.5, 83.7), turned to 90 degrees
- moved C59 73.5 mm to (176.7, 46.2)
- moved C30 71.7 mm to (112.8, 126.8), turned to 90 degrees
- moved C4 70.2 mm to (169.0, 83.7)
- moved C19 67.6 mm to (174.0, 83.7)
- moved C31 66.1 mm to (114.0, 129.1), turned to 0 degrees
- moved R67 64.5 mm to (123.5, 56.0)
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Connections:
- net /AIR_M renamed /AIR_M-
- net /AIR_P renamed /AIR_P-
- net /AIR_PRE renamed /AIR_PRE-
- net /Connectivity/AIR Minus/REF renamed Net-(U14A-+)
- net /TSMS_AIRS renamed /SDC_AIRS
- C10 pad 1: /Power/BOOT_12V -> GND
- C10 pad 2: /Power/SW_12V -> +5VISO
- C13 pad 1: +5V -> +5VIO
- C16 pad 1: /Power/F_12V -> /IsolationBarrier/ACU_GND
- C16 pad 2: GND -> /IsolationBarrier/ACU_DCDC
- C18 pad 1: +3.3VISO -> /IsolationBarrier/CAR_GND
- C18 pad 2: GNDISO -> /IsolationBarrier/CAR_DCDC
- C19 pad 1: /Power/F_12V -> GND
- C19 pad 2: GND -> +3.3VIO
- C20 pad 1: /Power/F_12V -> GND
- C20 pad 2: GND -> +3.3VA
- C23 pad 1: +3.3VIO -> +3.3VMCU
- C24 pad 1: +3.3VIO -> +3.3VMCU
- C25 pad 1: +3.3VIO -> +3.3VMCU
- C28 pad 1: +3.3VIO -> +3.3VMCU
- C29 pad 1: +3.3VIO -> +3.3VMCU
- C3 pad 2: /Power/F_U5V -> VBUS+
- C30 pad 1: /Isolated ADC/ACU- -> GND
- C30 pad 2: /Isolated ADC/ACU+ -> +5VIO
- C31 pad 1: +3.3VISO -> GND
- C31 pad 2: GNDISO -> +8V
- C32 pad 1: +5V -> +5VIO
- C33 pad 1: +5V -> +5VIO
- C34 pad 1: +3.3VISO -> /Connectivity/+3.3VFTDI
- C34 pad 2: GNDISO -> GND
- C36 pad 1: +3.3VIO -> +3.3VMCU
- C37 pad 2: +3.3V -> +3.3VIO
- C38 pad 2: +3.3V -> +3.3VIO
- C39 pad 1: +3.3V -> GND
- C39 pad 2: GND -> /Power/5VPWR
- C4 pad 1: +24V -> GND
- C4 pad 2: GND -> +5VIO
- C40 pad 1: /F_+5VISO -> GND
- C40 pad 2: GNDISO -> /Power/5VUSB
- C42 pad 1: +3.3VISO -> GND
- C42 pad 2: GNDISO -> +5VIO
- C43 pad 1: GNDISO -> GND
- C43 pad 2: +5VISO -> +5VIO
- C44 pad 1: +3.3VISO -> +5VIO
- C44 pad 2: GNDISO -> GND
- C45 pad 1: +3.3V -> +3.3VA
- C46 pad 1: +3.3VISO -> +3.3VA
- C46 pad 2: GNDISO -> GND
- C47 pad 1: GNDISO -> GND
- C47 pad 2: /F_+5VISO -> +3.3VIO
- C48 pad 1: /F_+3VISO -> GND
- C48 pad 2: GNDISO -> /ADC/CAP
- C49 pad 1: GNDISO -> +5VIO
- C49 pad 2: +3.3VISO -> GND
- C5 pad 1: /Connectivity/Input2/IN+ -> GND
- C5 pad 2: GND -> +5VA
- C50 pad 1: +24V -> +5VIO
- C52 pad 2: +24V -> +3.3VIO
- C53 pad 2: GNDISO -> GND
- C54 pad 1: GND -> /IsolationBarrier/ACU_LDO
- C54 pad 2: +24V -> /IsolationBarrier/ACU_GND
- C55 pad 1: /Power/F_12V -> Net-(IC6B-DCDC_IN)
- C56 pad 2: +5V -> +5VIO
- C58 pad 1: /AMS_ERROR -> +5VIO
- C59 pad 1: +5V -> /IsolationBarrier/CAR_LDO
- C59 pad 2: GND -> /IsolationBarrier/CAR_GND
- C6 pad 1: /Power/F_U5V -> VBUS+
- C67 pad 1: /Isolated ADC/CAR- -> /IsolationBarrier/ACU_DCDC
- C67 pad 2: /Isolated ADC/CAR+ -> /IsolationBarrier/ACU_GND
- C70 pad 1: +3.3VIO -> +3.3VMCU
- C76 pad 1: /Connectivity/Input1/REF -> /Connectivity/REF
- C77 pad 1: /F_+5VISO -> /IsolationBarrier/CAR_DCDC
- C77 pad 2: GNDISO -> /IsolationBarrier/CAR_GND
- C78 pad 1: +3.3VISO -> +3.3VIO
- C78 pad 2: GNDISO -> GND
- C79 pad 1: GNDISO -> GND
- C8 pad 2: +3.3V -> +3.3VIO
- C80 pad 1: GNDISO -> GND
- C81 pad 1: /Connectivity/Input1/IN+ -> Net-(T1-SEC_2)
- C9 pad 2: /Power/VCC_12V -> +5VISO
- D1 pad 2: +3.3V -> +3.3VIO
- D11 pad 1: /Connectivity/UC_D- -> /CANFD2+
- D11 pad 2: GND -> /CANFD2-
- D11 pad 3: /Connectivity/UC_D+ -> GND
- D13 pad 1: +12V -> +24V
- D14 pad 1: /Power/F_U5V -> VBUS+
- D18 pad 1: +12V -> +24V
- D19 pad 1: +12V -> +24V
- D2 pad 2: +3.3V -> +3.3VIO
- D20 pad 1: +12V -> +8V
- D20 pad 2: /FAN6- -> GND
- D21 pad 1: +12V -> /SWDIO
- D21 pad 2: /FAN7- -> GND
- D22 pad 1: /Connectivity/UC_D- -> /UART_RX
- D22 pad 3: /Connectivity/UC_D+ -> +3.3VIO
- D22 pad 4: /Connectivity/UC_D+ -> unconnected-(D22-A-Pad4)
- D22 pad 6: /Connectivity/UC_D- -> unconnected-(D22-A-Pad6)
- D3 pad 2: +3.3V -> +3.3VIO
- D4 pad 1: +24V -> /CANFD1+
- D4 pad 2: /Power/F_24V -> /CANFD1-
- D5 pad 1: /Power/F_U5V -> +24V
- D5 pad 2: VBUS+ -> Net-(D5-A)
- D6 pad 2: +3.3V -> +3.3VIO
- D7 pad 1: +5V -> +24V
- D8 pad 1: +12V -> +24V
- F4 pad 2: +5V -> /Power/5VPWR
- F5 pad 2: +3.3V -> +3.3VIO
- F8 pad 1: /Power/F_U5V -> VBUS+
- F8 pad 2: +5V -> /Power/5VUSB
- IC1 pad 1: +5V -> +5VIO
- IC3 pad 14: +5VISO -> +5VIO
- IC3 pad 15: +5VISO -> +5VIO
- IC3 pad 16: +5VISO -> +5VIO
- IC3 pad 3: +3.3VISO -> +3.3VIO
- IC3 pad 4: /ISO_COM_MOSI -> /UCTX
- IC3 pad 5: /ISO_COM_MISO -> /UCRX
- IC3 pad 6: /ISO_COM_SCK -> GND
- IC3 pad 7: /~{ISO_COM_CS} -> GND
- IC3 pad 8: /SPI_RDY -> GND
- IC3 pad 9: GNDISO -> GND
- IC4 pad 1: /Isolated ADC/ACU+ -> Net-(IC4-SW)
- IC4 pad 2: /Isolated ADC/ACU- -> GND
- IC4 pad 3: /Isolated ADC/CAR+ -> Net-(IC4-FB)
- IC4 pad 4: /Isolated ADC/CAR- -> +5VIO
- IC4 pad 5: /Isolated ADC/I+ -> +8V
- IC4 pad 6: /Isolated ADC/I- -> +5VIO
- IC6 pad 1: +3.3VISO -> /IsolationBarrier/ACU_DCDC
- IC6 pad 10: /OUT- -> /ADC/ACU_V-
- IC6 pad 11: /OUT+ -> /ADC/ACU_V+
- IC6 pad 12: +3.3VISO -> +5VISO
- IC6 pad 13: GNDISO -> Net-(IC6B-DCDC_IN)
- IC6 pad 14: GNDISO -> unconnected-(IC6B-DIAG-Pad14)
- IC6 pad 15: Net-(IC6-ICMP) -> GND
- IC6 pad 16: Net-(IC6-IBIAS) -> Net-(IC6B-DCDC_IN)
- IC6 pad 2: /ISO_COM_MOSI -> /IsolationBarrier/ACU_GND
- IC6 pad 3: /ISO_COM_MISO -> /IsolationBarrier/ACU_DCDC
- IC6 pad 4: /ISO_COM_SCK -> unconnected-(IC6B-NC-Pad4)
- IC6 pad 5: /~{ISO_COM_CS} -> /IsolationBarrier/ACU_LDO
- IC6 pad 6: +3.3VISO -> /IsolationBarrier/ACU+
- IC6 pad 7: +3.3VISO -> /IsolationBarrier/ACU_GND
- IC6 pad 8: +3.3VISO -> /IsolationBarrier/ACU_GND
- IC6 pad 9: +3.3VISO -> GND
- IC7 pad 1: +3.3V -> /IsolationBarrier/CAR_DCDC
- IC7 pad 10: /~{ISO_COM_CS} -> /ADC/CAR_V-
- IC7 pad 11: /ISO_COM_SCK -> /ADC/CAR_V+
- IC7 pad 12: /ISO_COM_MOSI -> +5VISO
- IC7 pad 13: /~{ISO_ADC_CS} -> Net-(IC7B-DCDC_IN)
- IC7 pad 14: /ISO_ADC_SCK -> unconnected-(IC7B-DIAG-Pad14)
- IC7 pad 15: /ISO_ADC_MOSI -> GND
- IC7 pad 16: +3.3VISO -> Net-(IC7B-DCDC_IN)
- IC7 pad 2: /MCU/ADC_MOSI -> /IsolationBarrier/CAR_GND
- IC7 pad 3: /MCU/ADC_SCK -> /IsolationBarrier/CAR_DCDC
- IC7 pad 4: /MCU/~{ADC_CS} -> unconnected-(IC7B-NC-Pad4)
- IC7 pad 5: /MCU/COM_MOSI -> /IsolationBarrier/CAR_LDO
- IC7 pad 6: /MCU/COM_SCK -> /IsolationBarrier/CAR+
- IC7 pad 7: /MCU/~{COM_CS} -> /IsolationBarrier/CAR_GND
- IC7 pad 8: GND -> /IsolationBarrier/CAR_GND
- IC7 pad 9: GNDISO -> GND
- IC8 pad 1: /F_+5VISO -> /ADC/I+
- IC8 pad 2: GNDISO -> GND
- IC8 pad 3: unconnected-(IC8-NC-Pad3) -> /ADC/ACU+
- IC8 pad 4: unconnected-(IC8-NC-Pad4) -> /ADC/ACU-
- IC8 pad 5: /F_+3VISO -> /ADC/CAR+
- J10 pad 1: /Isolated ADC/CAR_V+ -> /IsolationBarrier/CAR_IN+
- J10 pad 3: /Isolated ADC/CAR_V- -> /IsolationBarrier/CAR_GND
- J3 pad 5: /FAN5- -> +24V
- J3 pad 6: /FAN6- -> +24V
- J3 pad 7: /FAN7- -> +24V
- J3 pad 8: +12V -> +24V
- J4 pad 3: +3.3V -> +3.3VIO
- J7 pad 1: /Isolated ADC/ACU_V+ -> /IsolationBarrier/ACU_IN+
- J7 pad 3: /Isolated ADC/ACU_V- -> /IsolationBarrier/ACU_GND
- J8 pad 1: /Isolated ADC/I- -> +5VA
- J8 pad 2: /Isolated ADC/I+ -> /CAR_I
- J8 pad 3: +5VISO -> unconnected-(J8-Pin_3-Pad3)
- J8 pad 4: GNDISO -> GND
- K1 pad 1: /Safety/RELAY- -> +24V
- K1 pad 3: /SAFETY_OUT -> /SAFETY_IN
- K1 pad 6: /SAFETY_IN -> unconnected-(K1-COM_2-Pad6)
- K1 pad 8: +5V -> /Safety/RELAY-
- Q4 pad 1: /Fan Control/G5 -> Net-(D5-A)
- Q4 pad 2: GND -> +24V
- Q4 pad 3: GND -> /Power/F_24V
- Q8 pad 1: /Safety/WEB -> /MCU/SIGNAL_AMS_ERROR
- Q9 pad 1: /Safety/AMS_OK -> /AMS_ERROR
- R10 pad 1: /MCU/PG_12V -> Net-(D5-A)
- R10 pad 2: +3.3V -> GND
- R100 pad 1: /MCU/SIGNAL_AMS_ERROR -> /MCU/DETECT_WTDG
- R12 pad 1: +3.3V -> +3.3VIO
- R13 pad 1: /Safety/AMS_OK -> /AMS_ERROR
- R13 pad 2: +3.3V -> +3.3VIO
- R14 pad 2: /MCU/DETECT_WTDG -> Net-(R14-Pad2)
- R16 pad 1: Net-(IC6-ICMP) -> /Power/VSNS
- R16 pad 2: Net-(IC6-IBIAS) -> GND
- R17 pad 1: +3.3V -> +3.3VIO
- R17 pad 2: /Connectivity/Input1/REF -> /Connectivity/REF
- R20 pad 1: /OUT+ -> GND
- R20 pad 2: /OUT- -> Net-(U12A-+)
- R21 pad 1: Net-(IC4-~{SYNC}) -> GND
- R21 pad 2: +3.3VISO -> Net-(U12B-+)
- R22 pad 1: GNDISO -> Net-(IC8-~{SYNC})
- R22 pad 2: /F_+5VISO -> +3.3VIO
- R24 pad 1: GND -> /ADC/SET
- R24 pad 2: /Power/FB_12V -> +3.3VIO
- R25 pad 1: /Power/FB_12V -> GND
- R25 pad 2: /Power/F_12V -> Net-(U13A-+)
- R26 pad 1: /Connectivity/Input1/REF -> /Connectivity/REF
- R3 pad 1: +3.3V -> +3.3VIO
- R3 pad 2: +3.3VIO -> +3.3VMCU
- R32 pad 1: /AMS_ERROR -> GND
- R32 pad 2: /Safety/AMS_OK -> /VUSB
- R35 pad 1: /Connectivity/Input2/IN+ -> VBUS+
- R35 pad 2: GND -> /VUSB
- R38 pad 1: /Connectivity/Input2/IN+ -> /MCU/SIGNAL_AMS_ERROR
- R38 pad 2: /CHARGER_DETECTION -> Net-(R14-Pad2)
- R39 pad 1: /Connectivity/UC_D- -> /Power/5VPWR
- R39 pad 2: /USBR_D- -> /Power/VSNS
- R40 pad 1: /Connectivity/UC_D+ -> GND
- R40 pad 2: /USBR_D+ -> /Power/ILIM
- R41 pad 1: /AMS_ERROR -> GND
- R41 pad 2: /DASH_LED -> Net-(U13B-+)
- R42 pad 1: +3.3V -> GND
- R53 pad 1: /Isolated ADC/CAR+ -> Net-(U12B-+)
- R53 pad 2: /Isolated ADC/CAR_V+ -> /CHARGER_DETECTION
- R54 pad 1: /Isolated ADC/CAR_V- -> /ADC/CAR_V-
- R54 pad 2: /Isolated ADC/CAR- -> /ADC/CAR-
- R55 pad 1: /Isolated ADC/CAR- -> +8V
- R55 pad 2: /Isolated ADC/CAR+ -> Net-(IC4-FB)
- R62 pad 1: /FC5 -> GND
- R62 pad 2: /Fan Control/G5 -> Net-(IC4-FB)
- R63 pad 1: /FC6 -> Net-(U13A-+)
- R63 pad 2: /Fan Control/G6 -> /AIR_PRE_DETECTION
- R64 pad 1: GND -> /IsolationBarrier/ACU_IN+
- R64 pad 2: /Fan Control/G5 -> /IsolationBarrier/ACU+
- R65 pad 1: GND -> /IsolationBarrier/ACU_GND
- R65 pad 2: /Fan Control/G6 -> /IsolationBarrier/ACU+
- R66 pad 1: /FC7 -> /IsolationBarrier/CAR_IN+
- R66 pad 2: /Fan Control/G7 -> /IsolationBarrier/CAR+
- R67 pad 1: GND -> /IsolationBarrier/CAR_GND
- R67 pad 2: /Fan Control/G7 -> /IsolationBarrier/CAR+
- R68 pad 1: /Connectivity/AIR Precharge/IN+ -> Net-(U13B-+)
- R68 pad 2: GND -> /AIR_M_DETECTION
- R7 pad 1: /Connectivity/UC_D+ -> /D+
- R7 pad 2: /CC_D+ -> Net-(U2-USBDP)
- R70 pad 2: GND -> /AIR_P_DETECTION
- R8 pad 1: /Connectivity/UC_D- -> Net-(U2-USBDM)
- R8 pad 2: /CC_D- -> /D-
- R9 pad 1: /MCU/EN_12V -> GND
- R9 pad 2: GND -> Net-(U10-BOOT0)
- R93 pad 1: +3.3VISO -> +3.3VIO
- R93 pad 2: /ISO_ADC_MISO -> /ADC_MISO
- R96 pad 1: /OUT+ -> /Isolated SPI/OUT+
- R98 pad 1: /OUT- -> /Isolated SPI/OUT-
- R99 pad 1: +3.3VISO -> +3.3VIO
- T1 pad 2: /CCO+ -> unconnected-(T1-PRI_2-Pad2)
- T1 pad 3: /OUT+ -> /CCO+
- T1 pad 4: /OUT- -> /Isolated SPI/OUT+
- TP4 pad 1: /F_+5VISO -> GND
- TP9 pad 1: +3.3V -> +3.3VIO
- U10 pad 10: /MCU/~{FLT} -> /~{FLT}
- U10 pad 11: /MCU/SIGNAL_AMS_ERROR -> unconnected-(U10-PC3-Pad11)
- U10 pad 13: +3.3VIO -> +3.3VMCU
- U10 pad 19: +3.3VIO -> +3.3VMCU
- U10 pad 2: /CD -> unconnected-(U10-PC13-Pad2)
- U10 pad 20: /MCU/~{ADC_CS} -> /~{CS_MISO}
- U10 pad 21: /MCU/ADC_SCK -> /ADC_MISO
- U10 pad 22: /MCU/ADC_MISO -> /ADC_MISO
- U10 pad 23: /MCU/ADC_MOSI -> /ADC_MISO
- U10 pad 24: unconnected-(U10-PC4-Pad24) -> /UCRX
- U10 pad 25: /SAE -> unconnected-(U10-PC5-Pad25)
- U10 pad 26: /SAP -> /VUSB
- U10 pad 27: /SAM -> /MCU/DETECT_WTDG
- U10 pad 28: unconnected-(U10-PB2-Pad28) -> /MCU/SIGNAL_AMS_ERROR
- U10 pad 29: unconnected-(U10-PB10-Pad29) -> /UCTX
- U10 pad 3: /T -> unconnected-(U10-PC14-Pad3)
- U10 pad 32: +3.3VIO -> +3.3VMCU
- U10 pad 33: /MCU/PG_12V -> /SAM
- U10 pad 34: /MCU/EN_12V -> /SAP
- U10 pad 35: /AMD -> /SAE
- U10 pad 36: /AED -> unconnected-(U10-PB15-Pad36)
- U10 pad 37: /FC5 -> /AED
- U10 pad 38: /FC6 -> /AMD
- U10 pad 39: /FC7 -> /APD
- U10 pad 40: /APD -> /CD
- U10 pad 41: /MCU/DETECT_WTDG -> /T
- U10 pad 42: /UART_TX -> /UTX
- U10 pad 43: /UART_RX -> /URX
- U10 pad 44: /Connectivity/UC_D- -> /UART_RX
- U10 pad 45: /Connectivity/UC_D+ -> /UART_TX
- U10 pad 48: +3.3VIO -> +3.3VMCU
- U10 pad 5: /MCU/CLK_IN -> unconnected-(U10-PH0-Pad5)
- U10 pad 50: /MCU/~{COM_CS} -> unconnected-(U10-PA15(JTDI)-Pad50)
- U10 pad 51: /MCU/COM_SCK -> unconnected-(U10-PC10-Pad51)
- U10 pad 52: /MCU/COM_MISO -> unconnected-(U10-PC11-Pad52)
- U10 pad 53: /MCU/COM_MOSI -> unconnected-(U10-PC12-Pad53)
- U10 pad 59: /CRX1 -> /CTX1
- U10 pad 6: /MCU/CLK_OUT -> unconnected-(U10-PH1-Pad6)
- U10 pad 60: unconnected-(U10-BOOT0-Pad60) -> Net-(U10-BOOT0)
- U10 pad 61: /CTX1 -> /CRX1
- U10 pad 64: +3.3VIO -> +3.3VMCU
- U10 pad 8: /MCU/~{ADC_DRY} -> /~{ADC_DRY}
- U10 pad 9: /MCU/SPI_RDY -> unconnected-(U10-PC1-Pad9)
- U12 pad 1: GND -> /T
- U12 pad 2: +24V -> /Connectivity/REF
- U12 pad 3: /MCU/EN_12V -> Net-(U12A-+)
- U12 pad 4: /MCU/PG_12V -> GND
- U12 pad 5: /Power/FB_12V -> Net-(U12B-+)
- U12 pad 6: /Power/VCC_12V -> /Connectivity/REF
- U12 pad 7: /Power/BOOT_12V -> /CD
- U12 pad 8: /Power/SW_12V -> +5VIO
- U13 pad 1: /Connectivity/Input1/REF -> /AED
- U13 pad 2: GND -> /Connectivity/REF
- U13 pad 3: /Connectivity/Input1/IN+ -> Net-(U13A-+)
- U13 pad 4: /T -> GND
- U13 pad 5: +24V -> Net-(U13B-+)
- U2 pad 1: /Connectivity/Input1/REF -> /URX
- U2 pad 2: GND -> unconnected-(U2-~{RTS}-Pad2)
- U2 pad 3: /Connectivity/Input2/IN+ -> /Connectivity/+3.3VFTDI
- U2 pad 4: /CD -> /UTX
- U2 pad 5: +24V -> GND
- U3 pad 2: /MCU/DETECT_WTDG -> Net-(R14-Pad2)
- U3 pad 4: /MCU/DETECT_WTDG -> /MCU/SIGNAL_AMS_ERROR
- U3 pad 5: +3.3V -> +3.3VIO
- U4 pad 1: +5V -> unconnected-(U4-STAT-Pad1)
- U4 pad 3: +5V -> /Power/VSNS
- U4 pad 4: GND -> /Power/ILIM
- U4 pad 5: unconnected-(U4-SYNC_OK-Pad5) -> GND
- U4 pad 6: unconnected-(U4-NC-Pad6) -> /Power/5VUSB
- U4 pad 7: unconnected-(U4-NC-Pad7) -> +5VIO
- U4 pad 8: unconnected-(U4-NC-Pad8) -> /Power/5VPWR
- U6 pad 3: +5V -> +5VIO
- U6 pad 5: +3.3V -> +3.3VIO
- U7 pad 3: +5V -> +5VIO
- U7 pad 5: +3.3V -> +3.3VIO
Routing:
- net +3.3V: track 179.3 -> 0.00 mm, vias 8 -> 0
- net +24V: track 132.9 -> 1.94 mm, vias 15 -> 0
- net +5V: track 122.1 -> 0.00 mm, vias 4 -> 0
- net +3.3VISO: track 104.1 -> 0.00 mm, vias 7 -> 0
- net /Connectivity/UC_D+: track 98.6 -> 0.00 mm, vias 3 -> 0
- net /Connectivity/UC_D-: track 97.6 -> 0.00 mm, vias 3 -> 0
- net VBUS+: track 62.1 -> 0.00 mm, vias 2 -> 0
- net GNDISO: track 57.8 -> 0.00 mm, vias 57 -> 0
- net /NRST: track 56.4 -> 0.00 mm, vias 1 -> 0
- net /FC1: track 54.7 -> 0.00 mm, vias 2 -> 0
- net /SWCLK: track 53.9 -> 0.00 mm, vias 1 -> 0
- net /SDC_AIRS: track 53.4 -> 0.00 mm, vias 5 -> 0
- net /SWDIO: track 50.5 -> 0.00 mm, vias 1 -> 0
- net /FC2: track 50.1 -> 0.00 mm, vias 2 -> 0
- net /LED_ERROR: track 49.9 -> 0.00 mm, vias 2 -> 0
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- added copper zone on In2.Cu, net +3.3VIO
- removed copper zone on B.Cu, net +12V
- removed copper zone on B.Cu, net +24V
- removed copper zone on F.Cu, net +24V
- removed copper zone on B.Cu, net /Power/F_12V
- removed copper zone on F.Cu, net /Power/F_12V
- removed copper zone on B.Cu, net /Power/F_24V
- removed copper zone on F.Cu, net /Power/SW_12V
- removed copper zone on B.Cu, net GND
- removed copper zone on F.Cu, net GND
- removed copper zone on In2.Cu, net GND
- removed copper zone on B.Cu, net GNDISO
- removed copper zone on F.Cu, net GNDISO
- removed copper zone on In1.Cu, net GNDISO
- removed copper zone on In2.Cu, net GNDISO
Other:
- board text added: "8V"
- board text added: "BQ"
- board text added: "MUX5V"
- board text removed: "+"
- board text removed: "-"
- board text removed: "12V"
- board text removed: "3VI"
- board text removed: "5VI"
- board text removed: "AIR FB"
- board text removed: "GNDI"
- board text removed: "INPUTS"
- board text removed: "ISO"
- board text removed: "LEDS"
- board text removed: "TI"
- board text removed: "TRAN"

Commit message: layout
Parts:
- removed C96, C97: 1n, Capacitor_SMD:C_0603_1608Metric
- C93, C94, C95, C98, C99: moved to B.Cu
- moved C77 61.5 mm to (132.5, 62.0), turned to 180 degrees
- moved C10 60.4 mm to (125.5, 72.0), turned to 0 degrees
- moved H1 59.8 mm to (49.0, 32.0)
- moved C98 54.8 mm to (129.0, 72.0), turned to 180 degrees
- moved C95 54.1 mm to (129.0, 62.0), turned to 180 degrees
- moved C18 53.8 mm to (132.5, 60.0), turned to 0 degrees
- moved J4 53.2 mm to (105.5, 95.0), turned to 90 degrees
- moved C99 50.7 mm to (132.5, 72.0), turned to 180 degrees
- moved C59 49.7 mm to (129.0, 60.0)
- moved D1 44.7 mm to (155.5, 104.0)
- moved D6 44.7 mm to (155.5, 106.5)
- moved R34 44.7 mm to (157.0, 104.0)
- moved R36 44.7 mm to (157.0, 106.5)
- moved C55 44.3 mm to (155.0, 72.0), turned to 180 degrees
- moved FB2 40.5 mm to (142.5, 94.5)
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Routing:
- net /SAFETY_IN: track 9.38 -> 19.7 mm
- net /SAFETY_OUT: track 12.4 -> 20.5 mm
Other:
- board text added: "ANALOG PWR"
- board text added: "COM"
- board text added: "INPUTS"
- board text removed: "LTC"

Commit message: sync
Parts:
- moved C3 12.0 mm to (121.8, 138.5)
- moved C6 12.0 mm to (121.8, 143.0)
- moved D14 12.0 mm to (121.8, 143.0)
- moved F8 12.0 mm to (119.5, 138.5)
- moved R32 12.0 mm to (123.8, 138.5)
- moved R35 12.0 mm to (121.8, 138.5)
- moved C11 8.00 mm to (131.8, 142.5)
- moved C12 8.00 mm to (135.2, 140.5)
- moved C17 8.00 mm to (135.2, 138.5)
- moved C21 8.00 mm to (135.2, 142.5)
- moved C22 8.00 mm to (131.8, 138.5)
- moved C26 8.00 mm to (131.8, 140.5)
- moved C68 8.00 mm to (128.2, 138.5)
- moved F4 8.00 mm to (128.2, 140.5)
- moved IC2 8.00 mm to (135.2, 140.5)
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Connections:
- IC8 pad 12: /ADC_MISO -> /ADC_SCK
- IC8 pad 14: /ADC_MISO -> /ADC_MOSI
- U10 pad 21: /ADC_MISO -> /ADC_SCK
- U10 pad 23: /ADC_MISO -> /ADC_MOSI
Routing:
- net GND: track 23.5 -> 122.8 mm, vias 19 -> 93
- net +5VIO: track 7.24 -> 35.0 mm, vias 4 -> 12
- net /SDC_AIRS: track 0.00 -> 24.1 mm, vias 0 -> 10
- net /Connectivity/REF: track 0.00 -> 23.6 mm, vias 0 -> 1
- net /Isolated SPI/OUT-: track 0.00 -> 20.5 mm
- net /Isolated SPI/OUT+: track 0.00 -> 20.0 mm
- net +3.3VIO: track 6.66 -> 26.0 mm, vias 5 -> 18
- net +8V: track 0.00 -> 15.7 mm, vias 0 -> 1
- net /CCO-: track 0.00 -> 11.5 mm
- net /CCO+: track 0.00 -> 11.5 mm
- net +24V: track 1.94 -> 11.4 mm, vias 0 -> 2
- net /AIR_P-: track 0.00 -> 8.21 mm, vias 0 -> 1
- net /ADC/I+: track 0.00 -> 7.78 mm
- net /AIR_M-: track 0.00 -> 7.72 mm, vias 0 -> 1
- net VBUS+: track 0.00 -> 7.26 mm, vias 0 -> 1
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
Commit message: sync
Parts:
- turned D14 to 0 degrees
Routing:
- net GND: track 122.8 -> 150.6 mm, vias 93 -> 109
- net +24V: track 11.4 -> 37.4 mm, vias 2 -> 3
- net /IsolationBarrier/CAR_GND: track 0.00 -> 12.6 mm, vias 0 -> 4
- net /Power/FB_5V: track 0.00 -> 12.0 mm, vias 0 -> 1
- net /Power/F_5V: track 0.00 -> 12.0 mm, vias 0 -> 1
- net Net-(D5-A): track 0.00 -> 11.9 mm, vias 0 -> 1
- net /Power/F_24V: track 0.00 -> 11.8 mm, vias 0 -> 3
- net /IsolationBarrier/CAR+: track 0.00 -> 11.3 mm, vias 0 -> 1
- net /IsolationBarrier/ACU+: track 0.00 -> 11.3 mm, vias 0 -> 1
- net /IsolationBarrier/ACU_GND: track 0.00 -> 11.1 mm, vias 0 -> 4
- net VDD: track 0.00 -> 9.03 mm
- net /IsolationBarrier/ACU_DCDC: track 0.00 -> 8.08 mm, vias 0 -> 1
- net /IsolationBarrier/CAR_DCDC: track 0.00 -> 8.06 mm, vias 0 -> 1
- net /Power/EN_5V: track 0.00 -> 5.15 mm, vias 0 -> 1
- net /Power/SW_5V: track 0.00 -> 4.63 mm, vias 0 -> 1
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- added copper zone on In1.Cu, net /IsolationBarrier/ACU_GND
- added copper zone on In2.Cu, net /IsolationBarrier/ACU_GND
- added copper zone on In1.Cu, net /IsolationBarrier/CAR_GND

Commit message: sync
Parts:
- moved R7 7.04 mm to (150.2, 104.2)
- moved C34 6.18 mm to (144.5, 109.0), turned to 0 degrees
- moved R9 4.51 mm to (138.2, 113.8), turned to 180 degrees
- moved U2 4.30 mm to (144.5, 106.5), turned to 90 degrees
- moved D12 4.00 mm to (151.0, 108.5)
- moved R8 3.69 mm to (151.8, 104.2)
- moved C44 3.64 mm to (144.5, 104.0), turned to 180 degrees
- moved D21 3.50 mm to (114.2, 89.5)
- moved D22 3.50 mm to (114.2, 93.5)
- moved C36 2.36 mm to (133.0, 116.2), turned to 90 degrees
- moved C70 2.36 mm to (135.2, 116.2), turned to 90 degrees
- moved R3 2.00 mm to (138.2, 117.2)
- moved C86 0.79 mm to (129.8, 118.2)
- moved C43 0.25 mm to (121.8, 90.2)
- moved C53 0.25 mm to (119.2, 91.2)
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Connections:
- net /MCU/DETECT_WTDG renamed /DETERR
- net /VUSB renamed /DETVUSB
- net Net-(U2-USBDM) renamed /Connectivity/FTDIU-
- net Net-(U2-USBDP) renamed /Connectivity/FTDIU+
- Q8 pad 1: /MCU/SIGNAL_AMS_ERROR -> /Safety/LATCHERR
- Q8 pad 3: /AMS_ERROR -> /AMSERR
- Q9 pad 1: /AMS_ERROR -> /AMSERR
- R13 pad 1: /AMS_ERROR -> /AMSERR
- R38 pad 1: /MCU/SIGNAL_AMS_ERROR -> /Safety/LATCHERR
- U10 pad 28: /MCU/SIGNAL_AMS_ERROR -> /AMSERR
- U3 pad 4: /MCU/SIGNAL_AMS_ERROR -> /Safety/LATCHERR
Routing:
- net /CAR_I: track 0.00 -> 20.9 mm
- net GND: track 150.6 -> 170.2 mm, vias 109 -> 119
- net +3.3VMCU: track 0.00 -> 18.2 mm, vias 0 -> 6
- net /D+: track 2.79 -> 15.9 mm
- net /D-: track 3.18 -> 15.4 mm
- net /CANFD1-: track 2.57 -> 14.2 mm
- net /CANFD2-: track 2.57 -> 14.2 mm
- net /CANFD2+: track 2.57 -> 13.6 mm
- net /CANFD1+: track 2.57 -> 13.6 mm
- net /Safety/LATCHERR: track 0.00 -> 10.1 mm, vias 0 -> 1
- net /MCU/SIGNAL_AMS_ERROR: track 10.1 -> 0.00 mm, vias 1 -> 0
- net VDD: track 9.03 -> 0.00 mm
- net +5VA: track 2.62 -> 10.8 mm, vias 1 -> 2
- net /Connectivity/FTDIU+: track 1.62 -> 7.97 mm
- net /Connectivity/FTDIU-: track 1.62 -> 7.95 mm
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Other:
- board text added: "LEDS"
