File: hardware/mainboard/PUTM_EV_AMS_MASTER_2025.kicad_pcb (KiCad board)
At the start: 4 copper layers, 60 x 100 mm, 207 parts, among them IC1 3.3V/0.5A, IC2 TPS54202HDDCR, IC3 BQ79600PWRQ1, IC6 AMC3330DWER, IC7 AMC3330DWER, IC8 ADC 24bit, IC9 LTC1799, J1 M80-5100642, J10 M300-MV10345M1, J2 M80-5102042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

Commit message: isolated side, choose most components, some master changes tbc
Parts:
- removed TP2: TestPoint_Small, MountingHole:MountingHole_3.2mm_M3_Pad_Via
- added H3: M3, MountingHole:MountingHole_3.2mm_M3, F.Cu at (158.5, 144.5)
Routing:
- net /CTSMS: track 9.22 -> 10.1 mm, vias 0 -> 1
- net +3.3VIO: track 29.5 -> 28.6 mm, vias 19 -> 18

Commit message: chore: sync
Parts:
- moved R17 56.1 mm to (182.8, 91.5)
- moved R26 56.1 mm to (182.8, 87.5)
- moved C101 56.1 mm to (185.5, 91.5)
- moved C102 56.1 mm to (185.5, 87.5)
- moved C103 56.1 mm to (189.2, 91.5)
- moved C104 56.1 mm to (189.2, 87.5)
- moved C105 56.1 mm to (193.0, 91.5)
- moved R20 56.1 mm to (185.5, 93.8)
- moved R21 56.1 mm to (185.5, 85.2)
- moved R25 56.1 mm to (189.2, 93.8)
Routing:
- net /ERROR_RELAY-: track 130.1 -> 0.00 mm
