File: hardware/mainboard/Connectivity.kicad_sch (KiCad schematic)
At the start: 18 parts, among them U6 MCP2542FD-E/MF, U7 MCP2542FD-E/MF

Commit message: sync
Parts:
- removed D22: ESDA5V3SC5, Package_TO_SOT_SMD:SOT-23-6, symbol Power_Protection:ESDA5V3SC5
- removed R39, R40: 33, Resistor_SMD:R_0603_1608Metric, symbol Device:R_Small
Connections:
- net GND: no longer D11.2 (K), D11.5 (NC)
- net EX_D+: no longer names the net of R7.2
- net EX_D-: no longer names the net of R8.2
- removed net UC_D+: D11.3 (A), D11.4 (A), R7.1
- removed net UC_D-: D11.1 (A), D11.6 (A), R8.1
- new net: D11.2 (K), D11.5 (NC)

Commit message: schematic?
Parts:
- removed C60: 100nF, Capacitor_SMD:C_0603_1608Metric, symbol Device:C_Small
- removed D11: ESDA5V3SC5, Package_TO_SOT_SMD:SOT-23-6, symbol Power_Protection:ESDA5V3SC5
- added C101, C102, C103, C104, C105: 10nF, Capacitor_SMD:C_0603_1608Metric, symbol Device:C_Small
- added C34, C44, C49, C50, C58: 100nF, Capacitor_SMD:C_0603_1608Metric, symbol Device:C_Small
- added D11, D12, D4: 5.3V/400W, Package_TO_SOT_SMD:SOT-23-3, symbol Power_Protection:ESDA5V3L
- added R20, R21, R25, R41: 10k, Resistor_SMD:R_0603_1608Metric, symbol Device:R_Small
- added R49, R53, R63, R68: 100k, Resistor_SMD:R_0603_1608Metric, symbol Device:R_Small
- added U12, U13, U14: LM393, Package_SO:VSSOP-8_3x3mm_P0.65mm, symbol Comparator:LM393
- added U2: FT230XS, Package_SO:SSOP-16_3.9x4.9mm_P0.635mm, symbol Interface_USB:FT230XS
- R17: value 10k -> 20k
- R7, R8: value 33 -> 27
- R70: value 10k -> 100k
Connections:
- net EX_AIR_AUX_M: now also R68.2
- net EX_AIR_AUX_P: now also R70.2
- net EX_AIR_AUX_PRE: now also R63.2
- net EX_CANFD1+: now also D4.1 (K)
- net EX_CANFD1-: now also D4.2 (K)
- net EX_CANFD2+: now also D11.1 (K)
- net EX_CANFD2-: now also D11.2 (K)
- net EX_IN1: now also R49.2
- net EX_IN2: now also R53.2
- net GND: now also R42.1, C101.1, C102.1, C103.1, C104.1, C105.1, C34.2, C44.2, C49.2, C50.2, C58.2, D11.3 (A), D12.3 (A), D4.3 (A), R20.1, R21.1, R25.1, R41.1, U12.4 (V-), U13.4 (V-), U14.4 (V-), U14.5 (+), U14.6 (-), U14.7, U2.13 (GND), U2.5 (GND); no longer R70.2
- net UC_AIR_AUX_M: now also U13.7
- net UC_AIR_AUX_P: now also U14.1
- net UC_AIR_AUX_PRE: now also U13.1
- net UC_IN1: now also U12.1
- net UC_IN2: now also U12.7
- net at R8.1: now also U2.9 (USBDM)
- net EX_D-: now reaches R8.2
- net EX_D-: now also D12.2 (K)
- net EX_D+: now reaches R7.1
- net EX_D+: now also D12.1 (K)
- net at R7.2: now also U2.8 (USBDP)
- net +3.3V renamed +3.3VIO
- net +3.3VIO: no longer R42.1
- net +5V renamed +5VIO
- net +5VIO: now also C44.1, C49.1, C50.1, C58.1, U12.8 (V+), U13.8 (V+), U14.8 (V+), U2.12 (VCC)
- net AIR Minus/REF: no longer names the net of R42.2, R70.1
- net AIR Minus/REF: now also C105.2, U14.3 (+)
- net Input1/REF renamed REF
- net REF: now also U12.2 (-), U12.6 (-), U13.2 (-), U13.6 (-), U14.2 (-)
- new net: C101.2, R20.2, R49.1, U12.3 (+)
- new net: C103.2, R25.2, R63.1, U13.3 (+)
- new net: C104.2, R41.2, R68.1, U13.5 (+)
- new net: C102.2, R21.2, R53.1, U12.5 (+)
- new net +3.3VFTDI: C34.1, U2.10 (3V3OUT), U2.11 (~{RESET}), U2.3 (VCCIO)
- new net FTDI_RX: U2.4 (RXD)
- new net FTDI_TX: U2.1 (TXD)
- no-connect marks 0 -> 6
Other:
- removed sheet AIR Minus
- removed sheet AIR Plus
- removed sheet AIR Precharge
- removed sheet Input1
- removed sheet Input2
- note added: "INPUTS SEPERATION"
- note removed: "AIR FEEDBACK SEPERATION"
- note removed: "MCU MAIN CC USB"
- note removed: "REF2"
- note removed: "TSMS & CHARGER DETECET"
- moved on the sheet: C32, C33, C37, C38, C76, R17, R26, R7, R8, U6, U7

Commit message: sync
Connections:
- net FTDIU-: now reaches R8.1, U2.9 (USBDM)
- net FTDIU+: now reaches R7.2, U2.8 (USBDP)
Changed lines of the file:
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@@
+		)
+	)
+	(label "FTDIU+"
+		(at 365.6598 73.66 180)
+		(effects
+			(font
+				(size 0.508 0.508)
+			)
+			(justify right bottom)
 		)
 	)
@@
 		(effects
 			(font
+				(size 0.508 0.508)
+			)
+			(justify right bottom)
+		)
+	)
+	(label "FTDIU-"
+		(at 365.76 71.12 180)
+		(effects
+			(font

Commit message: hardware routing done, only touch ups will be needed if the board is aproved
Connections:
- net +3.3VIO: now also C49.1, C50.1, C58.1, U12.8 (V+), U13.8 (V+), U14.8 (V+)
- net +5VIO: no longer C49.1, C50.1, C58.1, U12.8 (V+), U13.8 (V+), U14.8 (V+)
Changed lines of the file:
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@@
 	)
 	(symbol
-		(lib_id "power:+5V")
-		(at 53.34 68.58 0)
-		(unit 1)
-		(exclude_from_sim no)
-		(in_bom yes)
-		(on_board yes)
-		(dnp no)
-		(property "Reference" "#PWR032"
-			(at 53.34 72.39 0)
-			(effects
-				(font
-					(size 1.27 1.27)
-				)
-				(hide yes)
-			)
-		)
-		(property "Value" "+5VIO"
-			(at 53.34 64.77 0)
-			(effects
-				(font
-					(size 1.27 1.27)
-				)
-			)
-		)
-		(property "Footprint" ""
-			(at 53.34 68.58 0)
-			(effects
-				(font
-					(size 1.27 1.27)
-				)
-				(hide yes)
-			)
-		)
-		(property "Datasheet" ""
-			(at 53.34 68.58 0)
-			(effects
-				(font
-					(size 1.27 1.27)
-				)
-				(hide yes)
-			)
-		)
-		(property "Description" ""
-			(at 53.34 68.58 0)
-			(effects
-				(font
-					(size 1.27 1.27)
-				)
-				(hide yes)
-			)
-		)
-		(pin "1"
-		)
-		(instances
-			(project "PUTM_EV_AMS_MASTER_2025"
-				(path "/b456cffc-d9d7-4c91-91f2-36ec9a65dd1b/c7d64097-44d3-49d9-9a80-8f2f4ff55e04"
-					(reference "#PWR032")
-					(unit 1)
-				)
-			)
-		)
-	)
-	(symbol
 		(lib_id "Comparator:LM393")
 		(at 105.41 68.58 0)
@@
 	)
 	(symbol
-		(lib_id "power:+5V")
-		(at 53.34 124.46 0)
-		(unit 1)
-		(exclude_from_sim no)
-		(in_bom yes)
-		(on_board yes)
-		(dnp no)
-		(property "Reference" "#PWR040"
-			(at 53.34 128.27 0)
-			(effects
-				(font
-					(size 1.27 1.27)
-				)
-				(hide yes)
-			)
-		)
-		(property "Value" "+5VIO"
-			(at 53.34 120.65 0)
-			(effects
-				(font
-					(size 1.27 1.27)
-				)
-			)
-		)
-		(property "Footprint" ""
-			(at 53.34 124.46 0)
-			(effects
-				(font
-					(size 1.27 1.27)
-				)
-				(hide yes)
-			)
-		)
-		(property "Datasheet" ""
-			(at 53.34 124.46 0)
-			(effects
-				(font
-					(size 1.27 1.27)
-				)
-				(hide yes)
-			)
-		)
-		(property "Description" ""
-			(at 53.34 124.46 0)
-			(effects
-				(font
-					(size 1.27 1.27)
-				)
-				(hide yes)
-			)
-		)
-		(pin "1"
-		)
-		(instances
-			(project "PUTM_EV_AMS_MASTER_2025"
-				(path "/b456cffc-d9d7-4c91-91f2-36ec9a65dd1b/c7d64097-44d3-49d9-9a80-8f2f4ff55e04"
-					(reference "#PWR040")
-					(unit 1)
-				)
-			)
-		)
-	)
-	(symbol
 		(lib_name "GND_1")
 		(lib_id "power:GND")
@@
 	)
 	(symbol
-		(lib_id "power:+5V")
-		(at 53.34 182.88 0)
-		(unit 1)
-		(exclude_from_sim no)
-		(in_bom yes)
-		(on_board yes)
-		(dnp no)
-		(property "Reference" "#PWR042"
-			(at 53.34 186.69 0)
-			(effects
-				(font
-					(size 1.27 1.27)
-				)
-				(hide yes)
-			)
-		)
-		(property "Value" "+5VIO"
-			(at 53.34 179.07 0)
-			(effects
-				(font
-					(size 1.27 1.27)
-				)
-			)
-		)
-		(property "Footprint" ""
-			(at 53.34 182.88 0)
-			(effects
-				(font
-					(size 1.27 1.27)
-				)
-				(hide yes)
-			)
-		)
-		(property "Datasheet" ""
-			(at 53.34 182.88 0)
-			(effects
-				(font
-					(size 1.27 1.27)
-				)
-				(hide yes)
-			)
-		)
-		(property "Description" ""
-			(at 53.34 182.88 0)
-			(effects
-				(font
-					(size 1.27 1.27)
-				)
-				(hide yes)
-			)
-		)
-		(pin "1"
-		)
-		(instances
-			(project "PUTM_EV_AMS_MASTER_2025"
-				(path "/b456cffc-d9d7-4c91-91f2-36ec9a65dd1b/c7d64097-44d3-49d9-9a80-8f2f4ff55e04"
-					(reference "#PWR042")
-					(unit 1)
-				)
-			)
-		)
-	)
-	(symbol
 		(lib_id "Device:C_Small")
 		(at 201.93 92.71 90)
@@
 	)
 	(symbol
+		(lib_id "power:+3.3V")
+		(at 53.34 182.88 0)
+		(unit 1)
+		(exclude_from_sim no)
+		(in_bom yes)
+		(on_board yes)
+		(dnp no)
+		(property "Reference" "#PWR0124"
+			(at 53.34 186.69 0)
+			(effects
+				(font
+					(size 1.27 1.27)
+				)
+				(hide yes)
+			)
+		)
+		(property "Value" "+3.3VIO"
+			(at 53.34 179.07 0)
+			(effects
+				(font
+					(size 1.27 1.27)
+				)
+			)
+		)
+		(property "Footprint" ""
+			(at 53.34 182.88 0)
+			(effects
+				(font
+					(size 1.27 1.27)
+				)
+				(hide yes)
+			)
+		)
+		(property "Datasheet" ""
+			(at 53.34 182.88 0)
+			(effects
+				(font
+					(size 1.27 1.27)
+				)
+				(hide yes)
+			)
+		)
+		(property "Description" ""
+			(at 53.34 182.88 0)
+			(effects
+				(font
+					(size 1.27 1.27)
+				)
+				(hide yes)
+			)
+		)
+		(pin "1"
+		)
+		(instances
+			(project "PUTM_EV_AMS_MASTER_2025"
+				(path "/b456cffc-d9d7-4c91-91f2-36ec9a65dd1b/c7d64097-44d3-49d9-9a80-8f2f4ff55e04"
+					(reference "#PWR0124")
+					(unit 1)
+				)
+			)
+		)
+	)
+	(symbol
 		(lib_id "Comparator:LM393")
 		(at 60.96 137.16 0)
@@
 	)
 	(symbol
+		(lib_id "power:+3.3V")
+		(at 53.34 124.46 0)
+		(unit 1)
+		(exclude_from_sim no)
+		(in_bom yes)
+		(on_board yes)
+		(dnp no)
+		(property "Reference" "#PWR0123"
+			(at 53.34 128.27 0)
+			(effects
+				(font
+					(size 1.27 1.27)
+				)
+				(hide yes)
+			)
+		)
+		(property "Value" "+3.3VIO"
+			(at 53.34 120.65 0)
+			(effects
+				(font
+					(size 1.27 1.27)
+				)
+			)
+		)
+		(property "Footprint" ""
+			(at 53.34 124.46 0)
+			(effects
+				(font
+					(size 1.27 1.27)
+				)
+				(hide yes)
+			)
+		)
+		(property "Datasheet" ""
+			(at 53.34 124.46 0)
+			(effects
+				(font
+					(size 1.27 1.27)
+				)
+				(hide yes)
+			)
+		)
+		(property "Description" ""
+			(at 53.34 124.46 0)
+			(effects
+				(font
+					(size 1.27 1.27)
+				)
+				(hide yes)
+			)
+		)
+		(pin "1"
+		)
+		(instances
+			(project "PUTM_EV_AMS_MASTER_2025"
+				(path "/b456cffc-d9d7-4c91-91f2-36ec9a65dd1b/c7d64097-44d3-49d9-9a80-8f2f4ff55e04"
+					(reference "#PWR0123")
+					(unit 1)
+				)
+			)
+		)
+	)
+	(symbol
 		(lib_id "power:+5V")
 		(at 214.63 29.21 0)
@@
 					(unit 1)
 				)
+			)
+		)
+	)
+	(symbol
+		(lib_id "power:+3.3V")
+		(at 53.34 68.58 0)
+		(unit 1)
+		(exclude_from_sim no)
+		(in_bom yes)
+		(on_board yes)
+		(dnp no)
+		(property "Reference" "#PWR0122"
+			(at 53.34 72.39 0)
+			(effects
+				(font
+					(size 1.27 1.27)
+				)
+				(hide yes)
+			)
+		)
+		(property "Value" "+3.3VIO"
+			(at 53.34 64.77 0)
+			(effects
+				(font
+					(size 1.27 1.27)
+				)
+			)
+		)
+		(property "Footprint" ""
+			(at 53.34 68.58 0)
+			(effects
+				(font
+					(size 1.27 1.27)
+				)
+				(hide yes)
+			)
+		)
+		(property "Datasheet" ""
+			(at 53.34 68.58 0)
+			(effects
+				(font
+					(size 1.27 1.27)
+				)
+				(hide yes)
+			)
+		)
+		(property "Description" ""
+			(at 53.34 68.58 0)
+			(effects
+				(font
+					(size 1.27 1.27)
+				)
+				(hide yes)
+			)
+		)
+		(pin "1"
+		)
+		(instances
+			(project "PUTM_EV_AMS_MASTER_2025"
+				(path "/b456cffc-d9d7-4c91-91f2-36ec9a65dd1b/c7d64097-44d3-49d9-9a80-8f2f4ff55e04"
+					(reference "#PWR0122")
+					(unit 1)
+				)

Commit message: v3.3
Connections:
- net +3.3VIO: now also U14.6 (-)
- net GND: no longer U14.6 (-)
Changed lines of the file:
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@@
 	)
 	(junction
-		(at 115.57 212.09)
-		(diameter 0)
-		(color 0 0 0 0)
-	)
-	(junction
 		(at 261.62 107.95)
 		(diameter 0)
@@
 	(wire
 		(pts
+			(xy 118.11 207.01) (xy 118.11 214.63)
+		)
+		(stroke
+			(width 0)
+			(type default)
+		)
+	)
+	(wire
+		(pts
 			(xy 130.81 66.04) (xy 130.81 68.58)
 		)
@@
 	(wire
 		(pts
-			(xy 115.57 212.09) (xy 115.57 214.63)
-		)
-		(stroke
-			(width 0)
-			(type default)
-		)
-	)
-	(wire
-		(pts
 			(xy 356.87 63.5) (xy 356.87 53.34)
 		)
@@
 	(wire
 		(pts
-			(xy 115.57 207.01) (xy 115.57 212.09)
-		)
-		(stroke
-			(width 0)
-			(type default)
-		)
-	)
-	(wire
-		(pts
 			(xy 196.85 118.11) (xy 196.85 110.49)
 		)
@@
 	(wire
 		(pts
+			(xy 115.57 201.93) (xy 115.57 212.09)
+		)
+		(stroke
+			(width 0)
+			(type default)
+		)
+	)
+	(wire
+		(pts
 			(xy 95.25 209.55) (xy 95.25 212.09)
 		)
@@
 	(wire
 		(pts
-			(xy 113.03 207.01) (xy 115.57 207.01)
+			(xy 113.03 207.01) (xy 118.11 207.01)
 		)
 		(stroke
@@
 	)
 	(symbol
+		(lib_id "power:+3.3V")
+		(at 115.57 201.93 0)
+		(unit 1)
+		(exclude_from_sim no)
+		(in_bom yes)
+		(on_board yes)
+		(dnp no)
+		(property "Reference" "#PWR0125"
+			(at 115.57 205.74 0)
+			(effects
+				(font
+					(size 1.27 1.27)
+				)
+				(hide yes)
+			)
+		)
+		(property "Value" "+3.3VIO"
+			(at 115.57 198.12 0)
+			(effects
+				(font
+					(size 1.27 1.27)
+				)
+			)
+		)
+		(property "Footprint" ""
+			(at 115.57 201.93 0)
+			(effects
+				(font
+					(size 1.27 1.27)
+				)
+				(hide yes)
+			)
+		)
+		(property "Datasheet" ""
+			(at 115.57 201.93 0)
+			(effects
+				(font
+					(size 1.27 1.27)
+				)
+				(hide yes)
+			)
+		)
+		(property "Description" ""
+			(at 115.57 201.93 0)
+			(effects
+				(font
+					(size 1.27 1.27)
+				)
+				(hide yes)
+			)
+		)
+		(pin "1"
+		)
+		(instances
+			(project "PUTM_EV_AMS_MASTER_2025"
+				(path "/b456cffc-d9d7-4c91-91f2-36ec9a65dd1b/c7d64097-44d3-49d9-9a80-8f2f4ff55e04"
+					(reference "#PWR0125")
+					(unit 1)
+				)
+			)
+		)
+	)
+	(symbol
 		(lib_id "Device:C_Small")
 		(at 334.01 48.26 270)
@@
 		(lib_name "GND_7")
 		(lib_id "power:GND")
-		(at 115.57 214.63 0)
+		(at 118.11 214.63 0)
 		(unit 1)
 		(exclude_from_sim no)
@@
 		(dnp no)
 		(property "Reference" "#PWR0116"
-			(at 115.57 220.98 0)
+			(at 118.11 220.98 0)
 			(effects
 				(font
@@
 		)
 		(property "Value" "GND"
-			(at 115.697 219.0242 0)
+			(at 118.237 219.0242 0)
 			(effects
 				(font
@@
 		)
 		(property "Footprint" ""
-			(at 115.57 214.63 0)
+			(at 118.11 214.63 0)
 			(effects
 				(font
@@
 		)
 		(property "Datasheet" ""
-			(at 115.57 214.63 0)
+			(at 118.11 214.63 0)
 			(effects
 				(font
@@
 		)
 		(property "Description" ""
-			(at 115.57 214.63 0)
+			(at 118.11 214.63 0)
 			(effects
 				(font

Commit message: isolation with every thing
Parts:
- removed C32, C33, C37, C38, C49, C50, C58, C76: 100nF, Capacitor_SMD:C_0603_1608Metric, symbol Device:C_Small
- removed R41, R42: 10k, Resistor_SMD:R_0603_1608Metric, symbol Device:R_Small
- removed R49, R53, R63, R68, R70: 100k, Resistor_SMD:R_0603_1608Metric, symbol Device:R_Small
- removed U12, U13, U14: LM393, Package_SO:VSSOP-8_3x3mm_P0.65mm, symbol Comparator:LM393
- removed U6, U7: MCP2542FD-E/MF, Package_DFN_QFN:DFN-8-1EP_3x3mm_P0.65mm_EP1.55x2.4mm, symbol Interface_CAN_LIN:MCP2542FDxMF
- added D25, D26: 3.6V/400W, Package_TO_SOT_SMD:SOT-23-6, symbol Power_Protection:ESDA5V3SC5
- added R15, R18, R19, R69: 27, Resistor_SMD:R_0603_1608Metric, symbol Device:R_Small
- added R71: 10k, Resistor_SMD:R_0603_1608Metric, symbol Device:R_Small
- R17: value 20k -> 27; Mouser Part Number -- -> 71-CRCW060333R0FKEC
- R20, R21, R25, R26: value 10k -> 27; Mouser Part Number -- -> 71-CRCW060333R0FKEC
Connections:
- net +3.3VIO is gone; now on net UC_IN1: R17.1
- net +3.3VFTDI: now also R71.1; no longer U2.11 (~{RESET})
- net EX_AIR_AUX_M: now also R25.2
- net EX_AIR_AUX_P: now also R26.2
- net EX_AIR_AUX_PRE: now also R21.2
- net EX_IN1: now also R17.2
- net EX_IN2: now also R20.2
- net GND: now also D25.2 (K), D25.5 (NC), D26.2 (K), D26.5 (NC); no longer R20.1, R21.1, R25.1, R26.2
- net UC_AIR_AUX_M: now also C104.2, R25.1, D25.3 (A)
- net UC_AIR_AUX_P: now also C105.2, R26.1, D25.4 (A)
- net UC_AIR_AUX_PRE: now also C103.2, R21.1, D25.1 (A)
- net UC_CANFD1_RX: now also R69.2
- net UC_CANFD1_TX: now also R19.1
- net UC_CANFD2_RX: now also R18.2
- net UC_CANFD2_TX: now also R15.1
- net UC_IN1: now also C101.2, D26.1 (A)
- net UC_IN2: now also C102.2, R20.1, D26.3 (A)
- net EX_CANFD1+ renamed EX_CANFD1_TX
- net EX_CANFD1_TX: now also R19.2
- net EX_CANFD1- renamed EX_CANFD1_RX
- net EX_CANFD1_RX: now also R69.1
- net EX_CANFD2+ renamed EX_CANFD2_TX
- net EX_CANFD2_TX: now also R15.2
- net EX_CANFD2- renamed EX_CANFD2_RX
- net EX_CANFD2_RX: now also R18.1
- removed net REF: R17.2, R26.1
- new net ~{FTDI_RST}: R71.2, U2.11 (~{RESET})
- no-connect marks 6 -> 9
Other:
- note removed: "REF1"
- moved on the sheet: C101, C102, C34, C44, D11, D12, D4, R7, R8, U2
