File: hardware/mainboard/Connectivity.kicad_sch (KiCad schematic)
At the start: 4 parts

Commit message: done
Parts:
- removed D31: 3.6V/400W, Package_TO_SOT_SMD:SOT-23-6, symbol Power_Protection:ESDA5V3SC5
Connections:
- net EX_AIR_AUX_M is gone; now on net EX_CANFD1_TX: D25.3 (A)
- net EX_AIR_AUX_P is gone; now on net EX_CANFD2_TX: D25.4 (A)
- net EX_AIR_AUX_PRE is gone; now on net EX_CANFD1_RX: D25.1 (A)
- net EX_CANFD2_RX: now also D25.6 (A)
- net EX_IN1: now also D26.6 (A)
- net EX_IN2: now also D26.4 (A)
- net EX_USB_DET: now reaches D29.6 (A)
- no-connect marks 4 -> 0
Other:
- moved on the sheet: D25, D29
