File: hardware/mainboard/AirControl.kicad_sch (KiCad schematic)
At the start: 23 parts, among them Q1 DMT6018LDR-7, Q7 DMT6018LDR-7

Commit message: isolation with every thing
Parts:
- removed C15, C51, C61, C62, C69: 22uF, Capacitor_SMD:C_0805_2012Metric, symbol Device:C_Small
- removed C63, C64: 22uF, Capacitor_SMD:CP_Elec_4x5.8, symbol Device:C_Polarized_Small
- removed D15: 60V/0.5/3A, Diode_SMD:D_SOD-123, symbol Device:D_Small
- removed TP11: TestPoint_Small, TestPoint:TestPoint_THTPad_D1.0mm_Drill0.5mm, symbol Connector:TestPoint_Small
Connections:
- net VDD renamed +24V
Other:
- note removed: "VDD DECOUPLING"

Commit message: chore: sync
Parts:
- removed C83, C84, C85: 100nF, Capacitor_SMD:C_0603_1608Metric, symbol Device:C_Small
