File: hardware/mainboard/PUTM_EV_AMS_MASTER_2025.kicad_sch (KiCad schematic)
At the start: 22 parts, among them J1 M80-5100642, J10 M300-MV10345M1, J2 M80-5102042, J3 M80-5100842, J4 FTSH-107-01-L-D-K, J5 M80-51004XX, J7 M300-MV10345M1, J8 M80-51004XX, T1 SM91502ALE

Commit message: chore: sync
Parts:
- removed J1: M80-5100642, Samacsys:M80-51006YY, symbol Samacsys_kicad_sym:M80-5100642
- removed J2: M80-5102042, Samacsys:M80-51020YY, symbol Samacsys_kicad_sym:M80-5102042
- removed J3: M80-5100842, Samacsys:M80-51008YY, symbol Samacsys_kicad_sym:M80-5100842
