File: hardware/mainboard/Power.kicad_sch (KiCad schematic)
At the start: 49 parts, among them IC1 3.3V/0.5A, IC2 TPS54202HDDCR, U12 LMR33640DDDA

Commit message: sync
Parts:
- removed C10: 100nF, Capacitor_SMD:C_0603_1608Metric, symbol Device:C_Small
- removed C16, C19, C20, C52, C54, C55: 22uF, Capacitor_SMD:C_0805_2012Metric, symbol Device:C_Small
- removed C4: 220nF, Capacitor_SMD:C_0603_1608Metric, symbol Device:C_Small
- removed C9: 1uF, Capacitor_SMD:C_0603_1608Metric, symbol Device:C_Small
- removed F3: 12V/4A, Fuse:Fuse_1206_3216Metric, symbol Device:Polyfuse_Small
- removed L2: 6.8uF/3.5A, Inductor_SMD:L_TDK_VLS6045EX_VLS6045AF, symbol Samacsys_kicad_sym:SRR4028-271Y
- removed R10, R9: 10k, Resistor_SMD:R_0603_1608Metric, symbol Device:R_Small
- removed R24: 9.09k, Resistor_SMD:R_0603_1608Metric, symbol Device:R_Small
- removed R25: 100k, Resistor_SMD:R_0603_1608Metric, symbol Device:R_Small
- removed U12: LMR33640DDDA, Package_SO:Texas_HSOP-8-1EP_3.9x4.9mm_P1.27mm, symbol Regulator_Switching:LMR33640DDDA
Other:
- note removed: "12V"

Commit message: schematic?
Parts:
- removed D4, D5: 60V/0.5/3A, Diode_SMD:D_SOD-123, symbol Device:D_Schottky_Small
- removed TP10: TestPoint_Small, TestPoint:TestPoint_THTPad_D1.0mm_Drill0.5mm, symbol Connector:TestPoint_Small
- added C19, C20, C4, C5: 2.2uF, Capacitor_SMD:C_0603_1608Metric, symbol Device:C_Small
- added C30, C31: 22uF, Capacitor_SMD:C_0805_2012Metric, symbol Device:C_Small
- added C39, C40, C42: 100nF, Capacitor_SMD:C_0603_1608Metric, symbol Device:C_Small
- added D20: 8V, Diode_SMD:D_SOD-123, symbol Device:D_Zener_Small
- added D5: 10V, Diode_SMD:D_SOD-123, symbol Device:D_Zener_Small
- added FB1, FB2: 100@100Mhz, Inductor_SMD:L_0603_1608Metric, symbol Device:FerriteBead_Small
- added IC4: TLV61046ADBVT, Package_TO_SOT_SMD:SOT-23-6, symbol Samacsys_kicad_sym:TLV61046ADBVT
- added L1: 10uH, Inductor_SMD:L_1008_2520Metric, symbol Device:L
- added Q4: SI2347DS-T1-GE3, Package_TO_SOT_SMD:SOT-23-3, symbol Transistor_FET:Q_PMOS_GSD
- added R10: 100k, Resistor_SMD:R_0603_1608Metric_Pad0.98x0.95mm_HandSolder, symbol Device:R_Small
- added R16: 20k, Resistor_SMD:R_0603_1608Metric, symbol Device:R_Small
- added R32: 10k, Resistor_SMD:R_0603_1608Metric, symbol Device:R_Small
- added R35, R39: 100k, Resistor_SMD:R_0603_1608Metric, symbol Device:R_Small
- added R40: 400, Resistor_SMD:R_0603_1608Metric, symbol Device:R_Small
- added R55: 649k, Resistor_SMD:R_0603_1608Metric, symbol Device:R_Small
- added R62: 71.5k, Resistor_SMD:R_0603_1608Metric, symbol Device:R_Small
- added U4: TPS2113PWR, Package_SO:TSSOP-8_4.4x3mm_P0.65mm, symbol Samacsys_kicad_sym:TPS2113PWR
Connections:
- net F_U5V is gone; now on net VBUS+: C3.2, C6.1, D14.1 (K), F8.1
- net +24V: now also D5.1 (K), Q4.2 (S)
- net F_24V: now also Q4.3 (D)
- net GND: now also C19.1, C20.1, C30.1, C31.1, C39.1, C4.1, C40.1, C42.1, C5.1, D20.2 (A), IC4.2 (GND), R10.2, R16.2, R32.1, R40.1, R62.1, U4.2 (~{EN}), U4.5 (GND)
- net VBUS+: now also R35.1
- net +3.3V renamed +3.3VIO
- net +3.3VIO: now also C19.2, FB2.1
- net +5V renamed +5VIO
- net +5VIO: now also C30.2, C4.2, C42.2, FB1.1, IC4.4 (EN), IC4.6 (VIN), L1.1, U4.7 (OUT); no longer F4.2, F8.2
- new net: D5.2 (A), Q4.1 (G), R10.1
- new net: IC4.3 (FB), R55.2, R62.2
- new net: IC4.1 (SW), L1.2
- new net +3.3VA: C20.2, FB2.2
- new net +5VA: C5.2, FB1.2
- new net +8V: C31.2, D20.1 (K), IC4.5 (VOUT), R55.1
- new net 5VPWR: C39.2, F4.2, R39.1, U4.8 (IN1)
- new net 5VUSB: C40.2, F8.2, U4.6 (IN2)
- new net ILIM: R40.2, U4.4 (ILIM)
- new net VBUS_SENSE: R32.2, R35.2
- new net VSNS: R16.1, R39.2, U4.3 (VSNS)
- no-connect marks 0 -> 1
Other:
- note added: "5V PWR MUX"
- note added: "8V"
- note added: "ANALOG PWR"
- note added: "TVS, RRP AND DECOUPLING"
- note removed: "PROTECTION AND DECOUPLING"
- moved on the sheet: C11, C12, C13, C14, C17, C21, C22, C26, C27, C3, C56, C57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

Commit message: v3.3
Changed lines of the file:
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@@
 	(wire
 		(pts
-			(xy 140.97 138.43) (xy 140.97 140.97)
-		)
-		(stroke
-			(width 0)
-			(type default)
-		)
-	)
-	(wire
-		(pts
 			(xy 110.49 46.99) (xy 110.49 44.45)
 		)
@@
 	(wire
 		(pts
+			(xy 140.97 138.43) (xy 140.97 143.51)
+		)
+		(stroke
+			(width 0)
+			(type default)
+		)
+	)
+	(wire
+		(pts
 			(xy 160.02 138.43) (xy 160.02 140.97)
 		)
@@
 		(lib_name "GND_2")
 		(lib_id "power:GND")
-		(at 140.97 140.97 0)
+		(at 140.97 143.51 0)
 		(unit 1)
 		(exclude_from_sim no)
@@
 		(dnp no)
 		(property "Reference" "#PWR07"
-			(at 140.97 147.32 0)
+			(at 140.97 149.86 0)
 			(effects
 				(font
@@
 		)
 		(property "Value" "GND"
-			(at 141.097 145.3642 0)
+			(at 141.097 147.9042 0)
 			(effects
 				(font
@@
 		)
 		(property "Footprint" ""
-			(at 140.97 140.97 0)
+			(at 140.97 143.51 0)
 			(effects
 				(font
@@
 		)
 		(property "Datasheet" ""
-			(at 140.97 140.97 0)
+			(at 140.97 143.51 0)
 			(effects
 				(font
@@
 		)
 		(property "Description" ""
-			(at 140.97 140.97 0)
+			(at 140.97 143.51 0)
 			(effects
 				(font

Commit message: isolation with every thing
Parts:
- removed C30, C31: 22uF, Capacitor_SMD:C_0805_2012Metric, symbol Device:C_Small
- removed D20: 8V, Diode_SMD:D_SOD-123, symbol Device:D_Zener_Small
- removed IC4: TLV61046ADBVT, Package_TO_SOT_SMD:SOT-23-6, symbol Samacsys_kicad_sym:TLV61046ADBVT
- removed L1: 10uH, Inductor_SMD:L_1008_2520Metric, symbol Device:L
- removed R55: 649k, Resistor_SMD:R_0603_1608Metric, symbol Device:R_Small
- removed R62: 71.5k, Resistor_SMD:R_0603_1608Metric, symbol Device:R_Small
Other:
- note removed: "8V"

Commit message: isolated side, choose most components, some master changes tbc
Changed lines of the file:
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@@
+	)
+	(rectangle
+		(start 194.31 109.22)
+		(end 280.67 119.38)
+		(stroke
+			(width 0)
+			(type dash)
+			(color 132 132 132 1)
+		)
+		(fill
+			(type none)
+		)
 	)
 	(rectangle
@@
 	)
 	(rectangle
-		(start 107.95 176.53)
-		(end 175.26 184.15)
-		(stroke
-			(width 0)
-			(type dash)
-			(color 132 132 132 1)
-		)
-		(fill
-			(type none)
-		)
-	)
-	(rectangle
 		(start 107.95 60.96)
 		(end 172.72 106.68)
@@
 		)
 	)
-	(text_box "WebenchSchematic8V.svg"
-		(exclude_from_sim yes)
-		(at 127 179.07 0)
-		(size 34.29 3.81)
+	(text_box "2*"
+		(exclude_from_sim no)
+		(at 227.33 49.53 0)
+		(size 3.81 3.81)
 		(margins 0.9525 0.9525 0.9525 0.9525)
 		(stroke
@@
 			(font
 				(size 1.27 1.27)
-				(color 0 0 194 1)
+				(color 132 0 132 1)
 			)
 			(justify left top)
-			(href "file://${KIPRJMOD}/images/WebenchSchematic8V.svg")
-		)
-	)
-	(text_box "8V:"
-		(exclude_from_sim no)
-		(at 110.49 179.07 0)
+		)
+	)
+	(text_box "Analog power:"
+		(exclude_from_sim no)
+		(at 110.49 167.64 0)
 		(size 16.51 3.81)
 		(margins 0.9525 0.9525 0.9525 0.9525)
@@
 		)
 	)
-	(text_box "Analog power:"
-		(exclude_from_sim no)
-		(at 110.49 167.64 0)
-		(size 16.51 3.81)
-		(margins 0.9525 0.9525 0.9525 0.9525)
-		(stroke
+	(text_box "1*"
+		(exclude_from_sim no)
+		(at 255.27 71.12 0)
+		(size 3.81 3.81)
+		(margins 0.9525 0.9525 0.9525 0.9525)
+		(stroke
+			(width -0.0001)
+			(type solid)
+		)
+		(fill
+			(type none)
+		)
+		(effects
+			(font
+				(size 1.27 1.27)
+				(color 132 0 132 1)
+			)
+			(justify left top)
+		)
+	)
+	(text_box "1: ILIM bypass 400 coresponds to 6.25A\n2: TPS2113 prioritises built in 5V, switches to USB when not powered from car"
+		(exclude_from_sim no)
+		(at 196.85 111.76 0)
+		(size 81.28 6.35)
+		(margins 0.9525 0.9525 0.9525 0.9525)
+		(stroke

Commit message: chore: sync
Parts:
- removed TP2: TestPoint_Small, MountingHole:MountingHole_3.2mm_M3_Pad_Via, symbol Connector:TestPoint_Small
- added C1: 22uF, Capacitor_SMD:C_0805_2012Metric, symbol Device:C_Small
Connections:
- net F_5V: now also C1.1
- net GND: now also C1.2
Other:
- moved on the sheet: F4
Changed lines of the file:
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@@
 	)
 	(junction
+		(at 154.94 46.99)
+		(diameter 0)
+		(color 0 0 0 0)
+	)
+	(junction
 		(at 120.65 130.81)
 		(diameter 0)
@@
 	)
 	(junction
+		(at 154.94 34.29)
+		(diameter 0)
+		(color 0 0 0 0)
+	)
+	(junction
 		(at 41.91 73.66)
 		(diameter 0)
@@
 	(wire
 		(pts
+			(xy 154.94 44.45) (xy 154.94 46.99)
+		)
+		(stroke
+			(width 0)
+			(type default)
+		)
+	)
+	(wire
+		(pts
 			(xy 31.75 46.99) (xy 43.18 46.99)
 		)
@@
 	(wire
 		(pts
-			(xy 151.13 34.29) (xy 180.34 34.29)
+			(xy 163.83 34.29) (xy 180.34 34.29)
 		)
 		(stroke
@@
 	(wire
 		(pts
+			(xy 154.94 34.29) (xy 154.94 39.37)
+		)
+		(stroke
+			(width 0)
+			(type default)
+		)
+	)
+	(wire
+		(pts
 			(xy 180.34 128.27) (xy 180.34 130.81)
 		)
@@
 	(wire
 		(pts
-			(xy 146.05 34.29) (xy 143.51 34.29)
+			(xy 158.75 34.29) (xy 154.94 34.29)
 		)
 		(stroke
@@
 	(wire
 		(pts
+			(xy 154.94 34.29) (xy 143.51 34.29)
+		)
+		(stroke
+			(width 0)
+			(type default)
+		)
+	)
+	(wire
+		(pts
 			(xy 128.27 92.71) (xy 138.43 92.71)
 		)
@@
 	(wire
 		(pts
+			(xy 154.94 46.99) (xy 143.51 46.99)
+		)
+		(stroke
+			(width 0)
+			(type default)
+		)
+	)
+	(wire
+		(pts
 			(xy 92.71 71.12) (xy 92.71 73.66)
 		)
@@
 	(wire
 		(pts
-			(xy 143.51 46.99) (xy 143.51 49.53)
+			(xy 154.94 46.99) (xy 154.94 49.53)
 		)
 		(stroke
@@
 	)
 	(label "5VPWR"
-		(at 152.4 34.29 0)
+		(at 163.83 34.29 0)
 		(effects
 			(font
@@
 	)
 	(symbol
+		(lib_id "Device:C_Small")
+		(at 154.94 41.91 0)
+		(unit 1)
+		(exclude_from_sim no)
+		(in_bom yes)
+		(on_board yes)
+		(dnp no)
+		(property "Reference" "C1"
+			(at 157.2768 40.7416 0)
+			(effects
+				(font
+					(size 1.27 1.27)
+				)
+				(justify left)
+			)
+		)
+		(property "Value" "22uF"
+			(at 157.2768 43.053 0)
+			(effects
+				(font
+					(size 1.27 1.27)
+				)
+				(justify left)
+			)
+		)
+		(property "Footprint" "Capacitor_SMD:C_0805_2012Metric"
+			(at 154.94 41.91 0)
+			(effects
+				(font
+					(size 1.27 1.27)
+				)
+				(hide yes)
+			)
+		)
+		(property "Datasheet" "~"
+			(at 154.94 41.91 0)
+			(effects
+				(font
+					(size 1.27 1.27)
+				)
+				(hide yes)
+			)
+		)
+		(property "Description" ""
+			(at 154.94 41.91 0)
+			(effects
+				(font
+					(size 1.27 1.27)
+				)
+				(hide yes)
+			)
+		)
+		(property "Manufacturer_Name" "MCASH21GCC7684MTCA1J"
+			(at 154.94 41.91 0)
+			(effects
+				(font
+					(size 1.27 1.27)
+				)
+				(hide yes)
+			)
+		)
+		(property "Manufacturer_Part_Number" "CL21A107MQYNNWE"
+			(at 154.94 41.91 0)
+			(effects
+				(font
+					(size 1.27 1.27)
+				)
+				(hide yes)
+			)
+		)
+		(property "In Order" ""
+			(at 154.94 41.91 0)
+			(effects
+				(font
+					(size 1.27 1.27)
+				)
+				(hide yes)
+			)
+		)
+		(property "Mouser Part Number" "810-C2012X5R1V226MAC"
+			(at 154.94 41.91 0)
+			(effects
+				(font
+					(size 1.27 1.27)
+				)
+				(hide yes)
+			)
+		)
+		(property "Mouser Price/Stock" ""
+			(at 154.94 41.91 0)
+			(effects
+				(font
+					(size 1.27 1.27)
+				)
+				(hide yes)
+			)
+		)
+		(property "Arrow Part Number" ""
+			(at 154.94 41.91 0)
+			(effects
+				(font
+					(size 1.27 1.27)
+				)
+				(hide yes)
+			)
+		)
+		(property "Arrow Price/Stock" ""
+			(at 154.94 41.91 0)
+			(effects
+				(font
+					(size 1.27 1.27)
+				)
+				(hide yes)
+			)
+		)
+		(property "DigiKey Part Number" ""
+			(at 154.94 41.91 0)
+			(effects
+				(font
+					(size 1.27 1.27)
+				)
+			)
+		)
+		(pin "1"
+		)
+		(pin "2"
+		)
+		(instances
+			(project "PUTM_EV_AMS_MASTER_2025"
+				(path "/b456cffc-d9d7-4c91-91f2-36ec9a65dd1b/fddfd40b-128d-4439-b7b1-2bfdbdc0083e"
+					(reference "C1")
+					(unit 1)
+				)
+			)
+		)
+	)
+	(symbol
 		(lib_id "Device:C_Polarized_Small")
 		(at 92.71 86.36 0)
@@
 	(symbol
 		(lib_id "power:GND")
-		(at 143.51 49.53 0)
+		(at 154.94 49.53 0)
 		(unit 1)
 		(exclude_from_sim no)
@@
 		(dnp no)
 		(property "Reference" "#PWR020"
-			(at 143.51 55.88 0)
+			(at 154.94 55.88 0)
 			(effects
 				(font
@@
 		)
 		(property "Value" "GND"
-			(at 143.637 53.9242 0)
+			(at 155.067 53.9242 0)
 			(effects
 				(font
@@
 		)
 		(property "Footprint" ""
-			(at 143.51 49.53 0)
+			(at 154.94 49.53 0)
 			(effects
 				(font
@@
 		)
 		(property "Datasheet" ""
-			(at 143.51 49.53 0)
+			(at 154.94 49.53 0)
 			(effects
 				(font
@@
 		)
 		(property "Description" ""
-			(at 143.51 49.53 0)
+			(at 154.94 49.53 0)
 			(effects
 				(font
@@
 	(symbol
 		(lib_id "Device:Polyfuse_Small")
-		(at 148.59 34.29 90)
+		(at 161.29 34.29 90)
 		(mirror x)
 		(unit 1)
@@
 		(dnp no)
 		(property "Reference" "F4"
-			(at 149.86 29.21 90)
+			(at 162.56 29.21 90)
 			(effects
 				(font
@@
 		)
 		(property "Value" "5V/0.5A"
-			(at 152.4 31.75 90)
+			(at 165.1 31.75 90)
 			(effects
 				(font
@@
 		)
 		(property "Footprint" "Fuse:Fuse_0805_2012Metric"
-			(at 153.67 35.56 0)
+			(at 166.37 35.56 0)
 			(effects
 				(font
@@
 		)
 		(property "Datasheet" "~"
-			(at 148.59 34.29 0)
+			(at 161.29 34.29 0)
 			(effects
 				(font
@@
 		)
 		(property "Description" "Resettable fuse, polymeric positive temperature coefficient, small symbol"
-			(at 148.59 34.29 0)
+			(at 161.29 34.29 0)
 			(effects
 				(font
@@
 		)
 		(property "Manufacturer_Part_Number" "0ZCH0050FF2G"
-			(at 148.59 34.29 0)
+			(at 161.29 34.29 0)
 			(effects
 				(font
@@
 		)
 		(property "Mouser Part Number" "530-0ZCH0050FF2G"
-			(at 148.59 34.29 0)
+			(at 161.29 34.29 0)
 			(effects
 				(font
@@
 		)
 		(property "Mouser Price/Stock" "https://www.mouser.pl/ProductDetail/Bel-Fuse/0ZCH0050FF2G?qs=SRYZG9HaIQ2VrAxOxbTdxQ%3D%3D"
-			(at 148.59 34.29 0)
+			(at 161.29 34.29 0)
 			(effects
 				(font
@@
 		)
 		(property "Arrow Part Number" ""
-			(at 148.59 34.29 0)
+			(at 161.29 34.29 0)
 			(effects
 				(font
@@
 		)
 		(property "Arrow Price/Stock" ""
-			(at 148.59 34.29 0)
+			(at 161.29 34.29 0)
 			(effects
 				(font
@@
 		)
 		(property "DigiKey Part Number" ""
-			(at 148.59 34.29 0)
+			(at 161.29 34.29 0)
 			(effects
 				(font
@@
 					(unit 1)
 				)
-			)
-		)
-	)
-	(symbol
-		(lib_id "Connector:TestPoint_Small")
-		(at 92.71 93.98 180)
-		(unit 1)
-		(exclude_from_sim no)
-		(in_bom yes)
-		(on_board yes)
-		(dnp no)
-		(property "Reference" "TP2"
-			(at 95.25 93.98 0)
-			(effects
-				(font
-					(size 1.27 1.27)
-				)
-				(justify right)
-			)
-		)
-		(property "Value" "TestPoint_Small"
-			(at 91.44 92.7101 0)
-			(effects
-				(font
-					(size 1.27 1.27)
-				)
-				(justify left)
-				(hide yes)
-			)
-		)
-		(property "Footprint" "MountingHole:MountingHole_3.2mm_M3_Pad_Via"
-			(at 87.63 93.98 0)
-			(effects
-				(font
-					(size 1.27 1.27)
-				)
-				(hide yes)
-			)
-		)
-		(property "Datasheet" "~"
-			(at 87.63 93.98 0)
-			(effects
-				(font
-					(size 1.27 1.27)
-				)
-				(hide yes)
-			)
-		)
-		(property "Description" "test point"
-			(at 92.71 93.98 0)
-			(effects
-				(font
-					(size 1.27 1.27)
-				)
-				(hide yes)
-			)
-		)
-		(property "Mouser Part Number" "--"
-			(at 92.71 93.98 0)
-			(effects
-				(font
-					(size 1.27 1.27)
-				)
-				(hide yes)
-			)
-		)
-		(property "DigiKey Part Number" ""
-			(at 92.71 93.98 0)
-			(effects
-				(font
-					(size 1.27 1.27)
-				)
-			)
-		)
-		(pin "1"
-		)
-		(instances
-			(project "PUTM_EV_AMS_MASTER_2025"
-				(path "/b456cffc-d9d7-4c91-91f2-36ec9a65dd1b/fddfd40b-128d-4439-b7b1-2bfdbdc0083e"
-					(reference "TP2")
-					(unit 1)
-				)

Commit message: chore: sync
Parts:
- removed C27, C65: 22uF, Capacitor_SMD:CP_Elec_4x5.8, symbol Device:C_Polarized_Small
- removed D16: 30V, Diode_SMD:D_SOD-123, symbol Device:D_Zener_Small
- removed D5: 10V, Diode_SMD:D_SOD-123, symbol Device:D_Zener_Small
- removed F2: 5A/24V, Fuse:Fuse_2920_7451Metric, symbol Device:Polyfuse_Small
- removed Q4: SI2347DS-T1-GE3, Package_TO_SOT_SMD:SOT-23-3, symbol Transistor_FET:Q_PMOS_GSD
- removed R10: 100k, Resistor_SMD:R_0603_1608Metric_Pad0.98x0.95mm_HandSolder, symbol Device:R_Small
- removed TP3: TestPoint_Small, TestPoint:TestPoint_THTPad_D1.0mm_Drill0.5mm, symbol Connector:TestPoint_Small
Other:
- note removed: "TVS, RRP AND DECOUPLING"
