File: hardware/mainboard/Mcu.kicad_sch (KiCad schematic)
At the start: 14 parts, among them U10 STM32H573RITx, Y1 50MHz

Commit message: sync
Connections:
- net CANFD1_RX: now also U10.61 (PB8); no longer U10.59 (PB7)
- net CANFD1_TX: now also U10.59 (PB7); no longer U10.61 (PB8)
- net EN_12V: no longer names the net of U10.34 (PB13)
- net FAN5_CTRL: no longer names the net of U10.37 (PC6)
- net FAN6_CTRL: no longer names the net of U10.38 (PC7)
- net FAN7_CTRL: no longer names the net of U10.39 (PC8)
- net PG_12V: no longer names the net of U10.33 (PB12)
- no-connect marks 6 -> 8
Other:
- note removed: "TIM3_CH1"
- note removed: "TIM3_CH2"
- note removed: "TIM3_CH3"
Changed lines of the file:
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@@
 (kicad_sch
-	(version 20231120)
+	(version 20250114)
 	(generator "eeschema")
-	(generator_version "8.0")
+	(generator_version "9.0")
 	(paper "A4")

Commit message: schematic?
Parts:
- removed C1, C2: 8pF/.1pF, Capacitor_SMD:C_0603_1608Metric, symbol Device:C_Small
- removed Y1: 50MHz, Crystal:Crystal_SMD_3225-4Pin_3.2x2.5mm, symbol Device:Crystal_GND24_Small
- added R9: 0, Resistor_SMD:R_0603_1608Metric, symbol Device:R_Small
Connections:
- net +3.3V is gone; now on net +3.3VIO: R3.1
- net +3.3VIO: no longer C23.1, C24.1, C25.1, C28.1, C29.1, C36.1, C70.1, R3.2, U10.13 (VDDA), U10.19 (VDD), U10.32 (VDD), U10.48 (VDD), U10.64 (VDD)
- net DETECT_AIR_M: now also U10.38 (PC7); no longer U10.35 (PB14)
- net DETECT_AIR_P: now also U10.39 (PC8); no longer U10.40 (PC9)
- net DETECT_AIR_PRE: now also U10.37 (PC6); no longer U10.36 (PB15)
- net DETECT_CHARGER: now also U10.40 (PC9); no longer U10.2 (PC13)
- net DETECT_TSMS: now also U10.41 (PA8); no longer U10.3 (PC14)
- net DETECT_WTDG: now also U10.27 (PB1); no longer U10.41 (PA8)
- net GND: now also R9.1
- net SIGNAL_AIR_M: now also U10.33 (PB12); no longer U10.27 (PB1)
- net SIGNAL_AIR_P: now also U10.34 (PB13); no longer U10.26 (PB0)
- net SIGNAL_AIR_PRE: now also U10.35 (PB14); no longer U10.25 (PC5)
- net SIGNAL_AMS_ERROR: now also U10.28 (PB2); no longer U10.11 (PC3)
- net UART_COM_RX: now reaches U10.24 (PC4)
- net UART_COM_TX: now reaches U10.29 (PB10)
- net at U10.60 (BOOT0): now also R9.2
- net CLK_IN: no longer names the net of U10.5 (PH0)
- net CLK_OUT: no longer names the net of U10.6 (PH1)
- net COM_MISO: no longer names the net of U10.52 (PC11)
- net COM_MOSI: no longer names the net of U10.53 (PC12)
- net COM_SCK: no longer names the net of U10.51 (PC10)
- net D+ renamed UART_DEBUG_TX
- net D- renamed UART_DEBUG_RX
- net SIGNAL_LED_1 renamed SIGNAL_LED_OK
- net SIGNAL_LED_2 renamed SIGNAL_LED_WRN
- net SIGNAL_LED_3 renamed SIGNAL_LED_ERR
- net SPI_RDY: no longer names the net of U10.9 (PC1)
- net UART_RX renamed UART_USB_RX
- net UART_TX renamed UART_USB_TX
- net ~{COM_CS}: no longer names the net of U10.50 (PA15(JTDI))
- new net +3.3VMCU: C23.1, C24.1, C25.1, C28.1, C29.1, C36.1, C70.1, R3.2, U10.13 (VDDA), U10.19 (VDD), U10.32 (VDD), U10.48 (VDD), U10.64 (VDD)
- new net DETECT_USB: U10.26 (PB0)
- no-connect marks 8 -> 14
Other:
- note removed: "CLOCKS"
- note removed: "D+"
- note removed: "D-"
- note removed: "FDCAN1_RX"
- note removed: "FDCAN1_TX"
- note removed: "FDCAN2_RX"
- note removed: "FDCAN2_TX"
- note removed: "OSC_IN"
- note removed: "OSC_OUT"
- note removed: "SPI1_MOSI"
- note removed: "SPI1_MSIO"
- note removed: "SPI1_NSS"
- note removed: "SPI1_SCK"
- note removed: "SPI2_MOSI"
- note removed: "SPI2_MSIO"
- note removed: "SPI2_NSS"
- note removed: "SPI2_SCK"
- note removed: "SPI3_MOSI"
- note removed: "SPI3_MSIO"
- note removed: "SPI3_NSS"
- note removed: "SPI3_SCK"
- note removed: "SWCLK"
- note removed: "SWDIO"
- note removed: "TIM2_CH1"
- note removed: "TIM2_CH2"
- note removed: "TIM2_CH3"
- note removed: "TIM2_CH4"
- note removed: "USART1_RX"
- note removed: "USART1_TX"

Commit message: hardware routing done, only touch ups will be needed if the board is aproved
Connections:
- net DETECT_AIR_M: now also U10.10 (PC2); no longer U10.38 (PC7)
- net DETECT_AIR_P: now also U10.4 (PC15); no longer U10.39 (PC8)
- net DETECT_AIR_PRE: now also U10.8 (PC0); no longer U10.37 (PC6)
- net DETECT_CHARGER: now also U10.11 (PC3); no longer U10.40 (PC9)
- net DETECT_TSMS: now also U10.9 (PC1); no longer U10.41 (PA8)
- net SIGNAL_AIR_M: now also U10.35 (PB14); no longer U10.33 (PB12)
- net SIGNAL_AIR_PRE: now also U10.33 (PB12); no longer U10.35 (PB14)
- net ~{ADC_DRY}: now also U10.25 (PC5); no longer U10.8 (PC0)
- net ~{FLT}: now also U10.36 (PB15); no longer U10.10 (PC2)
- net DETECT_WTDG: no longer names the net of U10.27 (PB1)
- no-connect marks 14 -> 13

Commit message: isolation with every thing
Connections:
- net ~{FTDI_RST}: now reaches U10.2 (PC13)
- no-connect marks 13 -> 14

Commit message: Layout ver.2
Parts:
- added J2: XIAO ESP32S3 Sense, xiao:XIAO-ESP32-S3-DIP, symbol Connector:Conn_01x04_Socket
- added U1: MAX40200AUK, Package_TO_SOT_SMD:SOT-23-5_HandSoldering, symbol Analog_Switch:MAX40200AUK
Connections:
- net +3.3VMCU: now also U1.1 (VDD), U1.3 (EN)
- net GND: now also J2.13 (GND), U1.2 (GND)
- net LOG_UART_TX: now reaches U10.37 (PC6)
- net LOG_UART_TX: now also J2.8 (RX)
- net LOG_UART_RX: now reaches U10.38 (PC7)
- net LOG_UART_RX: now also J2.7 (TX)
- new net 3.3V_PROT: J2.12 (3V3), U1.5 (OUT)
- no-connect marks 14 -> 21
Other:
- note added: "DATA ACQUIRY"
- note added: "STM UART XIAO UART PC6(TX) ---> RX (RX) PC7(RX) <--- TX (TX)"
- note added: "backcurrent protection"
- note added: "μC"
- moved on the sheet: C23, C24, C25, C28, C29, C36, C70, R3

Commit message: New HV layout and also a lazy prolly bad main layout that i didnt think much about yet tbh
Connections:
- net +3.3VIO: now also U1.1 (VDD), U1.3 (EN)
- net +3.3VMCU: no longer U1.1 (VDD), U1.3 (EN)
Changed lines of the file:
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@@
 (kicad_sch
-	(version 20250114)
+	(version 20260306)
 	(generator "eeschema")
-	(generator_version "9.0")
+	(generator_version "10.0")
 	(paper "A4")
