File: hardware/mainboard/Mcu.kicad_sch (KiCad schematic)
At the start: 15 parts, among them J2 XIAO ESP32S3 Sense, U1 MAX40200AUK, U10 STM32H573RITx

Commit message: done
Parts:
- removed TP3: +3.3VMCU, TestPoint:TestPoint_Pad_D1.0mm, symbol Connector:TestPoint_Small

Commit message: bom update
Parts:
- C23, C24, C25, C28, C29: Mouser Part Number -- -> 81-GCM188R71H104KA7D
- C36, C70: Mouser Part Number 810-C2012X5R1V226MAC -> 81-GRM188R71H224MA4D
- C86, C87: Mouser Part Number 603-CC603KPX7R9BB222 -> 81-GRM188R61H225ME1D
- J2: Mouser Part Number (none) -> --
- R3, R9: Mouser Part Number -- -> ERJ-1GJ0R00C
