File: hardware/mainboard/PUTM_EV_AMS_MASTER.kicad_sch (KiCad schematic)
At the start: 47 parts, among them J1 Conn_02x10_Odd_Even, J10 M300-MV10345M1, J3 Conn_02x04_Odd_Even, J4 FTSH-107-01-L-D-K, J5 M80-51004XX, J7 M300-MV10345M1, J8 M80-51004XX, T1 SM91502ALE

Commit message: master main board changes in progress
Other:
- note added: "zmienić konektor na kątowy"

Commit message: sync
Parts:
- removed ACU_OUT+1: ACU_OUT+, TestPoint:TestPoint_Pad_D1.0mm, symbol Connector:TestPoint_Small
- removed ACU_OUT-1: ACU_OUT-, TestPoint:TestPoint_Pad_D1.0mm, symbol Connector:TestPoint_Small
- removed CAR_OUT+1: CAR_OUT+, TestPoint:TestPoint_Pad_D1.0mm, symbol Connector:TestPoint_Small
- removed CAR_OUT-1: CAR_OUT-, TestPoint:TestPoint_Pad_D1.0mm, symbol Connector:TestPoint_Small
- removed ISO_SPI_OUT+1: ISO_SPI_OUT+, TestPoint:TestPoint_Pad_D1.0mm, symbol Connector:TestPoint_Small
- removed ISO_SPI_OUT-1: ISO_SPI_OUT-, TestPoint:TestPoint_Pad_D1.0mm, symbol Connector:TestPoint_Small
- removed J4: FTSH-107-01-L-D-K, Samacsys:FTSH-107-XX-YYY-D-K, symbol Samacsys_kicad_sym:FTSH-107-01-L-D-K
- removed SWDIO1: SWDIO, TestPoint:TestPoint_Pad_D1.0mm, symbol Connector:TestPoint_Small
- removed TP31: DBG_RX, TestPoint:TestPoint_Pad_D1.0mm, symbol Connector:TestPoint_Small
- removed TP32: DBG_TX, TestPoint:TestPoint_Pad_D1.0mm, symbol Connector:TestPoint_Small
- removed TP33: NRST, TestPoint:TestPoint_Pad_D1.0mm, symbol Connector:TestPoint_Small
- removed TP34: SWCLK, TestPoint:TestPoint_Pad_D1.0mm, symbol Connector:TestPoint_Small
- removed TP43: SPI_TX, TestPoint:TestPoint_Pad_D1.0mm, symbol Connector:TestPoint_Small
- removed TP44: SPI_RX, TestPoint:TestPoint_Pad_D1.0mm, symbol Connector:TestPoint_Small
- removed TP45: FLT, TestPoint:TestPoint_Pad_D1.0mm, symbol Connector:TestPoint_Small
- removed TP9: AMS_ERROR, symbol Connector:TestPoint_Small
- removed UC_AIR_AUX_M1, UC_AIR_AUX_P1, UC_AIR_AUX_PRE1, UC_CANFD1_RX1, UC_CANFD1_TX1, UC_CANFD1_TX2, UC_CANFD2_RX1, UC_IN1, UC_IN2: TestPoint_Small, TestPoint:TestPoint_Pad_D1.0mm, symbol Connector:TestPoint_Small
- added D30: 3.6V/400W, Package_TO_SOT_SMD:SOT-23-6, symbol Power_Protection:ESDA5V3SC5
- added J6: FTSH10701LDRA, Samacsys:FTSH-107-01-L-D-RA, symbol Connector_Generic:Conn_02x07_Odd_Even
Connections:
- net +3.3VA: now also D30.1 (A), D30.3 (A)
- net +3.3VIO: now also D30.4 (A), D30.6 (A); no longer D27.1 (K)
- net +3.3VMCU: now also D22.6 (A), J6.3 (Pin_3); no longer D22.4 (A)
- net +5VA: now also D27.2 (K)
- net +5VIO: now also D27.1 (K); no longer D27.2 (K)
- net AIR_P-: now also D24.6 (A); no longer D28.3 (A)
- net AIR_PRE-: now also D24.4 (A); no longer D28.1 (A)
- net FAN1-: now also D24.3 (A); no longer D24.6 (A)
- net FAN2-: now also D24.1 (A); no longer D24.4 (A)
- net FAN3-: now also D28.3 (A); no longer D24.3 (A)
- net FAN4-: now also D28.1 (A); no longer D24.1 (A)
- net GND: now also D30.2 (K), D30.5 (NC), J6.11 (Pin_11), J6.5 (Pin_5), J6.7 (Pin_7)
- net NRST: now also D21.1 (A), J6.12 (Pin_12); no longer D21.4 (A)
- net SWCLK: now also D22.3 (A), J6.6 (Pin_6); no longer D22.1 (A)
- net SWDIO: now also D22.1 (A), J6.4 (Pin_4); no longer D22.6 (A)
- net UART_DBG_RX: now also D21.4 (A), J6.13 (Pin_13); no longer D21.1 (A)
- net UART_DBG_TX: now also D21.3 (A), J6.14 (Pin_14); no longer D21.6 (A)
- no-connect marks 11 -> 9
Other:
- note added: "OTHER IO"
- note removed: "AIR & FAN"
- note removed: "zmienić konektor na kątowy"
- moved on the sheet: D21, D27
