File: hardware/mainboard/PUTM_EV_AMS_MASTER.kicad_sch (KiCad schematic)
At the start: 24 parts, among them J1 Conn_02x10_Odd_Even, J10 M300-MV10345M1, J3 Conn_02x04_Odd_Even, J5 M80-51004XX, J6 FTSH10701LDRA, J7 M300-MV10345M1, J8 M80-51004XX, T1 SM91502ALE

Commit message: done
Connections:
- net +3.3VMCU is gone; now on net NRST: D22.6 (A), J6.3 (Pin_3)
- net +3.3VA: now also D30.4 (A); no longer D30.1 (A)
- net +3.3VIO: now also D21.6 (A), D30.1 (A), J6.12 (Pin_12); no longer D30.4 (A)
- net AIR_M_DETECTION: no longer J1.10 (Pin_10)
- net AIR_PRE_DETECTION: no longer J1.8 (Pin_8)
- net AIR_P_DETECTION: no longer J1.12 (Pin_12)
- net GND: now also J6.10 (Pin_10), J6.4 (Pin_4), J6.8 (Pin_8), J8.3 (Pin_3); no longer J6.11 (Pin_11), J6.5 (Pin_5), J6.7 (Pin_7)
- net NRST: no longer D21.1 (A), J6.12 (Pin_12)
- net SWCLK: now also D21.3 (A), J6.9 (Pin_9); no longer D22.3 (A), J6.6 (Pin_6)
- net SWDIO: now also D21.1 (A), J6.11 (Pin_11); no longer D22.1 (A), J6.4 (Pin_4)
- net UART_DBG_RX: now also D22.3 (A), J6.2 (Pin_2); no longer D21.4 (A), J6.13 (Pin_13)
- net UART_DBG_TX: now also D22.1 (A), J6.1 (Pin_1); no longer D21.3 (A), J6.14 (Pin_14)
- net DETVUSB renamed DET_USB
- no-connect marks 9 -> 11
Other:
- sheet Connectivity ports: added EX_USB_DET, USB_DET; removed none

Commit message: bom update
Parts:
- C81: Mouser Part Number -- -> 81-GCM1885C1H101JA6D
- J1: Mouser Part Number (none) -> 200-MTMM11002GD120
- J3: Mouser Part Number (none) -> 200-MTMM10402SD120
- R27, R31, R34, R36: Mouser Part Number -- -> 667-ERJ-1GNF1001C
Changed lines of the file:
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@@
 			)
 		)
-		(property "Mouser Part Number" "--"
+		(property "Mouser Part Number" "667-ERJ-1GNF1001C"
 			(at 269.24 38.1 0)
 			(hide yes)
@@
 			)
 		)
-		(property "Mouser Part Number" "--"
+		(property "Mouser Part Number" "667-ERJ-1GNF1001C"
 			(at 269.24 30.48 0)
 			(hide yes)
@@
 			)
 		)
+		(property "Mouser Part Number" "200-MTMM10402SD120"
+			(at 121.92 199.39 90)
+			(hide yes)
+			(show_name no)
+			(do_not_autoplace no)
+			(effects
+				(font
+					(size 1.27 1.27)
+				)
+			)
+		)
 		(pin "3"
 		)
@@
 			)
 		)
-		(property "Mouser Part Number" "--"
+		(property "Mouser Part Number" "81-GCM1885C1H101JA6D"
 			(at 106.68 158.75 0)
 			(hide yes)
@@
 			)
 		)
+		(property "Mouser Part Number" "200-MTMM11002GD120 "
+			(at 337.82 190.5 0)
+			(hide yes)
+			(show_name no)
+			(do_not_autoplace no)
+			(effects
+				(font
+					(size 1.27 1.27)
+				)
+			)
+		)
 		(pin "18"
 		)
@@
 			)
 		)
-		(property "Mouser Part Number" "--"
+		(property "Mouser Part Number" "667-ERJ-1GNF1001C"
 			(at 269.24 45.72 0)
 			(hide yes)
@@
 			)
 		)
-		(property "Mouser Part Number" "--"
+		(property "Mouser Part Number" "667-ERJ-1GNF1001C"
 			(at 269.24 53.34 0)
 			(hide yes)
