File: hardware/mainboard/IsolationBarrier.kicad_sch (KiCad schematic)
At the start: 24 parts, among them IC6 AMC3330DWER, IC7 AMC3330DWER

Commit message: layout
Parts:
- removed C96, C97: 1n, Capacitor_SMD:C_0603_1608Metric, symbol Device:C_Small
Other:
- moved on the sheet: C16, C18

Commit message: hardware routing done, only touch ups will be needed if the board is aproved
Connections:
- net +5VISO renamed +5VIO
Changed lines of the file:
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@@
-	)
-	(symbol
-		(lib_name "+3.3V_11")
-		(lib_id "power:+3.3V")
-		(at 171.45 110.49 0)
-		(mirror y)
-		(unit 1)
-		(exclude_from_sim no)
-		(in_bom yes)
-		(on_board yes)
-		(dnp no)
-		(property "Reference" "#PWR035"
-			(at 171.45 114.3 0)
-			(effects
-				(font
-					(size 1.27 1.27)
-				)
-				(hide yes)
-			)
-		)
-		(property "Value" "+5VISO"
-			(at 171.45 106.68 0)
-			(effects
-				(font
-					(size 1.27 1.27)
-				)
-			)
-		)
-		(property "Footprint" ""
-			(at 171.45 110.49 0)
-			(effects
-				(font
-					(size 1.27 1.27)
-				)
-				(hide yes)
-			)
-		)
-		(property "Datasheet" ""
-			(at 171.45 110.49 0)
-			(effects
-				(font
-					(size 1.27 1.27)
-				)
-				(hide yes)
-			)
-		)
-		(property "Description" ""
-			(at 171.45 110.49 0)
-			(effects
-				(font
-					(size 1.27 1.27)
-				)
-				(hide yes)
-			)
-		)
-		(pin "1"
-		)
-		(instances
-			(project "PUTM_EV_AMS_MASTER_2025"
-				(path "/b456cffc-d9d7-4c91-91f2-36ec9a65dd1b/966640b3-7a11-41e5-818e-eba0d3c90b57"
-					(reference "#PWR035")
-					(unit 1)
-				)
-			)
-		)
 	)
 	(symbol
@@
 			)
 		)
-		(property "Value" "+5VISO"
+		(property "Value" "+5VIO"
 			(at 171.45 19.05 0)
 			(effects
@@
 					(unit 1)
 				)
+			)
+		)
+	)
+	(symbol
+		(lib_name "+3.3V_11")
+		(lib_id "power:+3.3V")
+		(at 171.45 110.49 0)
+		(mirror y)
+		(unit 1)
+		(exclude_from_sim no)
+		(in_bom yes)
+		(on_board yes)
+		(dnp no)
+		(property "Reference" "#PWR056"
+			(at 171.45 114.3 0)
+			(effects
+				(font
+					(size 1.27 1.27)
+				)
+				(hide yes)
+			)
+		)
+		(property "Value" "+5VIO"
+			(at 171.45 106.68 0)
+			(effects
+				(font
+					(size 1.27 1.27)
+				)
+			)
+		)
+		(property "Footprint" ""
+			(at 171.45 110.49 0)
+			(effects
+				(font
+					(size 1.27 1.27)
+				)
+				(hide yes)
+			)
+		)
+		(property "Datasheet" ""
+			(at 171.45 110.49 0)
+			(effects
+				(font
+					(size 1.27 1.27)
+				)
+				(hide yes)
+			)
+		)
+		(property "Description" ""
+			(at 171.45 110.49 0)
+			(effects
+				(font
+					(size 1.27 1.27)
+				)
+				(hide yes)
+			)
+		)
+		(pin "1"
+		)
+		(instances
+			(project "PUTM_EV_AMS_MASTER_2025"
+				(path "/b456cffc-d9d7-4c91-91f2-36ec9a65dd1b/966640b3-7a11-41e5-818e-eba0d3c90b57"
+					(reference "#PWR056")
+					(unit 1)
+				)

Commit message: v3.3
Parts:
- C91, C92, C93, C94, C95, C98: value 1n -> 1nF
Changed lines of the file:
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@@
 			)
 		)
-		(property "Value" "1n"
+		(property "Value" "1nF"
 			(at 165.1 39.37 0)
 			(effects
@@
 			)
 		)
-		(property "Value" "1n"
+		(property "Value" "1nF"
 			(at 111.76 153.67 0)
 			(effects
@@
 			)
 		)
-		(property "Value" "1n"
+		(property "Value" "1nF"
 			(at 106.68 39.37 0)
 			(effects
@@
 			)
 		)
-		(property "Value" "1n"
+		(property "Value" "1nF"
 			(at 106.68 127 0)
 			(effects
@@
 			)
 		)
-		(property "Value" "1n"
+		(property "Value" "1nF"
 			(at 165.1 127 0)
 			(effects
@@
 			)
 		)
-		(property "Value" "1n"
+		(property "Value" "1nF"
 			(at 111.76 66.04 0)
 			(effects

Commit message: master main board changes in progress
Parts:
- added FB1, FB10, FB2, FB3, FB4, FB5, FB6, FB7, FB8, FB9: 2.7k@100MHz, Inductor_SMD:L_0805_2012Metric, symbol Device:FerriteBead_Small
- added R68, R70: 1M/700V/.1%, Resistor_SMD:R_1206_3216Metric, symbol Device:R_Small
- R65, R67: value 1k/.1% -> 4.02k/.1%; Mouser Part Number 708-RNCF1206BKE100R -> 279-RQ73C2B4K02BTD
Connections:
- net ACU+: now also FB2.2; no longer R64.2, R65.2
- net ACU_IN-: now also R68.1; no longer C16.1, C54.2, C67.2, C91.1, C94.1, IC6.2 (DCDC_HGND), IC6.7 (INN), IC6.8 (HGND), R65.1
- net ACU_OUT+: now also FB7.2; no longer IC6.11 (OUTP)
- net ACU_OUT-: now also FB8.2; no longer IC6.10 (OUTN)
- net CAR+: now also FB5.2; no longer R66.2, R67.2
- net CAR_IN-: now also R70.1; no longer C18.1, C59.2, C77.2, C92.1, C95.1, IC7.2 (DCDC_HGND), IC7.7 (INN), IC7.8 (HGND), R67.1
- net CAR_OUT+: now also FB9.2; no longer IC7.11 (OUTP)
- net CAR_OUT-: now also FB10.2; no longer IC7.10 (OUTN)
- new net: FB10.1, IC7.10 (OUTN)
- new net: C16.1, C54.2, C67.2, C94.1, FB1.2, IC6.2 (DCDC_HGND), IC6.8 (HGND)
- new net: FB1.1, FB3.1, R65.1, R68.2
- new net: FB5.1, R66.2, R67.2
- new net: FB9.1, IC7.11 (OUTP)
- new net: FB2.1, R64.2, R65.2
- new net: FB7.1, IC6.11 (OUTP)
- new net: FB4.1, FB6.1, R67.1, R70.2
- new net: FB8.1, IC6.10 (OUTN)
- new net ACU_GND: C91.1, FB3.2, IC6.7 (INN)
- new net CAR_GND: C18.1, C59.2, C77.2, C92.1, C95.1, FB4.2, FB6.2, IC7.2 (DCDC_HGND), IC7.7 (INN), IC7.8 (HGND)
Other:
- moved on the sheet: R64, R65, R66, R67

Commit message: sync
Parts:
- removed FB10, FB7, FB8, FB9: 2.7k@100MHz, Inductor_SMD:L_0805_2012Metric, symbol Device:FerriteBead_Small
Connections:
- net ACU_OUT+: now also IC6.11 (OUTP)
- net ACU_OUT-: now also IC6.10 (OUTN)
- net CAR_OUT+: now also IC7.11 (OUTP)
- net CAR_OUT-: now also IC7.10 (OUTN)
- net GND: no longer C55.2, C9.1, C93.1, IC6.15 (DCDC_GND)
- new net: C55.2, C9.1, C93.1, IC6.15 (DCDC_GND)

Commit message: sync
Connections:
- net GND: now also C55.2, C9.1, C93.1, IC6.15 (DCDC_GND)
Changed lines of the file:
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@@
 	)
 	(junction
+		(at 162.56 45.72)
+		(diameter 0)
+		(color 0 0 0 0)
+	)
+	(junction
 		(at 120.65 115.57)
 		(diameter 0)
@@
 	(wire
 		(pts
-			(xy 180.34 45.72) (xy 160.02 45.72)
+			(xy 162.56 45.72) (xy 160.02 45.72)
 		)
 		(stroke
@@
 	(wire
 		(pts
-			(xy 180.34 45.72) (xy 180.34 48.26)
+			(xy 162.56 45.72) (xy 162.56 48.26)
 		)
 		(stroke
@@
 	(wire
 		(pts
+			(xy 162.56 43.18) (xy 162.56 45.72)
+		)
+		(stroke
+			(width 0)
+			(type default)
+		)
+	)
+	(wire
+		(pts
 			(xy 76.2 130.81) (xy 87.63 130.81)
 		)
@@
 		(lib_name "GND_7")
 		(lib_id "power:GND")
-		(at 180.34 48.26 0)
+		(at 162.56 48.26 0)
 		(unit 1)
 		(body_style 1)
@@
 		(dnp no)
 		(property "Reference" "#PWR0179"
-			(at 180.34 54.61 0)
+			(at 162.56 54.61 0)
 			(hide yes)
 			(show_name no)
@@
 		)
 		(property "Value" "GND"
-			(at 180.34 52.07 0)
+			(at 162.56 52.07 0)
 			(show_name no)
 			(do_not_autoplace no)
@@
 		)
 		(property "Footprint" ""
-			(at 180.34 48.26 0)
+			(at 162.56 48.26 0)
 			(hide yes)
 			(show_name no)
@@
 		)
 		(property "Datasheet" ""
-			(at 180.34 48.26 0)
+			(at 162.56 48.26 0)
 			(hide yes)
 			(show_name no)
@@
 		)
 		(property "Description" ""
-			(at 180.34 48.26 0)
+			(at 162.56 48.26 0)
 			(hide yes)
 			(show_name no)

Commit message: kek
Parts:
- R65, R67: value 4.02k/.1% -> 2k/.1%
Changed lines of the file:
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@@
 			)
 		)
-		(property "Value" "4.02k/.1%"
+		(property "Value" "2k/.1%"
 			(at 52.07 153.67 0)
 			(show_name no)
@@
 			)
 		)
-		(property "Value" "4.02k/.1%"
+		(property "Value" "2k/.1%"
 			(at 52.07 66.04 0)
 			(show_name no)
