File: hardware/mainboard/IsolationBarrier.kicad_sch (KiCad schematic)
At the start: 30 parts, among them IC6 AMC3330DWER, IC7 AMC3330DWER

Commit message: done
Connections:
- net ACU_GND: now also C16.1, C54.2, C67.2, C94.1, FB1.2, IC6.2 (DCDC_HGND), IC6.8 (HGND); no longer C91.1, FB3.2, IC6.7 (INN)
- net CAR_GND: no longer C92.1, FB6.2, IC7.7 (INN)
- new net ACU-: C91.1, FB3.2, IC6.7 (INN)
- new net CAR-: C92.1, FB6.2, IC7.7 (INN)
Changed lines of the file:
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@@
-	)
-	(junction
-		(at 120.65 153.67)
-		(diameter 0)
-		(color 0 0 0 0)
 	)
 	(junction
@@
 	)
 	(junction
-		(at 120.65 133.35)
-		(diameter 0)
-		(color 0 0 0 0)
-	)
-	(junction
 		(at 120.65 118.11)
 		(diameter 0)
@@
 	(wire
 		(pts
-			(xy 109.22 59.69) (xy 118.11 59.69)
+			(xy 109.22 59.69) (xy 120.65 59.69)
 		)
 		(stroke
@@
 	(wire
 		(pts
-			(xy 118.11 59.69) (xy 118.11 63.5)
+			(xy 120.65 59.69) (xy 120.65 63.5)
 		)
 		(stroke
@@
 	(wire
 		(pts
-			(xy 120.65 133.35) (xy 120.65 153.67)
-		)
-		(stroke
-			(width 0)
-			(type default)
-		)
-	)
-	(wire
-		(pts
 			(xy 123.19 153.67) (xy 120.65 153.67)
 		)
@@
 	(wire
 		(pts
-			(xy 118.11 63.5) (xy 123.19 63.5)
+			(xy 120.65 63.5) (xy 123.19 63.5)
 		)
 		(stroke
@@
 		)
 	)
-	(label "CAR_GND"
+	(label "CAR-"
 		(at 116.84 157.48 180)
 		(effects
@@
 	)
 	(label "ACU_GND"
-		(at 116.84 69.85 180)
+		(at 116.84 43.18 180)
+		(effects
+			(font
+				(size 0.508 0.508)
+			)
+			(justify right bottom)
+		)
+	)
+	(label "CAR_GND"
+		(at 119.38 130.81 180)
 		(effects
 			(font
@@
 		(effects
 			(font
+				(size 0.508 0.508)
+			)
+			(justify right bottom)
+		)
+	)
+	(label "ACU-"
+		(at 116.84 69.85 180)
+		(effects
+			(font

Commit message: bom update
Parts:
- R67: Mouser Part Number 279-RQ73C2B4K02BTD -> 667-ERA-8AEB202V
Changed lines of the file:
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@@
 			)
 		)
-		(property "Mouser Part Number" "279-RQ73C2B4K02BTD"
+		(property "Mouser Part Number" "667-ERA-8AEB202V "
 			(at 50.8 152.4 0)
 			(hide yes)

Commit message: bom update
Parts:
- C54, C55, C59, C67, C77, C99: Mouser Part Number -- -> 81-GCM188R71H104KA7D
- C91, C92, C93, C94, C95, C98: Mouser Part Number -- -> 81-GCD188R71H102MA1D
- R64, R66, R68, R70: Mouser Part Number 754-RGV3216P-1004BT1 -> 667-ERA-8AEB105V
- R65: Mouser Part Number 279-RQ73C2B4K02BTD -> 667-ERA-8ARW202V
- R67: Mouser Part Number 667-ERA-8AEB202V -> 667-ERA-8ARW202V
Changed lines of the file:
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@@
 			)
 		)
-		(property "Mouser Part Number" "--"
+		(property "Mouser Part Number" "81-GCM188R71H104KA7D"
 			(at 120.65 125.73 0)
 			(hide yes)
@@
 			)
 		)
-		(property "Mouser Part Number" "--"
+		(property "Mouser Part Number" "81-GCD188R71H102MA1D"
 			(at 162.56 38.1 0)
 			(hide yes)
@@
 			)
 		)
-		(property "Mouser Part Number" "--"
+		(property "Mouser Part Number" "81-GCD188R71H102MA1D"
 			(at 109.22 152.4 0)
 			(hide yes)
@@
 			)
 		)
-		(property "Mouser Part Number" "754-RGV3216P-1004BT1"
+		(property "Mouser Part Number" "667-ERA-8AEB105V"
 			(at 41.91 147.32 0)
 			(hide yes)
@@
 			)
 		)
-		(property "Mouser Part Number" "--"
+		(property "Mouser Part Number" "81-GCM188R71H104KA7D"
 			(at 180.34 125.73 0)
 			(hide yes)
@@
 			)
 		)
-		(property "Mouser Part Number" "--"
+		(property "Mouser Part Number" "81-GCD188R71H102MA1D"
 			(at 109.22 38.1 0)
 			(hide yes)
@@
 			)
 		)
-		(property "Mouser Part Number" "754-RGV3216P-1004BT1"
+		(property "Mouser Part Number" "667-ERA-8AEB105V"
 			(at 41.91 69.85 0)
 			(hide yes)
@@
 			)
 		)
-		(property "Mouser Part Number" "--"
+		(property "Mouser Part Number" "81-GCM188R71H104KA7D"
 			(at 99.06 38.1 0)
 			(hide yes)
@@
 			)
 		)
-		(property "Mouser Part Number" "--"
+		(property "Mouser Part Number" "81-GCD188R71H102MA1D"
 			(at 109.22 125.73 0)
 			(hide yes)
@@
 			)
 		)
-		(property "Mouser Part Number" "--"
+		(property "Mouser Part Number" "81-GCD188R71H102MA1D"
 			(at 162.56 125.73 0)
 			(hide yes)
@@
 			)
 		)
-		(property "Mouser Part Number" "754-RGV3216P-1004BT1"
+		(property "Mouser Part Number" "667-ERA-8AEB105V"
 			(at 41.91 59.69 0)
 			(hide yes)
@@
 			)
 		)
-		(property "Mouser Part Number" "--"
+		(property "Mouser Part Number" "81-GCM188R71H104KA7D"
 			(at 180.34 38.1 0)
 			(hide yes)
@@
 			)
 		)
-		(property "Mouser Part Number" "754-RGV3216P-1004BT1"
+		(property "Mouser Part Number" "667-ERA-8AEB105V"
 			(at 41.91 157.48 0)
 			(hide yes)
@@
 			)
 		)
-		(property "Mouser Part Number" "667-ERA-8AEB202V "
+		(property "Mouser Part Number" "667-ERA-8ARW202V"
 			(at 50.8 152.4 0)
 			(hide yes)
@@
 			)
 		)
-		(property "Mouser Part Number" "279-RQ73C2B4K02BTD"
+		(property "Mouser Part Number" "667-ERA-8ARW202V"
 			(at 50.8 64.77 0)
 			(hide yes)
@@
 			)
 		)
-		(property "Mouser Part Number" "--"
+		(property "Mouser Part Number" "81-GCM188R71H104KA7D"
 			(at 99.06 125.73 0)
 			(hide yes)
@@
 			)
 		)
-		(property "Mouser Part Number" "--"
+		(property "Mouser Part Number" "81-GCM188R71H104KA7D"
 			(at 120.65 38.1 0)
 			(hide yes)
@@
 			)
 		)
-		(property "Mouser Part Number" "--"
+		(property "Mouser Part Number" "81-GCD188R71H102MA1D"
 			(at 109.22 64.77 0)
 			(hide yes)
