File: hardware/mainboard/ADC.kicad_sch (KiCad schematic)
At the start: 23 parts, among them IC8 ADC 24bit, IC9 LTC1799

Commit message: done
Parts:
- added TP17: GND, TestPoint:TestPoint_Pad_D1.0mm, symbol Connector:TestPoint_Small
Connections:
- net GND: now also TP17.1
Other:
- moved on the sheet: TP16
Changed lines of the file:
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@@
 	)
 	(junction
-		(at 191.77 78.74)
+		(at 228.6 88.9)
 		(diameter 0)
 		(color 0 0 0 0)
 	)
 	(junction
-		(at 223.52 88.9)
+		(at 191.77 78.74)
 		(diameter 0)
 		(color 0 0 0 0)
@@
 	)
 	(junction
+		(at 228.6 93.98)
+		(diameter 0)
+		(color 0 0 0 0)
+	)
+	(junction
 		(at 96.52 105.41)
 		(diameter 0)
@@
 	(wire
 		(pts
+			(xy 228.6 88.9) (xy 231.14 88.9)
+		)
+		(stroke
+			(width 0)
+			(type default)
+		)
+	)
+	(wire
+		(pts
 			(xy 146.05 78.74) (xy 148.59 78.74)
 		)
@@
 	(wire
 		(pts
-			(xy 223.52 86.36) (xy 223.52 88.9)
-		)
-		(stroke
-			(width 0)
-			(type default)
-		)
-	)
-	(wire
-		(pts
 			(xy 196.85 106.68) (xy 194.31 106.68)
 		)
@@
 	(wire
 		(pts
-			(xy 223.52 88.9) (xy 231.14 88.9)
-		)
-		(stroke
-			(width 0)
-			(type default)
-		)
-	)
-	(wire
-		(pts
 			(xy 167.64 116.84) (xy 165.1 116.84)
 		)
@@
 	(wire
 		(pts
-			(xy 179.07 88.9) (xy 223.52 88.9)
+			(xy 179.07 88.9) (xy 228.6 88.9)
 		)
 		(stroke
@@
 	)
 	(symbol
+		(lib_id "Connector:TestPoint_Small")
+		(at 228.6 93.98 90)
+		(unit 1)
+		(body_style 1)
+		(exclude_from_sim no)
+		(in_bom yes)
+		(on_board yes)
+		(in_pos_files yes)
+		(dnp no)
+		(property "Reference" "TP17"
+			(at 224.79 92.71 90)
+			(show_name no)
+			(do_not_autoplace no)
+			(effects
+				(font
+					(size 1.27 1.27)
+				)
+			)
+		)
+		(property "Value" "GND"
+			(at 224.79 95.25 90)
+			(show_name no)
+			(do_not_autoplace no)
+			(effects
+				(font
+					(size 1.27 1.27)
+				)
+			)
+		)
+		(property "Footprint" "TestPoint:TestPoint_Pad_D1.0mm"
+			(at 228.6 88.9 0)
+			(hide yes)
+			(show_name no)
+			(do_not_autoplace no)
+			(effects
+				(font
+					(size 1.27 1.27)
+				)
+			)
+		)
+		(property "Datasheet" ""
+			(at 228.6 88.9 0)
+			(hide yes)
+			(show_name no)
+			(do_not_autoplace no)
+			(effects
+				(font
+					(size 1.27 1.27)
+				)
+			)
+		)
+		(property "Description" "test point"
+			(at 228.6 93.98 0)
+			(hide yes)
+			(show_name no)
+			(do_not_autoplace no)
+			(effects
+				(font
+					(size 1.27 1.27)
+				)
+			)
+		)
+		(property "Author" ""
+			(at 228.6 93.98 90)
+			(hide yes)
+			(show_name no)
+			(do_not_autoplace no)
+			(effects
+				(font
+					(size 1.27 1.27)
+				)
+			)
+		)
+		(property "License" ""
+			(at 228.6 93.98 90)
+			(hide yes)
+			(show_name no)
+			(do_not_autoplace no)
+			(effects
+				(font
+					(size 1.27 1.27)
+				)
+			)
+		)
+		(property "MPN" ""
+			(at 228.6 93.98 90)
+			(hide yes)
+			(show_name no)
+			(do_not_autoplace no)
+			(effects
+				(font
+					(size 1.27 1.27)
+				)
+			)
+		)
+		(property "Manufacturer" ""
+			(at 228.6 93.98 90)
+			(hide yes)
+			(show_name no)
+			(do_not_autoplace no)
+			(effects
+				(font
+					(size 1.27 1.27)
+				)
+			)
+		)
+		(property "Mouser" ""
+			(at 228.6 93.98 90)
+			(hide yes)
+			(show_name no)
+			(do_not_autoplace no)
+			(effects
+				(font
+					(size 1.27 1.27)
+				)
+			)
+		)
+		(property "Sim.Device" ""
+			(at 228.6 93.98 90)
+			(hide yes)
+			(show_name no)
+			(do_not_autoplace no)
+			(effects
+				(font
+					(size 1.27 1.27)
+				)
+			)
+		)
+		(property "Sim.Pins" ""
+			(at 228.6 93.98 90)
+			(hide yes)
+			(show_name no)
+			(do_not_autoplace no)
+			(effects
+				(font
+					(size 1.27 1.27)
+				)
+			)
+		)
+		(property "Sim.Type" ""
+			(at 228.6 93.98 90)
+			(hide yes)
+			(show_name no)
+			(do_not_autoplace no)
+			(effects
+				(font
+					(size 1.27 1.27)
+				)
+			)
+		)
+		(pin "1"
+		)
+		(instances
+			(project "PUTM_EV_AMS_MASTER"
+				(path "/b456cffc-d9d7-4c91-91f2-36ec9a65dd1b/6dd12385-8249-456a-9bdd-ab767e747ed7"
+					(reference "TP17")
+					(unit 1)
+				)
+			)
+		)
+	)
+	(symbol
 		(lib_name "GND_7")
 		(lib_id "power:GND")
@@
 	(symbol
 		(lib_id "Connector:TestPoint_Small")
-		(at 223.52 86.36 90)
+		(at 228.6 88.9 90)
 		(unit 1)
 		(body_style 1)
@@
 		(fields_autoplaced yes)
 		(property "Reference" "TP16"
-			(at 223.52 81.28 90)
+			(at 228.6 83.82 90)
 			(show_name no)
 			(do_not_autoplace no)
@@
 		)
 		(property "Value" "4MHz"
-			(at 223.52 83.82 90)
+			(at 228.6 86.36 90)
 			(show_name no)
 			(do_not_autoplace no)
@@
 		)
 		(property "Footprint" "TestPoint:TestPoint_Pad_D1.0mm"
-			(at 223.52 81.28 0)
+			(at 228.6 83.82 0)
 			(hide yes)
 			(show_name no)
@@
 		)
 		(property "Datasheet" ""
-			(at 223.52 81.28 0)
+			(at 228.6 83.82 0)
 			(hide yes)
 			(show_name no)
@@
 		)
 		(property "Description" "test point"
-			(at 223.52 86.36 0)
+			(at 228.6 88.9 0)
 			(hide yes)
 			(show_name no)
@@
 		)
 		(property "Author" ""
-			(at 223.52 86.36 90)
+			(at 228.6 88.9 90)
 			(hide yes)
 			(show_name no)
@@
 		)
 		(property "License" ""
-			(at 223.52 86.36 90)
+			(at 228.6 88.9 90)
 			(hide yes)
 			(show_name no)
@@
 		)
 		(property "MPN" ""
-			(at 223.52 86.36 90)
+			(at 228.6 88.9 90)
 			(hide yes)
 			(show_name no)
@@
 		)
 		(property "Manufacturer" ""
-			(at 223.52 86.36 90)
+			(at 228.6 88.9 90)
 			(hide yes)
 			(show_name no)
@@
 		)
 		(property "Mouser" ""
-			(at 223.52 86.36 90)
+			(at 228.6 88.9 90)
 			(hide yes)
 			(show_name no)
@@
 		)
 		(property "Sim.Device" ""
-			(at 223.52 86.36 90)
+			(at 228.6 88.9 90)
 			(hide yes)
 			(show_name no)
@@
 		)
 		(property "Sim.Pins" ""
-			(at 223.52 86.36 90)
+			(at 228.6 88.9 90)
 			(hide yes)
 			(show_name no)
@@
 		)
 		(property "Sim.Type" ""
-			(at 223.52 86.36 90)
+			(at 228.6 88.9 90)
 			(hide yes)
 			(show_name no)

Commit message: bom update
Parts:
- C45, C47, C52: Mouser Part Number -- -> 81-GCM188R71H104KA7D
- C46, C89, C90: Mouser Part Number -- -> 81-GCM188L81H103MA3D
- C48: Mouser Part Number 963-H168SC7224KTCA1J -> 81-GRM188R71H224MA4D
- C88, C96: Mouser Part Number -- -> 81-GCD188R71H102MA1D
- R22, R93: Mouser Part Number -- -> 667-ERJ-3EKF1002V
- R24: Mouser Part Number 603-RT0603FRD078K2L -> 71-PNM0603E2502BST5
- R33: Mouser Part Number -- -> 667-ERA-3AEB203V
- R43, R73: Mouser Part Number 708-RNCF1206BKE100R -> 667-ERA-3AEB103V
- R50, R51, R52, R54: Mouser Part Number -- -> 667-ERA-3AEB102V
- TP16, TP17: Mouser Part Number (none) -> --
Changed lines of the file:
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@@
 			)
 		)
-		(property "Mouser Part Number" "--"
+		(property "Mouser Part Number" "81-GCM188L81H103MA3D"
 			(at 96.52 100.33 0)
 			(hide yes)
@@
 			)
 		)
-		(property "Mouser Part Number" "708-RNCF1206BKE100R"
+		(property "Mouser Part Number" "667-ERA-3AEB103V"
 			(at 77.47 44.45 0)
 			(hide yes)
@@
 			)
 		)
-		(property "Mouser Part Number" "--"
+		(property "Mouser Part Number" "667-ERA-3AEB102V"
 			(at 72.39 105.41 0)
 			(hide yes)
@@
 			)
 		)
-		(property "Mouser Part Number" "--"
+		(property "Mouser Part Number" "667-ERA-3AEB102V"
 			(at 72.39 95.25 0)
 			(hide yes)
@@
 			)
 		)
-		(property "Mouser Part Number" "--"
+		(property "Mouser Part Number" "81-GCM188R71H104KA7D"
 			(at 186.69 78.74 0)
 			(hide yes)
@@
 			)
 		)
-		(property "Mouser Part Number" "--"
+		(property "Mouser Part Number" "81-GCD188R71H102MA1D"
 			(at 96.52 72.39 0)
 			(hide yes)
@@
 			)
 		)
-		(property "Mouser Part Number" "--"
+		(property "Mouser Part Number" "81-GCM188L81H103MA3D"
 			(at 96.52 128.27 0)
 			(hide yes)
@@
 			)
 		)
-		(property "Mouser Part Number" "--"
+		(property "Mouser Part Number" "81-GCM188L81H103MA3D"
 			(at 143.51 78.74 0)
 			(hide yes)
@@
 			)
 		)
-		(property "Mouser Part Number" "--"
+		(property "Mouser Part Number" "667-ERJ-3EKF1002V"
 			(at 191.77 106.68 0)
 			(hide yes)
@@
 			)
 		)
+		(property "Mouser Part Number" "--"
+			(at 228.6 93.98 90)
+			(hide yes)
+			(show_name no)
+			(do_not_autoplace no)
+			(effects
+				(font
+					(size 1.27 1.27)
+				)
+			)
+		)
 		(pin "1"
 		)
@@
 			)
 		)
-		(property "Mouser Part Number" "--"
+		(property "Mouser Part Number" "81-GCM188R71H104KA7D"
 			(at 143.51 68.58 0)
 			(hide yes)
@@
 			)
 		)
-		(property "Mouser Part Number" "--"
+		(property "Mouser Part Number" "81-GCM188R71H104KA7D"
 			(at 251.46 83.82 0)
 			(hide yes)
@@
 			)
 		)
-		(property "Mouser Part Number" "603-RT0603FRD078K2L"
+		(property "Mouser Part Number" "71-PNM0603E2502BST5"
 			(at 259.08 91.44 0)
 			(hide yes)
@@
 			)
 		)
-		(property "Mouser Part Number" "--"
+		(property "Mouser Part Number" "667-ERA-3AEB102V"
 			(at 72.39 123.19 0)
 			(hide yes)
@@
 			)
 		)
-		(property "Mouser Part Number" "--"
+		(property "Mouser Part Number" "667-ERA-3AEB102V"
 			(at 72.39 133.35 0)
 			(hide yes)
@@
 			)
 		)
-		(property "Mouser Part Number" "--"
+		(property "Mouser Part Number" "81-GCD188R71H102MA1D"
 			(at 96.52 44.45 0)
 			(hide yes)
@@
 			)
 		)
-		(property "Mouser Part Number" "--"
+		(property "Mouser Part Number" "667-ERJ-3EKF1002V"
 			(at 199.39 45.72 0)
 			(hide yes)
@@
 			)
 		)
-		(property "Mouser Part Number" "708-RNCF1206BKE100R"
+		(property "Mouser Part Number" "667-ERA-3AEB103V"
 			(at 77.47 72.39 0)
 			(hide yes)
@@
 			)
 		)
-		(property "Mouser Part Number" "963-H168SC7224KTCA1J"
+		(property "Mouser Part Number" "81-GRM188R71H224MA4D"
 			(at 186.69 83.82 0)
 			(hide yes)
@@
 			)
 		)
+		(property "Mouser Part Number" "--"
+			(at 228.6 88.9 90)
+			(hide yes)
+			(show_name no)
+			(do_not_autoplace no)
+			(effects
+				(font
+					(size 1.27 1.27)
+				)
+			)
+		)
 		(pin "1"
 		)
@@
 			)
 		)
-		(property "Mouser Part Number" "--"
+		(property "Mouser Part Number" "667-ERA-3AEB203V"
 			(at 72.39 67.31 0)
 			(hide yes)
