File: hardware/mainboard/IsolatedSPI.kicad_sch (KiCad schematic)
At the start: 10 parts, among them IC3 BQ79600PWRQ1

Commit message: bom update
Parts:
- C43: Mouser Part Number 963-H168SC7224KTCA1J -> 81-GRM188R71H224MA4D
- C53, C78: Mouser Part Number -- -> 81-GCM188R71H104KA7D
- C79, C80: Mouser Part Number 581-06035A101K -> 81-GCM1885C1H101JA6D
- R97: Mouser Part Number -- -> 667-ERJ-1GNF1001C
- R99: Mouser Part Number -- -> 667-ERJ-3EKF1003V
Changed lines of the file:
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@@
 			)
 		)
-		(property "Mouser Part Number" "581-06035A101K"
+		(property "Mouser Part Number" "81-GCM1885C1H101JA6D"
 			(at 153.67 102.87 0)
 			(hide yes)
@@
 			)
 		)
-		(property "Mouser Part Number" "--"
+		(property "Mouser Part Number" "667-ERJ-1GNF1001C"
 			(at 146.05 92.71 0)
 			(hide yes)
@@
 			)
 		)
-		(property "Mouser Part Number" "963-H168SC7224KTCA1J"
+		(property "Mouser Part Number" "81-GRM188R71H224MA4D"
 			(at 146.05 74.93 0)
 			(hide yes)
@@
 			)
 		)
-		(property "Mouser Part Number" "--"
+		(property "Mouser Part Number" "667-ERJ-3EKF1003V"
 			(at 179.07 64.77 0)
 			(hide yes)
@@
 			)
 		)
-		(property "Mouser Part Number" "581-06035A101K"
+		(property "Mouser Part Number" "81-GCM1885C1H101JA6D"
 			(at 165.1 102.87 0)
 			(hide yes)
@@
 			)
 		)
-		(property "Mouser Part Number" "--"
+		(property "Mouser Part Number" "81-GCM188R71H104KA7D"
 			(at 107.95 74.93 0)
 			(hide yes)
@@
 			)
 		)
-		(property "Mouser Part Number" "--"
+		(property "Mouser Part Number" "81-GCM188R71H104KA7D"
 			(at 107.95 110.49 0)
 			(hide yes)
