File: hardware/mainboard/Safety.kicad_sch (KiCad schematic)
At the start: 17 parts, among them Q6 2N7002, Q8 2N7002, Q9 2N7002, U3 74AUP1G32

Commit message: done
Parts:
- added TP18: GND, TestPoint:TestPoint_Pad_D1.0mm, symbol Connector:TestPoint_Small
Connections:
- net GND: now also TP18.1
Other:
- moved on the sheet: TP5, TP6, TP7

Commit message: bom update
Parts:
- C7, C8: Mouser Part Number -- -> 81-GCM188R71H104KA7D
- R100: Mouser Part Number -- -> 667-ERJ-3EKF1000V
- R11, R13, R14: Mouser Part Number -- -> 667-ERJ-3EKF1002V
- R12: Mouser Part Number -- -> 667-ERJ-3EKF1004V
- R38: Mouser Part Number -- -> 667-ERJ-1GNF1001C
- TP1, TP18, TP4, TP5, TP6, TP7: Mouser Part Number (none) -> --
Changed lines of the file:
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@@
 			)
 		)
-		(property "Mouser Part Number" "--"
+		(property "Mouser Part Number" "81-GCM188R71H104KA7D"
 			(at 123.19 124.46 0)
 			(hide yes)
@@
 			)
 		)
+		(property "Mouser Part Number" "--"
+			(at 85.09 132.08 0)
+			(hide yes)
+			(show_name no)
+			(do_not_autoplace no)
+			(effects
+				(font
+					(size 1.27 1.27)
+				)
+			)
+		)
 		(pin "1"
 		)
@@
 			)
 		)
-		(property "Mouser Part Number" "--"
+		(property "Mouser Part Number" "667-ERJ-3EKF1002V"
 			(at 50.8 144.78 0)
 			(hide yes)
@@
 			)
 		)
+		(property "Mouser Part Number" "--"
+			(at 105.41 140.97 0)
+			(hide yes)
+			(show_name no)
+			(do_not_autoplace no)
+			(effects
+				(font
+					(size 1.27 1.27)
+				)
+			)
+		)
 		(pin "1"
 		)
@@
 			)
 		)
-		(property "Mouser Part Number" "--"
+		(property "Mouser Part Number" "667-ERJ-3EKF1002V"
 			(at 105.41 146.05 0)
 			(hide yes)
@@
 			)
 		)
+		(property "Mouser Part Number" "--"
+			(at 52.07 68.58 90)
+			(hide yes)
+			(show_name no)
+			(do_not_autoplace no)
+			(effects
+				(font
+					(size 1.27 1.27)
+				)
+			)
+		)
 		(pin "1"
 		)
@@
 			)
 		)
+		(property "Mouser Part Number" "--"
+			(at 105.41 151.13 0)
+			(hide yes)
+			(show_name no)
+			(do_not_autoplace no)
+			(effects
+				(font
+					(size 1.27 1.27)
+				)
+			)
+		)
 		(pin "1"
 		)
@@
 			)
 		)
+		(property "Mouser Part Number" "--"
+			(at 74.93 149.86 90)
+			(hide yes)
+			(show_name no)
+			(do_not_autoplace no)
+			(effects
+				(font
+					(size 1.27 1.27)
+				)
+			)
+		)
 		(pin "1"
 		)
@@
 			)
 		)
+		(property "Mouser Part Number" "--"
+			(at 62.23 83.82 0)
+			(hide yes)
+			(show_name no)
+			(do_not_autoplace no)
+			(effects
+				(font
+					(size 1.27 1.27)
+				)
+			)
+		)
 		(pin "1"
 		)
@@
 			)
 		)
-		(property "Mouser Part Number" "--"
+		(property "Mouser Part Number" "81-GCM188R71H104KA7D"
 			(at 74.93 139.7 0)
 			(hide yes)
@@
 			)
 		)
-		(property "Mouser Part Number" "--"
+		(property "Mouser Part Number" "667-ERJ-3EKF1002V"
 			(at 62.23 68.58 0)
 			(hide yes)
@@
 			)
 		)
-		(property "Mouser Part Number" "--"
+		(property "Mouser Part Number" "667-ERJ-3EKF1004V"
 			(at 74.93 127 0)
 			(hide yes)
@@
 			)
 		)
-		(property "Mouser Part Number" "--"
+		(property "Mouser Part Number" "667-ERJ-1GNF1001C"
 			(at 110.49 140.97 0)
 			(hide yes)
@@
 			)
 		)
-		(property "Mouser Part Number" "--"
+		(property "Mouser Part Number" "667-ERJ-3EKF1000V"
 			(at 43.18 139.7 0)
 			(hide yes)
