File: hardware/InputSeperation.kicad_sch (KiCad schematic)
At the start: 5 parts, among them U9 LM397

Commit message: sync
Parts:
- renumbered C74 to C5, C75 to C50, R82 to R35, R83 to R38, U9 to U2
