File: hardware/isolation/PUTM_AMS_MASTER_ISOLATION_2026.kicad_sch (KiCad schematic)
At the start: 7 parts, among them IC4 TLV61046ADBVT

Commit message: isolated side, choose most components, some master changes tbc
Other:
- note added: "595-ISO6740FDWR"
- note added: "595-ISOUSB111DWXR"
- note added: "595-ISOW1044BDFMR"
- note added: "919-REC5A-0505SW/H2"
- note added: "967-CCG152412D"
- note added: "add filtration"
- note added: "move 5A transisors to the isolated side, fuck it"
- note removed: "https://www.mouser.pl/ProductDetail/Murata-Power-Solutions/MTC2S2412MC-R7?qs=mQP6vorrPAdLKyJ%252BjYwifA%3D%3D"
- note removed: "https://www.ti.com/product/UCC33020-Q1"
Changed lines of the file:
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@@
 	(generator_version "9.0")
 	(paper "A2")
-	(text "https://www.mouser.pl/ProductDetail/Murata-Power-Solutions/MTC2S2412MC-R7?qs=mQP6vorrPAdLKyJ%252BjYwifA%3D%3D"
+	(rectangle
+		(start 370.84 158.75)
+		(end 438.15 167.64)
+		(stroke
+			(width 0)
+			(type dash)
+			(color 132 132 132 1)
+		)
+		(fill
+			(type none)
+		)
+	)
+	(text "595-ISOUSB111DWXR "
 		(exclude_from_sim no)
-		(at 316.23 196.85 0)
+		(at 351.282 202.438 0)
 		(effects
 			(font
@@
 		)
 	)
-	(text "https://www.ti.com/product/UCC33020-Q1"
+	(text "move 5A transisors to the isolated side, fuck it "
 		(exclude_from_sim no)
-		(at 323.85 165.1 0)
+		(at 474.98 141.224 0)
 		(effects
 			(font
@@
 		)
 	)
+	(text "967-CCG152412D"
+		(exclude_from_sim no)
+		(at 325.628 202.438 0)
+		(effects
+			(font
+				(size 1.27 1.27)
+			)
+		)
+	)
+	(text "595-ISOW1044BDFMR "
+		(exclude_from_sim no)
+		(at 351.79 192.532 0)
+		(effects
+			(font
+				(size 1.27 1.27)
+			)
+		)
+	)
+	(text "595-ISO6740FDWR"
+		(exclude_from_sim no)
+		(at 423.164 182.372 0)
+		(effects
+			(font
+				(size 1.27 1.27)
+			)
+		)
+	)
+	(text "919-REC5A-0505SW/H2 "
+		(exclude_from_sim no)
+		(at 326.39 192.786 0)
+		(effects
+			(font
+				(size 1.27 1.27)
+			)
+		)
+	)
+	(text "add filtration"
+		(exclude_from_sim no)
+		(at 425.196 186.944 0)
+		(effects
+			(font
+				(size 1.27 1.27)
+			)
+		)
+	)
+	(text_box "WebenchSchematic8V.svg"
+		(exclude_from_sim yes)
+		(at 389.89 161.29 0)
+		(size 34.29 3.81)
+		(margins 0.9525 0.9525 0.9525 0.9525)
+		(stroke
+			(width -0.0001)
+			(type solid)
+		)
+		(fill
+			(type none)
+		)
+		(effects
+			(font
+				(size 1.27 1.27)
+				(color 0 0 194 1)
+			)
+			(justify left top)
+			(href "file://${KIPRJMOD}/images/WebenchSchematic8V.svg")
+		)
+	)
+	(text_box "8V:"
+		(exclude_from_sim no)
+		(at 373.38 161.29 0)
+		(size 16.51 3.81)
+		(margins 0.9525 0.9525 0.9525 0.9525)
+		(stroke
+			(width -0.0001)
+			(type solid)
+		)
+		(fill
+			(type none)
+		)
+		(effects
+			(font
+				(size 1.27 1.27)
+				(color 132 0 132 1)
+			)
+			(justify left top)
+		)
+	)

Commit message: sync
Other:
- note added: "200-PTF10601LD"
- note added: "200-PTF10801LD"
- note added: "200-PTF12001LD"
- note added: "200-PTT10601SD"
- note added: "200-PTT10801SD"
- note added: "200-PTT12001SD"
Changed lines of the file:
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@@
 	(paper "A2")
 	(rectangle
-		(start 370.84 158.75)
-		(end 438.15 167.64)
+		(start 363.22 147.32)
+		(end 401.32 156.21)
 		(stroke
 			(width 0)
@@
 		(fill
 			(type none)
+		)
+	)
+	(text "200-PTT10801SD"
+		(exclude_from_sim no)
+		(at 414.02 225.806 0)
+		(effects
+			(font
+				(size 1.27 1.27)
+			)
 		)
 	)
@@
 		)
 	)
+	(text "200-PTT10601SD"
+		(exclude_from_sim no)
+		(at 411.988 244.602 0)
+		(effects
+			(font
+				(size 1.27 1.27)
+			)
+		)
+	)
 	(text "967-CCG152412D"
 		(exclude_from_sim no)
 		(at 325.628 202.438 0)
+		(effects
+			(font
+				(size 1.27 1.27)
+			)
+		)
+	)
+	(text "200-PTT12001SD "
+		(exclude_from_sim no)
+		(at 415.544 216.916 0)
+		(effects
+			(font
+				(size 1.27 1.27)
+			)
+		)
+	)
+	(text "200-PTF10801LD"
+		(exclude_from_sim no)
+		(at 413.512 230.378 0)
+		(effects
+			(font
+				(size 1.27 1.27)
+			)
+		)
+	)
+	(text "200-PTF10601LD"
+		(exclude_from_sim no)
+		(at 412.75 249.682 0)
+		(effects
+			(font
+				(size 1.27 1.27)
+			)
+		)
+	)
+	(text "200-PTF12001LD "
+		(exclude_from_sim no)
+		(at 415.544 210.82 0)
 		(effects
 			(font
@@
 	(text_box "WebenchSchematic8V.svg"
 		(exclude_from_sim yes)
-		(at 389.89 161.29 0)
-		(size 34.29 3.81)
+		(at 372.11 149.86 0)
+		(size 26.67 3.81)
 		(margins 0.9525 0.9525 0.9525 0.9525)
 		(stroke
@@
 	(text_box "8V:"
 		(exclude_from_sim no)
-		(at 373.38 161.29 0)
-		(size 16.51 3.81)
+		(at 365.76 149.86 0)
+		(size 5.08 3.81)
 		(margins 0.9525 0.9525 0.9525 0.9525)
 		(stroke

Commit message: chore: sync
Parts:
- added C34, C44: 100nF, Capacitor_SMD:C_0603_1608Metric, symbol Device:C_Small
- added R71: 10k, Resistor_SMD:R_0603_1608Metric, symbol Device:R_Small
- added U2: FT230XS, Package_SO:SSOP-16_3.9x4.9mm_P0.635mm, symbol Interface_USB:FT230XS
Connections:
- net +5VIO: now also C44.1, U2.12 (VCC)
- net GND: now also C34.2, C44.2, U2.13 (GND), U2.5 (GND)
- new net +3.3VFTDI: C34.1, R71.1, U2.10 (3V3OUT), U2.3 (VCCIO)
- new net ~{FTDI_RST}: R71.2, U2.11 (~{RESET})
- no-connect marks 0 -> 6
