File: hardware/isolation/PUTM_AMS_MASTER_ISOLATION.kicad_pcb (KiCad board)
At the start: 2 copper layers, 60 x 100 mm, 20 parts, among them IC4 TLV61046ADBVT, J1 Conn_02x10_Odd_Even, J3 Conn_02x04_Odd_Even, J4 FTSH-107-01-L-D-K, J8 M80-51004XX, U2 FT230XS

Commit message: chore: sync
Parts:
- added C1: C_Polarized_Small, Capacitor_THT:CP_Axial_L18.0mm_D10.0mm_P25.00mm_Horizontal, F.Cu at (193.2, 130.0)
- moved PS1 9.00 mm to (183.2, 115.0)

Commit message: chore:sync
Parts:
- added C2: 4.7uF, Capacitor_SMD:C_1812_4532Metric, F.Cu at (242.6, 102.1)
- added C3: 4.7uF, Capacitor_SMD:C_1812_4532Metric, F.Cu at (242.6, 107.0)
- added FL1: ACM55V-701-2PL-TL00, Samacsys:ACM55V7012PLTL00, F.Cu at (222.5, 131.0)
- added PS2: EC5DAW-24D12N, Samacsys:EC5DAW24D12N, F.Cu at (163.6, 128.1)
- moved PS1 92.2 mm to (273.7, 132.5)

Commit message: chore: sync
Parts:
- removed the H3 at (205.6, 137.7)
- removed PS1: CCG15-24-12D, Samacsys:CCG152403S
- added C10: 4.7uF, Capacitor_SMD:C_1812_4532Metric, B.Cu at (261.5, 108.0)
- added C11: 4.7uF, Capacitor_SMD:C_1812_4532Metric, B.Cu at (172.6, 95.4)
- added C12: 4.7uF, Capacitor_SMD:C_1812_4532Metric, B.Cu at (172.6, 100.3)
- added C13: 4.7uF, Capacitor_SMD:C_1812_4532Metric, B.Cu at (172.6, 105.3)
- added C4: 4.7uF, Capacitor_SMD:C_1812_4532Metric, B.Cu at (198.0, 125.0)
- added C5: 4.7uF, Capacitor_SMD:C_1812_4532Metric, B.Cu at (198.0, 116.0)
- added C6: X1,Y2/1.8nF, Samacsys:CAPC5728X280N, B.Cu at (183.0, 118.5)
- added C7: X1,Y2/1.8nF, Samacsys:CAPC5728X280N, B.Cu at (183.0, 122.5)
- added C8: X1,Y2/1.8nF, Samacsys:CAPC5728X280N, B.Cu at (171.0, 122.5)
- added C9: 4.7uF, Capacitor_SMD:C_1812_4532Metric, B.Cu at (172.6, 85.5)
- added H1: MountingHole_Pad, MountingHole:MountingHole_3.2mm_M3_Pad_Via, F.Cu at (205.6, 137.7)
- added J2: M80-5102042, Samacsys:M80-51020YY, F.Cu at (205.5, 112.0)
- added J4: M80-5100642, Samacsys:M80-51006YY, F.Cu at (153.0, 105.0)
- added J5: M80-5100842, Samacsys:M80-51008YY, F.Cu at (153.0, 124.0)
- C1: value C_Polarized_Small -> X1,Y2/1.8nF; footprint Capacitor_THT:CP_Axial_L18.0mm_D10.0mm_P25.00mm_Horizontal -> Samacsys:CAPC5728X280N; moved to B.Cu
- C2, C3: moved to B.Cu
- FL1: value ACM55V-701-2PL-TL00 -> 701@100MHz
- moved C2 55.1 mm to (192.5, 125.0), turned to 90 degrees
- moved C3 50.9 mm to (192.5, 116.0), turned to -90 degrees
- moved FL1 29.4 mm to (195.0, 120.5), turned to 180 degrees
- moved PS2 25.6 mm to (185.9, 115.4), turned to -90 degrees
- moved C1 25.0 mm to (171.0, 118.5), turned to 180 degrees
- moved J3 15.2 mm to (159.0, 139.5), turned to -90 degrees
- moved J1 10.0 mm to (169.0, 139.5)
Connections:
- C1 pad 1: unconnected-(C1-Pad1) -> Earth
- C1 pad 2: unconnected-(C1-Pad2) -> Net-(PS2--VOUT)
- C2 pad 1: unconnected-(C2-Pad1) -> Net-(PS2-+VIN)
- C2 pad 2: unconnected-(C2-Pad2) -> Net-(PS2--VIN)
- C3 pad 1: unconnected-(C3-Pad1) -> Net-(PS2-+VIN)
- C3 pad 2: unconnected-(C3-Pad2) -> Net-(PS2--VIN)
- FL1 pad 1: unconnected-(FL1-Pad1) -> +24V
- FL1 pad 2: unconnected-(FL1-Pad2) -> GND
- FL1 pad 3: unconnected-(FL1-Pad3) -> Net-(PS2--VIN)
- FL1 pad 4: unconnected-(FL1-Pad4) -> Net-(PS2-+VIN)
- PS2 pad 1: unconnected-(PS2--VIN-Pad1) -> Net-(PS2--VIN)
- PS2 pad 10: unconnected-(PS2--VOUT-Pad10) -> Net-(PS2--VOUT)
- PS2 pad 16: unconnected-(PS2-+VIN-Pad16) -> Net-(PS2-+VIN)
- PS2 pad 8: unconnected-(PS2-COM-Pad8) -> Net-(PS2-COM)
- PS2 pad 9: unconnected-(PS2-+VOUT-Pad9) -> Net-(PS2-+VOUT)

Commit message: chore: sync
Parts:
- removed ?: , 
- added C14: 22uF, Capacitor_SMD:C_0805_2012Metric, F.Cu at (232.8, 105.5)
- added C15: 22uF, Capacitor_SMD:C_0805_2012Metric, F.Cu at (232.8, 108.5)
- added C16: 22uF, Capacitor_SMD:C_0805_2012Metric, F.Cu at (232.8, 111.5)
- added C17: 22uF, Capacitor_SMD:C_0805_2012Metric, F.Cu at (232.8, 114.5)
- added C18: 1uF, Capacitor_SMD:C_0603_1608Metric, F.Cu at (237.1, 105.2)
- added C19: 1uF, Capacitor_SMD:C_0603_1608Metric, F.Cu at (237.1, 107.7)
- added C20: 1uF, Capacitor_SMD:C_0603_1608Metric, F.Cu at (237.1, 110.2)
- added C21: 100nF, Capacitor_SMD:C_0603_1608Metric, F.Cu at (237.1, 112.8)
- added C22: 100nF, Capacitor_SMD:C_0603_1608Metric, F.Cu at (237.1, 115.3)
- added C23: 1uF, Capacitor_SMD:C_0603_1608Metric, F.Cu at (241.1, 105.2)
- added C24: 1uF, Capacitor_SMD:C_0603_1608Metric, F.Cu at (241.1, 107.7)
- added C25: 1uF, Capacitor_SMD:C_0603_1608Metric, F.Cu at (241.1, 110.2)
- added C26: 22uF, Capacitor_SMD:C_0805_2012Metric, F.Cu at (232.8, 117.5)
- added C27: 1uF, Capacitor_SMD:C_0603_1608Metric, F.Cu at (241.1, 112.8)
- added C28: 1uF, Capacitor_SMD:C_0603_1608Metric, F.Cu at (241.1, 115.3)
- added C29: 100n, Capacitor_SMD:C_0603_1608Metric_Pad1.08x0.95mm_HandSolder, F.Cu at (246.2, 83.0)
- added C32: 10n, Capacitor_SMD:C_0603_1608Metric_Pad1.08x0.95mm_HandSolder, F.Cu at (246.2, 85.5)
- added C35: 47u, Capacitor_SMD:C_0603_1608Metric_Pad1.08x0.95mm_HandSolder, F.Cu at (246.2, 90.5)
- added C38: 220n, Capacitor_SMD:C_0603_1608Metric_Pad1.08x0.95mm_HandSolder, F.Cu at (246.2, 98.0)
- added C40: 100n, Capacitor_SMD:C_0603_1608Metric_Pad1.08x0.95mm_HandSolder, F.Cu at (250.5, 85.5)
- added C41: 47u, Capacitor_SMD:C_0603_1608Metric_Pad1.08x0.95mm_HandSolder, F.Cu at (250.5, 88.0)
- added C45: 100n, Capacitor_SMD:C_0603_1608Metric_Pad1.08x0.95mm_HandSolder, F.Cu at (250.5, 95.5)
- added C46: 10n, Capacitor_SMD:C_0603_1608Metric_Pad1.08x0.95mm_HandSolder, F.Cu at (250.5, 98.0)
- added C68: 22uF, Capacitor_SMD:C_0805_2012Metric, F.Cu at (232.8, 120.5)
- added D16: 30V, Diode_SMD:D_SOD-123, F.Cu at (231.4, 89.9)
- added D5: 10V, Diode_SMD:D_SOD-123, F.Cu at (231.4, 86.5)
- added F2: 5A/24V, Fuse:Fuse_2920_7451Metric, F.Cu at (233.6, 81.3)
- added F4: 5V/0.5A, Fuse:Fuse_0805_2012Metric, F.Cu at (242.4, 125.5)
- added FB1: 2K@100MHz, Inductor_SMD:L_0603_1608Metric_Pad1.05x0.95mm_HandSolder, F.Cu at (254.9, 88.0)
- added FB2: 2K@100MHz, Inductor_SMD:L_0603_1608Metric_Pad1.05x0.95mm_HandSolder, F.Cu at (254.9, 90.5)
- added FB5: 2K@100MHz, Inductor_SMD:L_0603_1608Metric_Pad1.05x0.95mm_HandSolder, F.Cu at (254.9, 98.0)
- added FB6: 2K@100MHz, Inductor_SMD:L_0603_1608Metric_Pad1.05x0.95mm_HandSolder, F.Cu at (259.2, 83.0)
- added IC1: ISO7141, Package_SO:SSOP-16_3.9x4.9mm_P0.635mm, F.Cu at (226.6, 107.6)
- added IC2: ISO7141, Package_SO:SSOP-16_3.9x4.9mm_P0.635mm, F.Cu at (226.6, 114.5)
- added IC3: ISO7141, Package_SO:SSOP-16_3.9x4.9mm_P0.635mm, F.Cu at (226.6, 121.4)
- added IC5: ISO7141, Package_SO:SSOP-16_3.9x4.9mm_P0.635mm, F.Cu at (226.6, 128.3)
- added IC6: TPS54202HDDCR, Package_TO_SOT_SMD:SOT-23-6, F.Cu at (237.6, 126.5)
- added K1: IM07DTS, Samacsys:IM23TS, F.Cu at (194.5, 120.5)
- added L4: 68uF/1.4A, Inductor_SMD:L_TDK_VLS6045EX_VLS6045AF, F.Cu at (238.9, 120.3)
- added Q4: SI2347DS-T1-GE3, Package_TO_SOT_SMD:SOT-23-3, F.Cu at (231.0, 93.9)
- added R1: 100K, Resistor_SMD:R_0603_1608Metric_Pad0.98x0.95mm_HandSolder, F.Cu at (259.2, 90.5)
- added R10: 100k, Resistor_SMD:R_0603_1608Metric_Pad0.98x0.95mm_HandSolder, F.Cu at (235.8, 92.8)
- added R23: 510k, Resistor_SMD:R_0603_1608Metric, F.Cu at (245.1, 105.2)
- added R28: 100k, Resistor_SMD:R_0603_1608Metric, F.Cu at (245.1, 107.7)
- added R29: 13.3k, Resistor_SMD:R_0603_1608Metric, F.Cu at (245.1, 110.2)
- added TP3: TestPoint_Small, TestPoint:TestPoint_THTPad_D1.0mm_Drill0.5mm, F.Cu at (230.0, 97.7)
- added U1: ADM3057ExRW, Package_SO:SOIC-20W_7.5x12.8mm_P1.27mm, F.Cu at (179.8, 103.0)
- C11, C9: moved to F.Cu
- moved J5 61.1 mm to (205.8, 93.2), turned to -90 degrees
- moved H1 52.9 mm to (205.8, 79.8)
- moved C9 45.6 mm to (161.3, 129.7), turned to -90 degrees
- moved C11 43.1 mm to (161.0, 137.0), turned to 90 degrees
- moved J3 35.5 mm to (151.8, 104.8), turned to 180 degrees
- moved C13 33.7 mm to (161.0, 137.0), turned to -90 degrees
- moved C12 31.5 mm to (161.2, 129.8), turned to 90 degrees
- moved J1 30.2 mm to (151.8, 114.8), turned to 180 degrees
- moved J4 16.9 mm to (136.6, 93.8)
- moved J4 12.5 mm to (152.8, 92.5)
- moved C1 12.5 mm to (171.0, 131.0)
- moved C3 12.5 mm to (192.5, 128.5)
- moved C4 12.5 mm to (198.0, 137.5)
- moved C5 12.5 mm to (198.0, 128.5)
- moved C6 12.5 mm to (183.0, 131.0)
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Other:
- board size 60 x 100 mm -> 60 x 65 mm

Commit message: chore:sync
Parts:
- removed L4: 68uF/1.4A, Inductor_SMD:L_TDK_VLS6045EX_VLS6045AF
- added L2: 68uF/0.3A, Samacsys:LQH3NPN100MMEL, F.Cu at (237.6, 121.3)
