File: hardware/isolation/PUTM_AMS_MASTER_ISOLATION.kicad_pcb (KiCad board)
At the start: 2 copper layers, 60 x 65 mm, 150 parts, among them IC1 ISO6542DBQR, IC4 LMZM23601V5SILT, IC6 3.3V/0.5A, IC7 3.3V/0.5A, J1 Conn_02x10_Odd_Even, J2 M80-5102042, J3 Conn_02x04_Odd_Even, J4 M80-5100642, K1 IM07DTS, K2 IM07DTS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

Commit message: sync
Parts:
- D11, D13: moved to F.Cu
- moved F2 84.5 mm to (203.8, 128.0)
- moved D1 84.5 mm to (201.5, 132.5), turned to 180 degrees
- moved D5 78.4 mm to (195.0, 127.8), turned to 90 degrees
- moved R10 75.7 mm to (197.2, 128.0), turned to -90 degrees
- moved Q4 73.8 mm to (196.2, 132.0)
- moved D17 62.0 mm to (227.7, 124.0)
- moved C5 40.9 mm to (190.5, 127.0), turned to 180 degrees
- moved C4 32.2 mm to (190.5, 131.0), turned to 180 degrees
- moved FL1 18.8 mm to (196.5, 137.5), turned to -90 degrees
- moved J2 17.0 mm to (205.8, 109.0)
- moved D12 11.6 mm to (318.4, 93.5), turned to -90 degrees
- moved D13 10.6 mm to (316.4, 95.0), turned to 90 degrees
- moved D11 8.23 mm to (303.2, 94.2)
- moved C2 8.00 mm to (190.5, 135.0), turned to 180 degrees
- moved C3 8.00 mm to (190.5, 139.0), turned to 180 degrees
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Routing:
- net Net-(D12-A): track 9.39 -> 0.00 mm
- net Net-(D11-A): track 5.84 -> 0.00 mm
- net /Interface connectors/AIR_M-: track 2.77 -> 0.00 mm
- net /Interface connectors/AIR_M+: track 2.77 -> 0.00 mm
- net /Relay Driver M/EN: track 2.11 -> 0.00 mm
- net +24ISO: track 4.17 -> 2.09 mm
Other:
- copper layers 2 -> 6

Commit message: sync
Parts:
- removed C18, C19: 1uF, Capacitor_SMD:C_0603_1608Metric
- removed C52, C53: 22uF, Capacitor_SMD:C_0805_2012Metric
- added C66: 47uF, Capacitor_SMD:C_0805_2012Metric, F.Cu at (181.4, 94.4)
- added C67: 47uF, Capacitor_SMD:C_0805_2012Metric, F.Cu at (177.0, 94.4)
- added C68: 47uF, Capacitor_SMD:C_0805_2012Metric, F.Cu at (180.9, 80.2)
- added C69: 47uF, Capacitor_SMD:C_0805_2012Metric, F.Cu at (180.9, 77.2)
- added H3: M3, MountingHole:MountingHole_3.2mm_M3, F.Cu at (205.8, 137.8)
- C21, C22, C36, C56: moved to B.Cu
- C40, C51: value 22uF -> 100nF; footprint Capacitor_SMD:C_0805_2012Metric -> Capacitor_SMD:C_0603_1608Metric
- C45, C46, C50, C57, C58, C59, C61, C62, C63, C64: footprint Capacitor_SMD:C_0603_1608Metric_Pad1.08x0.95mm_HandSolder -> Capacitor_SMD:C_0805_2012Metric
- D14, D16, D2, D4: moved to F.Cu
- FB1, FB2, FB3, FB4, FB5, FB6, FB8, FB9: footprint Inductor_SMD:L_0603_1608Metric_Pad1.05x0.95mm_HandSolder -> Inductor_SMD:L_0805_2012Metric
- moved D3 193.2 mm to (159.9, 84.8)
- moved R72 193.0 mm to (159.9, 81.8)
- moved D15 187.2 mm to (159.9, 78.2)
- moved R85 187.1 mm to (159.9, 75.2)
- moved D4 186.7 mm to (161.8, 83.2), turned to -90 degrees
- moved D16 180.6 mm to (161.8, 76.8), turned to -90 degrees
- moved K1 179.1 mm to (168.2, 83.2), turned to 180 degrees
- moved K4 172.8 mm to (168.2, 76.8), turned to 180 degrees
- moved D2 172.5 mm to (166.4, 94.6), turned to 180 degrees
- moved Q8 169.6 mm to (166.8, 97.5), turned to 180 degrees
- moved R73 169.3 mm to (167.2, 100.0), turned to 0 degrees
- moved D14 161.6 mm to (171.2, 94.6), turned to 180 degrees
- moved Q10 159.1 mm to (171.6, 97.5), turned to 180 degrees
- moved R84 158.7 mm to (172.0, 100.0), turned to 0 degrees
- moved R83 158.7 mm to (159.9, 88.2), turned to 90 degrees
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Connections:
- net Net-(C38-Pad1) renamed /FDCAN CAR/GNDCANOUT
- net Net-(C41-Pad1) renamed /FDCAN CHG/GNDCANOUT
- net Net-(U1-RS) renamed /FDCAN CAR/RS
- net Net-(U1-VCC) renamed /FDCAN CAR/VCC
- net Net-(U1-VIO) renamed /FDCAN CAR/VIO
- net Net-(U1-VISOOUT) renamed /FDCAN CAR/VDDCANOUT
- net Net-(U2-VCC) renamed /USB/VCC
- net Net-(U5-RS) renamed /FDCAN CHG/RS
- net Net-(U5-VCC) renamed /FDCAN CHG/VCC
- net Net-(U5-VIO) renamed /FDCAN CHG/VIO
- net Net-(U5-VISOOUT) renamed /FDCAN CHG/VDDCANOUT
- C40 pad 1: GNDISO -> GNDUSB
- C40 pad 2: +5VUSBISO -> +3.3VUSB
- C51 pad 2: +5VUSBISO -> +3.3VISO
- D17 pad 2: Net-(D17-A) -> /Interface connectors/_VDDRLY
- J2 pad 1: /Interface connectors/D- -> /Interface connectors/_VDDRLY
- J2 pad 11: GNDUSB -> GND
- J2 pad 12: +5VUSB -> /Interface connectors/SDC_OUT
- J2 pad 13: /Charger Detect/IN -> GNDUSB
- J2 pad 14: unconnected-(J2-Pad14) -> +5VUSB
- J2 pad 18: /Interface connectors/SDC_OUT -> unconnected-(J2-Pad18)
- J2 pad 2: /Interface connectors/D+ -> /Interface connectors/SDC_IN
- J2 pad 3: /FDCAN CHG/CANH -> /Interface connectors/D-
- J2 pad 4: /FDCAN CHG/CANL -> /Interface connectors/D+
- J2 pad 5: /FDCAN CAR/CANH -> /FDCAN CHG/CANH
- J2 pad 6: /FDCAN CAR/CANL -> /FDCAN CHG/CANL
- J2 pad 7: GND -> /FDCAN CAR/CANH
- J2 pad 8: /Interface connectors/SDC_IN -> /FDCAN CAR/CANL
- J2 pad 9: Net-(D17-A) -> /Charger Detect/IN
- R72 pad 2: +24V -> VDDRLY
- R83 pad 2: +24V -> VDDRLY
- R85 pad 2: +24V -> VDDRLY
Routing:
- net GNDISO: track 0.00 -> 28.3 mm, vias 0 -> 24
- net GNDUSB: track 0.00 -> 12.9 mm, vias 0 -> 7
- net Net-(Q3-D): track 0.00 -> 12.2 mm
- net Net-(D3-A): track 0.00 -> 11.1 mm
- net Net-(D12-A): track 0.00 -> 11.1 mm
- net Net-(U3-+VIN): track 0.00 -> 9.79 mm
- net /USB/RX_LED: track 0.00 -> 9.69 mm, vias 0 -> 2
- net /FDCAN CHG/GNDCAN: track 0.00 -> 9.40 mm, vias 0 -> 4
- net /FDCAN CAR/GNDCAN: track 0.00 -> 9.40 mm, vias 0 -> 4
- net +3.3VUSB: track 0.00 -> 8.76 mm, vias 0 -> 5
- net /Interface connectors/AIR_P+: track 0.00 -> 8.40 mm, vias 0 -> 1
- net /Interface connectors/AIR_M+: track 0.00 -> 8.40 mm, vias 0 -> 1
- net +5VUSB: track 0.00 -> 8.26 mm, vias 0 -> 2
- net Net-(Q3-G): track 0.00 -> 8.17 mm
- net /FDCAN CAR/VDDCAN: track 0.00 -> 7.21 mm, vias 0 -> 2
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Other:
- board size 60 x 65 mm -> 60 x 71 mm
- board text added: "AIR M"
- board text added: "AIR P"
- board text added: "FDCAN CAR"
- board text added: "FDCAN CHARGER"
- board text added: "ISO +24V"
- board text added: "ISO USB"
- board text added: "PRE"
- board text added: "SDC"
- board text added: "T R"

Commit message: pcb finished
Parts:
- removed the H3 at (205.8, 137.8)
- removed TP10, TP11, TP12, TP3, TP9: TestPoint_Small, TestPoint:TestPoint_THTPad_D1.0mm_Drill0.5mm
- added D18: 5.3V/400W, Package_TO_SOT_SMD:SOT-23-3, F.Cu at (197.8, 90.5)
- added D19: 5.3V/400W, Package_TO_SOT_SMD:SOT-23-3, F.Cu at (197.8, 118.5)
- added D20: 5.3V/400W, Package_TO_SOT_SMD:SOT-23-3, F.Cu at (197.8, 105.0)
- added J5: Conn_01x02, Connector_PinHeader_2.00mm:PinHeader_1x02_P2.00mm_Vertical, F.Cu at (196.8, 139.0)
- C29, C32, C38, C41, C54, C55, C60, C65: footprint Capacitor_SMD:C_0603_1608Metric_Pad1.08x0.95mm_HandSolder -> Capacitor_SMD:C_0603_1608Metric
- R1, R10, R11, R2: footprint Resistor_SMD:R_0603_1608Metric_Pad0.98x0.95mm_HandSolder -> Resistor_SMD:R_0603_1608Metric
- moved D6 70.1 mm to (168.5, 107.2), turned to 90 degrees
- moved C48 68.4 mm to (173.0, 101.0), turned to -90 degrees
- moved C43 64.5 mm to (170.0, 101.0), turned to -90 degrees
- moved R11 63.1 mm to (166.0, 112.2), turned to -90 degrees
- moved R39 57.0 mm to (168.5, 101.0), turned to -90 degrees
- moved C49 56.1 mm to (171.5, 101.0), turned to -90 degrees
- moved R82 55.5 mm to (172.0, 112.8)
- moved R40 54.9 mm to (172.0, 111.2), turned to 180 degrees
- moved U4 54.8 mm to (172.0, 106.5), turned to 90 degrees
- moved R16 53.4 mm to (168.5, 104.0), turned to -90 degrees
- moved IC4 51.5 mm to (168.5, 117.5), turned to 90 degrees
- moved C37 47.2 mm to (168.5, 114.2)
- moved C33 46.9 mm to (168.5, 112.2)
- moved C15 46.7 mm to (172.0, 122.5), turned to 180 degrees
- moved C30 45.9 mm to (168.5, 120.8)
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Connections:
- net /Charger Detect/OUTISO renamed /CHARGER_DETECTION
- net /FDCAN CAR/CANH renamed /FDCAN2+
- net /FDCAN CAR/CANL renamed /FDCAN2-
- net /FDCAN CHG/CANH renamed /FDCAN1+
- net /FDCAN CHG/CANL renamed /FDCAN1-
- net /Stack Connectors/TSMS_DETECTION renamed /TSMS_DETECTION
- C14 pad 2: /Power/F_+3.3V -> /Power/F_+3.3VIO
- C17 pad 2: /Power/F_+3.3V -> /Power/F_+3.3VA
- C51 pad 2: +3.3VISO -> +3.3VIOISO
- D1 pad 1: GND -> /Power/F_24V
- D1 pad 2: /Power/F_24V -> GND
- D11 pad 1: +24ISO -> +24VISO
- D14 pad 1: +24ISO -> +24VISO
- D2 pad 1: +24ISO -> +24VISO
- D7 pad 1: +24ISO -> +24VISO
- F5 pad 1: /Power/F_+3.3V -> /Power/F_+3.3VIO
- F6 pad 1: /Power/F_+3.3V -> /Power/F_+3.3VA
- IC1 pad 1: +3.3VISO -> +3.3VIOISO
- IC1 pad 12: /Stack Connectors/UART_TX -> /USB/_TXD
- IC1 pad 5: /USB/_TXD -> /Stack Connectors/UART_TX
- IC6 pad 5: /Power/F_+3.3V -> /Power/F_+3.3VIO
- IC7 pad 5: /Power/F_+3.3V -> /Power/F_+3.3VA
- J1 pad 14: +3.3VIO -> +3.3VIOISO
- J1 pad 15: +5VA -> +5VAISO
- J1 pad 16: +5VIO -> +5VIOISO
- J1 pad 19: +3.3VA -> +3.3VAISO
- J1 pad 2: GND -> GNDISO
- J1 pad 20: GND -> GNDISO
- J2 pad 11: GND -> /CHARGER
- J2 pad 3: /Interface connectors/D- -> /Interface connectors/D+
- J2 pad 4: /Interface connectors/D+ -> /Interface connectors/D-
- J2 pad 9: /Charger Detect/IN -> unconnected-(J2-Pad9)
- J3 pad 8: GND -> GNDISO
- K1 pad 1: +24ISO -> +24VISO
- K2 pad 1: +24ISO -> +24VISO
- K3 pad 1: +24ISO -> +24VISO
- K4 pad 1: +24ISO -> +24VISO
- R88 pad 1: /Charger Detect/IN -> /CHARGER
Routing:
- net +24VISO: track 0.00 -> 149.2 mm, vias 0 -> 7
- net GNDISO: track 28.3 -> 135.5 mm, vias 24 -> 107
- net /CHARGER: track 0.00 -> 103.6 mm, vias 0 -> 1
- net /SDC Driver/RELAY-: track 0.00 -> 93.3 mm
- net +3.3VIOISO: track 3.79 -> 91.8 mm, vias 0 -> 9
- net +5VIOISO: track 3.79 -> 81.8 mm, vias 0 -> 6
- net VDDRLY: track 2.43 -> 72.1 mm, vias 3 -> 5
- net /Stack Connectors/UART_RST: track 0.93 -> 55.3 mm
- net /Stack Connectors/UART_RX: track 0.92 -> 55.0 mm
- net /Stack Connectors/UART_TX: track 1.17 -> 51.4 mm
- net /Stack Connectors/USB_DETECTION: track 1.18 -> 50.0 mm
- net /FDCAN CHG/RXD: track 0.00 -> 47.9 mm, vias 0 -> 1
- net /FDCAN CHG/TXD: track 0.00 -> 45.0 mm, vias 0 -> 1
- net /Interface connectors/_VDDRLY: track 0.00 -> 39.7 mm
- net /FDCAN CAR/RXD: track 0.00 -> 35.2 mm, vias 0 -> 1
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- added copper zone on F.Cu, net +24V
- added copper zone on In3.Cu, net +24V
- added copper zone on B.Cu, net +24VISO
- added copper zone on F.Cu, net +24VISO
- added copper zone on B.Cu, net /FDCAN CAR/GNDCAN
- added copper zone on In1.Cu, net /FDCAN CAR/GNDCAN
- added copper zone on In4.Cu, net /FDCAN CAR/GNDCAN
- added copper zone on In2.Cu, net /FDCAN CAR/VDDCAN
- added copper zone on B.Cu, net /FDCAN CHG/GNDCAN
- added copper zone on In1.Cu, net /FDCAN CHG/GNDCAN
- added copper zone on In4.Cu, net /FDCAN CHG/GNDCAN
- added copper zone on In2.Cu, net /FDCAN CHG/VDDCAN
- added copper zone on F.Cu, net /Power/F_24V
- added copper zone on In2.Cu, net /Power/F_24V
- added copper zone on B.Cu, net /Power/PS_+24V
- added copper zone on F.Cu, net /Power/PS_+24V
- added copper zone on B.Cu, net /Power/PS_GND
- added copper zone on F.Cu, net /Power/PS_GND
- added copper zone on B.Cu, net Earth
- added copper zone on F.Cu, net GND
- added copper zone on In1.Cu, net GND
- added copper zone on B.Cu, net GNDISO
- added copper zone on F.Cu, net GNDISO
- added copper zone on In1.Cu, net GNDISO
- added copper zone on In4.Cu, net GNDISO
- added copper zone on B.Cu, net GNDUSB
- added copper zone on In1.Cu, net GNDUSB
- added copper zone on In4.Cu, net GNDUSB
- added copper zone on In2.Cu, net Net-(PS2-COM)
- added copper zone on F.Cu, net VDD
Other:
- board text added: "DIOD TM"
- board text added: "ISO FDCAN CAR"
- board text added: "ISO FDCAN CHG"
- board text added: "OK"
- board text added: "POWER MANAGEMENT & INPUTS"
- board text removed: "FDCAN CAR"
- board text removed: "FDCAN CHARGER"
