File: hardware/isolation/PUTM_AMS_MASTER_ISOLATION.kicad_pcb (KiCad board)
At the start: 6 copper layers, 60 x 71 mm, 149 parts, among them IC1 ISO6542DBQR, IC4 LMZM23601V5SILT, IC6 3.3V/0.5A, IC7 3.3V/0.5A, J1 Conn_02x10_Odd_Even, J2 M80-5102042, J3 Conn_02x04_Odd_Even, J4 M80-5100642, J5 Conn_01x02, K1 IM07DTS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

Commit message: sync
Parts:
- removed C35: 100nF, Capacitor_SMD:C_0603_1608Metric
- removed Q3: Si2365EDS, Package_TO_SOT_SMD:SOT-23-3
- removed R80: 1k, Resistor_SMD:R_0603_1608Metric
- removed R81: 100k, Resistor_SMD:R_0603_1608Metric
- added R76: 0, Resistor_SMD:R_0603_1608Metric, F.Cu at (189.2, 82.0)
- added R89: 120, Resistor_SMD:R_0603_1608Metric, F.Cu at (198.0, 122.2)
- added R90: 120, Resistor_SMD:R_0603_1608Metric, F.Cu at (198.0, 108.8)
- IC1: value ISO6542DBQR -> ISO6542FDBQR
- R72, R75, R83, R85, R86, R88: value 1k -> 10k
Connections:
- C69 pad 1: Net-(Q3-D) -> +5VUSB
- IC1 pad 14: /USB/_~{RST} -> Net-(IC1-OUTA)
- L2 pad 2: Net-(Q3-D) -> +5VUSB
Routing:
- net +5VUSB: track 35.5 -> 48.6 mm
- net Net-(Q3-D): track 12.0 -> 0.00 mm
- net Net-(Q3-G): track 7.91 -> 0.00 mm
- net /USB/_~{RST}: track 20.2 -> 12.4 mm, vias 3 -> 2
- net Net-(IC1-OUTA): track 0.00 -> 7.08 mm, vias 0 -> 2
- net /FDCAN1+: track 16.5 -> 21.2 mm, vias 0 -> 2
- net /FDCAN2+: track 25.3 -> 30.0 mm, vias 0 -> 2
- net /FDCAN1-: track 16.5 -> 20.7 mm, vias 0 -> 2
- net /FDCAN2-: track 25.3 -> 29.3 mm, vias 0 -> 2
- net /USB/_~{PWR_EN}: track 2.03 -> 0.00 mm
- net /USB/_RXD: track 13.1 -> 14.0 mm
