File: hardware/isolation/PUTM_AMS_MASTER_ISOLATION.kicad_sch (KiCad schematic)
At the start: 11 parts, among them IC4 TLV61046ADBVT, U2 FT230XS

Commit message: chore: sync
Parts:
- added J1: Conn_02x10_Odd_Even, Connector_PinSocket_2.00mm:PinSocket_2x10_P2.00mm_Vertical, symbol Connector_Generic:Conn_02x10_Odd_Even
- added J3: Conn_02x04_Odd_Even, Connector_PinSocket_2.00mm:PinSocket_2x04_P2.00mm_Vertical, symbol Connector_Generic:Conn_02x04_Odd_Even
- added PS1: CCG15-24-12D, Samacsys:CCG152403S, symbol Samacsys:CCG15-24-12D

Commit message: chore: sync
Parts:
- added C1: C_Polarized_Small, Capacitor_THT:CP_Axial_L18.0mm_D10.0mm_P25.00mm_Horizontal, symbol Device:C_Polarized_Small
Other:
- note added: "594-2222-021-37221"
- note added: "810-ACM55V7012PLTL00"
- note added: "EC5DAW-24D12N"

Commit message: chore:sync
Parts:
- added C2, C3: 4.7uF, Capacitor_SMD:C_1812_4532Metric, symbol Device:C_Small
- added FL1: ACM55V-701-2PL-TL00, Samacsys:ACM55V7012PLTL00, symbol Samacsys:ACM55V-701-2PL-TL00
- added PS2: EC5DAW-24D12N, Samacsys:EC5DAW24D12N, symbol Samacsys:EC5DAW-24D12N
Other:
- moved on the sheet: C1

Commit message: chore: sync
Parts:
- removed C1: C_Polarized_Small, Capacitor_THT:CP_Axial_L18.0mm_D10.0mm_P25.00mm_Horizontal, symbol Device:C_Polarized_Small
- removed PS1: CCG15-24-12D, Samacsys:CCG152403S, symbol Samacsys:CCG15-24-12D
- added C1, C6, C7, C8: X1,Y2/1.8nF, Samacsys:CAPC5728X280N, symbol Device:C_Small
- added C10, C11, C12, C13, C4, C5, C9: 4.7uF, Capacitor_SMD:C_1812_4532Metric, symbol Device:C_Small
- added H1: MountingHole_Pad, MountingHole:MountingHole_3.2mm_M3_Pad_Via, symbol Mechanical:MountingHole_Pad
- added J2: M80-5102042, Samacsys:M80-51020YY, symbol Samacsys_kicad_sym:M80-5102042
- added J4: M80-5100642, Samacsys:M80-51006YY, symbol Samacsys_kicad_sym:M80-5100642
- added J5: M80-5100842, Samacsys:M80-51008YY, symbol Samacsys_kicad_sym:M80-5100842
- FL1: value ACM55V-701-2PL-TL00 -> 701@100MHz
Connections:
- net GND: now also FL1.2, C4.2, C5.2
- net at PS2.1 (-VIN): now also C2.2, C3.2, FL1.3, C6.2
- net at PS2.10 (-VOUT): now also C1.2, C11.2, C13.2
- net at PS2.16 (+VIN): now also C2.1, C3.1, FL1.4, C7.2
- net at PS2.8 (COM): now also C11.1, C12.2, C13.1, C9.2
- net at PS2.9 (+VOUT): now also C12.1, C8.2, C9.1
- net +24V: now reaches FL1.1
- net +24V: now also C4.1, C5.1
- new net Earth: C1.1, C6.1, C7.1, C8.1, H1.1
- no-connect marks 6 -> 7
Other:
- note removed: "EC5DAW-24D12N"
- moved on the sheet: C2, C3, C34, C44, FL1, PS2, R71, U2

Commit message: chore: sync
Parts:
- added C14, C15, C16, C17, C26, C68: 22uF, Capacitor_SMD:C_0805_2012Metric, symbol Device:C_Small
- added C18, C19, C20, C23, C24, C25, C27, C28: 1uF, Capacitor_SMD:C_0603_1608Metric, symbol Device:C_Small
- added C21, C22: 100nF, Capacitor_SMD:C_0603_1608Metric, symbol Device:C_Small
- added C29, C40, C45: 100n, Capacitor_SMD:C_0603_1608Metric_Pad1.08x0.95mm_HandSolder, symbol Device:C_Small
- added C32, C46: 10n, Capacitor_SMD:C_0603_1608Metric_Pad1.08x0.95mm_HandSolder, symbol Device:C_Small
- added C35, C41: 47u, Capacitor_SMD:C_0603_1608Metric_Pad1.08x0.95mm_HandSolder, symbol Device:C_Small
- added C38: 220n, Capacitor_SMD:C_0603_1608Metric_Pad1.08x0.95mm_HandSolder, symbol Device:C_Small
- added D16: 30V, Diode_SMD:D_SOD-123, symbol Device:D_Zener_Small
- added D5: 10V, Diode_SMD:D_SOD-123, symbol Device:D_Zener_Small
- added F2: 5A/24V, Fuse:Fuse_2920_7451Metric, symbol Device:Polyfuse_Small
- added F4: 5V/0.5A, Fuse:Fuse_0805_2012Metric, symbol Device:Polyfuse_Small
- added FB1, FB2, FB5, FB6: 2K@100MHz, Inductor_SMD:L_0603_1608Metric_Pad1.05x0.95mm_HandSolder, symbol Device:FerriteBead_Small
- added IC1, IC2, IC3, IC5: ISO7141, Package_SO:SSOP-16_3.9x4.9mm_P0.635mm, symbol Samacsys:ISO7141FCCDBQR
- added IC6: TPS54202HDDCR, Package_TO_SOT_SMD:SOT-23-6, symbol SamacsysNew:TPS54202HDDCR
- added K1: IM07DTS, Samacsys:IM23TS, symbol Samacsys_kicad_sym:IM07DTS
- added L4: 68uF/1.4A, Inductor_SMD:L_TDK_VLS6045EX_VLS6045AF, symbol Samacsys_kicad_sym:SRR4028-271Y
- added Q4: SI2347DS-T1-GE3, Package_TO_SOT_SMD:SOT-23-3, symbol Transistor_FET:Q_PMOS_GSD
- added R1: 100K, Resistor_SMD:R_0603_1608Metric_Pad0.98x0.95mm_HandSolder, symbol Device:R_Small
- added R10: 100k, Resistor_SMD:R_0603_1608Metric_Pad0.98x0.95mm_HandSolder, symbol Device:R_Small
- added R23: 510k, Resistor_SMD:R_0603_1608Metric, symbol Device:R_Small
- added R28: 100k, Resistor_SMD:R_0603_1608Metric, symbol Device:R_Small
- added R29: 13.3k, Resistor_SMD:R_0603_1608Metric, symbol Device:R_Small
- added TP3: TestPoint_Small, TestPoint:TestPoint_THTPad_D1.0mm_Drill0.5mm, symbol Connector:TestPoint_Small
- added U1: ADM3057ExRW, Package_SO:SOIC-20W_7.5x12.8mm_P1.27mm, symbol Interface_CAN_LIN:ADM3057ExRW
Connections:
- net +24V: now also C14.2, C17.2, C21.2, D5.1 (K), IC6.3 (VIN), Q4.2 (S), R23.2, TP3.1
- net GND: now also C14.1, C15.2, C16.2, C17.1, C21.1, C26.2, C40.1, C41.1, C45.2, C46.2, C68.2, D16.2 (A), IC6.1 (GND), R10.2, R29.1, U1.1 (GND1), U1.10 (GND1), U1.2 (GND1), U1.9 (AUXIN)
- new net: D5.2 (A), Q4.1 (G), R10.1
- new net: C46.1, FB6.1, U1.4 (VIO)
- new net: C29.2, C32.1, C35.2, FB1.1, U1.16 (VISOIN)
- new net: C19.1, IC1.2 (GND1), IC1.8 (GND1)
- new net: C23.1, IC2.15 (GND2), IC2.9 (GND2)
- new net: C20.1, IC2.2 (GND1), IC2.8 (GND1)
- new net: C28.1, IC5.15 (GND2), IC5.9 (GND2)
- new net: C27.1, IC5.2 (GND1), IC5.8 (GND1)
- new net: C41.2, FB5.1, U1.3 (VCC)
- new net: C18.1, IC1.15 (GND2), IC1.9 (GND2)
- new net: C25.1, IC3.15 (GND2), IC3.9 (GND2)
- new net: C24.1, IC3.2 (GND1), IC3.8 (GND1)
- new net: R1.2, U1.12 (RS)
- new net: C38.1, FB2.2, U1.18 (GNDISO), U1.20 (GNDISO)
- new net: C38.2, FB1.2, U1.19 (VISOOUT)
- new net +3.3V: C18.2, C23.2, C25.2, C28.2, C45.1, F4.2, FB6.2, IC1.16 (VCC2), IC2.16 (VCC2), IC3.16 (VCC2), IC5.16 (VCC2)
- new net +3.3VISO: C19.2, C20.2, C24.2, C27.2, IC1.1 (VCC1), IC2.1 (VCC1), IC3.1 (VCC1), IC5.1 (VCC1)
- new net +5V: C40.2, FB5.2
- new net BOOT_5V: C22.1, IC6.6 (BOOT)
- new net CAN1+: U1.14 (CANH)
- new net CAN1-: U1.13 (CANL)
- new net CAN1_RX: U1.5 (RXD)
- new net CAN1_TX: U1.7 (TXD)
- new net EN_5V: IC6.5 (EN), R23.1
- new net FB_5V: IC6.4 (FB), R28.1, R29.2
- new net F_24V: D16.1 (K), F2.1, Q4.3 (D)
- new net F_5V: C15.1, C16.1, C26.1, C68.1, F4.1, L4.2, R28.2
- new net GND_CAN_ISO1: C29.1, C32.2, C35.1, FB2.1, R1.1, U1.11 (GND2), U1.15 (GND2)
- new net STBY_CAN_1: U1.8 (STBY)
- new net SW_5V: C22.2, IC6.2 (SW), L4.1
- new net VDD: F2.2
- no-connect marks 7 -> 17
Other:
- note added: "1*"
- note added: "TVS, RRP AND DECOUPLING"
- note added: "idk co z tym zrobic chuj z tym?"
- note added: "zmienić na 3.3"
- moved on the sheet: C1, C11, C12, C13, C2, C3, C4, C5, C6, C7, C8, C9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

Commit message: chore:sync
Parts:
- removed L4: 68uF/1.4A, Inductor_SMD:L_TDK_VLS6045EX_VLS6045AF, symbol Samacsys_kicad_sym:SRR4028-271Y
- added L2: 68uF/0.3A, Samacsys:LQH3NPN100MMEL, symbol Samacsys:LQH3NPZ680MMEL
Connections:
- net F_5V: now also L2.2
- net SW_5V: now also L2.1
Other:
- note added: "ADD CMC in master on isolated ADC"
- note added: "reset z płytki"
Changed lines of the file:
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@@
 		)
 	)
+	(text "595-ISO6740FDWR"
+		(exclude_from_sim no)
+		(at 193.04 34.29 0)
+		(effects
+			(font
+				(size 1.27 1.27)
+			)
+		)
+	)
 	(text "594-2222-021-37221"
 		(exclude_from_sim no)
@@
 		)
 	)
+	(text "ADD CMC in master on isolated ADC"
+		(exclude_from_sim no)
+		(at 137.16 123.19 0)
+		(effects
+			(font
+				(size 1.27 1.27)
+			)
+		)
+	)
 	(text "zmienić na 3.3\n"
 		(exclude_from_sim no)
@@
 		)
 	)
+	(text "reset z płytki"
+		(exclude_from_sim no)
+		(at 199.39 78.74 0)
+		(effects
+			(font
+				(size 1.27 1.27)
+			)
+		)
+	)
 	(text "200-PTF12001LD "
 		(exclude_from_sim no)
@@
 	)
 	(symbol
+		(lib_id "Samacsys:LQH3NPZ680MMEL")
+		(at 508 55.88 90)
+		(unit 1)
+		(exclude_from_sim no)
+		(in_bom yes)
+		(on_board yes)
+		(dnp no)
+		(fields_autoplaced yes)
+		(property "Reference" "L2"
+			(at 508 49.53 90)
+			(effects
+				(font
+					(size 1.27 1.27)
+				)
+			)
+		)
+		(property "Value" "68uF/0.3A"
+			(at 508 52.07 90)
+			(effects
+				(font
+					(size 1.27 1.27)
+				)
+			)
+		)
+		(property "Footprint" "Samacsys:LQH3NPN100MMEL"
+			(at 604.19 39.37 0)
+			(effects
+				(font
+					(size 1.27 1.27)
+				)
+				(justify left top)
+				(hide yes)
+			)
+		)
+		(property "Datasheet" "https://search.murata.co.jp/Ceramy/image/img/P02/JELF243A-9140.pdf"
+			(at 704.19 39.37 0)
+			(effects
+				(font
+					(size 1.27 1.27)
+				)
+				(justify left top)
+				(hide yes)
+			)
+		)
+		(property "Description" "LQH3NPZ_ME Series Inductor 68uH +/-20% 1212 (3030)"
+			(at 508 55.88 0)
+			(effects
+				(font
+					(size 1.27 1.27)
+				)
+				(hide yes)
+			)
+		)
+		(property "Height" "1.5"
+			(at 904.19 39.37 0)
+			(effects
+				(font
+					(size 1.27 1.27)
+				)
+				(justify left top)
+				(hide yes)
+			)
+		)
+		(property "Mouser Part Number" "81-LQH3NPZ680MMEL"
+			(at 1004.19 39.37 0)
+			(effects
+				(font
+					(size 1.27 1.27)
+				)
+				(justify left top)
+				(hide yes)
+			)
+		)
+		(property "Mouser Price/Stock" "https://www.mouser.co.uk/ProductDetail/Murata-Electronics/LQH3NPZ680MMEL?qs=d0WKAl%252BL4KZmq4JOnggsSg%3D%3D"
+			(at 1104.19 39.37 0)
+			(effects
+				(font
+					(size 1.27 1.27)
+				)
+				(justify left top)
+				(hide yes)
+			)
+		)
+		(property "Manufacturer_Name" "Murata Electronics"
+			(at 1204.19 39.37 0)
+			(effects
+				(font
+					(size 1.27 1.27)
+				)
+				(justify left top)
+				(hide yes)
+			)
+		)
+		(property "Manufacturer_Part_Number" "LQH3NPZ680MMEL"
+			(at 1304.19 39.37 0)
+			(effects
+				(font
+					(size 1.27 1.27)
+				)
+				(justify left top)
+				(hide yes)
+			)
+		)
+		(pin "1"
+		)
+		(pin "2"
+		)
+		(instances
+			(project ""
+				(path "/9b254bae-97c6-45e7-8618-9f461c55b31a"
+					(reference "L2")
+					(unit 1)
+				)
+			)
+		)
+	)
+	(symbol
 		(lib_name "+5V_2")
 		(lib_id "power:+5V")
@@
 					(unit 1)
 				)
-			)
-		)
-	)
-	(symbol
-		(lib_id "Samacsys_kicad_sym:SRR4028-271Y")
-		(at 508 55.88 0)
-		(unit 1)
-		(exclude_from_sim no)
-		(in_bom yes)
-		(on_board yes)
-		(dnp no)
-		(property "Reference" "L4"
-			(at 508 50.8 0)
-			(effects
-				(font
-					(size 1.27 1.27)
-				)
-			)
-		)
-		(property "Value" "68uF/1.4A"
-			(at 508 53.34 0)
-			(effects
-				(font
-					(size 1.27 1.27)
-				)
-			)
-		)
-		(property "Footprint" "Inductor_SMD:L_TDK_VLS6045EX_VLS6045AF"
-			(at 516.89 64.77 0)
-			(effects
-				(font
-					(size 1.27 1.27)
-				)
-				(hide yes)
-			)
-		)
-		(property "Datasheet" "https://product.tdk.com/system/files/dam/doc/product/inductor/inductor/smd/catalog/inductor_commercial_power_vls6045ex_en.pdf"
-			(at 508 71.12 0)
-			(effects
-				(font
-					(size 1.27 1.27)
-				)
-				(justify left)
-				(hide yes)
-			)
-		)
-		(property "Description" "Power Inductors - SMD 68uH 20% 0.31mohms 1A 6x6x4.5mm"
-			(at 508 71.12 0)
-			(effects
-				(font
-					(size 1.27 1.27)
-				)
-				(justify left)
-				(hide yes)
-			)
-		)
-		(property "Height" "4.5mm"
-			(at 519.43 68.58 0)
-			(effects
-				(font
-					(size 1.27 1.27)
-				)
-				(justify left)
-				(hide yes)
-			)
-		)
-		(property "Mouser Part Number" "810-VLS6045EX-680M"
-			(at 508 71.12 0)
-			(effects
-				(font
-					(size 1.27 1.27)
-				)
-				(justify left)
-				(hide yes)
-			)
-		)
-		(property "Mouser Price/Stock" "https://www.mouser.pl/ProductDetail/TDK/VLS6045EX-680M?qs=oF%2FSscNnLpBLjomrKRgHaA%3D%3D"
-			(at 508 71.12 0)
-			(effects
-				(font
-					(size 1.27 1.27)
-				)
-				(justify left)
-				(hide yes)
-			)
-		)
-		(property "Manufacturer_Name" "TDK"
-			(at 508 71.12 0)
-			(effects
-				(font
-					(size 1.27 1.27)
-				)
-				(justify left)
-				(hide yes)
-			)
-		)
-		(property "Manufacturer_Part_Number" " VLS6045EX-680M"
-			(at 508 71.12 0)
-			(effects
-				(font
-					(size 1.27 1.27)
-				)
-				(justify left)
-				(hide yes)
-			)
-		)
-		(property "Arrow Part Number" ""
-			(at 508 55.88 0)
-			(effects
-				(font
-					(size 1.27 1.27)
-				)
-				(hide yes)
-			)
-		)
-		(property "Arrow Price/Stock" ""
-			(at 508 55.88 0)
-			(effects
-				(font
-					(size 1.27 1.27)
-				)
-				(hide yes)
-			)
-		)
-		(property "DigiKey Part Number" ""
-			(at 508 55.88 0)
-			(effects
-				(font
-					(size 1.27 1.27)
-				)
-			)
-		)
-		(pin "1"
-		)
-		(pin "2"
-		)
-		(instances
-			(project "PUTM_AMS_MASTER_ISOLATION"
-				(path "/9b254bae-97c6-45e7-8618-9f461c55b31a"
-					(reference "L4")
-					(unit 1)
-				)

Commit message: isolation schematich done
Parts:
- removed C1, C6, C7, C8: X1,Y2/1.8nF, Samacsys:CAPC5728X280N, symbol Device:C_Small
- removed C10, C11, C12, C13, C2, C3, C4, C5, C9: 4.7uF, Capacitor_SMD:C_1812_4532Metric, symbol Device:C_Small
- removed C14, C15, C16, C17, C26, C30, C31, C68: 22uF, Capacitor_SMD:C_0805_2012Metric, symbol Device:C_Small
- removed C18, C19, C20, C23, C24, C25, C27, C28: 1uF, Capacitor_SMD:C_0603_1608Metric, symbol Device:C_Small
- removed C21, C22, C34, C44: 100nF, Capacitor_SMD:C_0603_1608Metric, symbol Device:C_Small
- removed C29, C40, C45: 100n, Capacitor_SMD:C_0603_1608Metric_Pad1.08x0.95mm_HandSolder, symbol Device:C_Small
- removed C32, C46: 10n, Capacitor_SMD:C_0603_1608Metric_Pad1.08x0.95mm_HandSolder, symbol Device:C_Small
- removed C35, C41: 47u, Capacitor_SMD:C_0603_1608Metric_Pad1.08x0.95mm_HandSolder, symbol Device:C_Small
- removed C38: 220n, Capacitor_SMD:C_0603_1608Metric_Pad1.08x0.95mm_HandSolder, symbol Device:C_Small
- removed D16: 30V, Diode_SMD:D_SOD-123, symbol Device:D_Zener_Small
- removed D20: 8V, Diode_SMD:D_SOD-123, symbol Device:D_Zener_Small
- removed D5: 10V, Diode_SMD:D_SOD-123, symbol Device:D_Zener_Small
- removed F2: 5A/24V, Fuse:Fuse_2920_7451Metric, symbol Device:Polyfuse_Small
- removed F4: 5V/0.5A, Fuse:Fuse_0805_2012Metric, symbol Device:Polyfuse_Small
- removed FB1, FB2, FB5, FB6: 2K@100MHz, Inductor_SMD:L_0603_1608Metric_Pad1.05x0.95mm_HandSolder, symbol Device:FerriteBead_Small
- removed FL1: 701@100MHz, Samacsys:ACM55V7012PLTL00, symbol Samacsys:ACM55V-701-2PL-TL00
- removed H1: MountingHole_Pad, MountingHole:MountingHole_3.2mm_M3_Pad_Via, symbol Mechanical:MountingHole_Pad
- removed IC1, IC2, IC3, IC5: ISO7141, Package_SO:SSOP-16_3.9x4.9mm_P0.635mm, symbol Samacsys:ISO7141FCCDBQR
- removed IC4: TLV61046ADBVT, Package_TO_SOT_SMD:SOT-23-6, symbol Samacsys_kicad_sym:TLV61046ADBVT
- removed IC6: TPS54202HDDCR, Package_TO_SOT_SMD:SOT-23-6, symbol SamacsysNew:TPS54202HDDCR
- removed J1: Conn_02x10_Odd_Even, Connector_PinSocket_2.00mm:PinSocket_2x10_P2.00mm_Vertical, symbol Connector_Generic:Conn_02x10_Odd_Even
- removed J2: M80-5102042, Samacsys:M80-51020YY, symbol Samacsys_kicad_sym:M80-5102042
- removed J3: Conn_02x04_Odd_Even, Connector_PinSocket_2.00mm:PinSocket_2x04_P2.00mm_Vertical, symbol Connector_Generic:Conn_02x04_Odd_Even
- removed J4: M80-5100642, Samacsys:M80-51006YY, symbol Samacsys_kicad_sym:M80-5100642
- removed J5: M80-5100842, Samacsys:M80-51008YY, symbol Samacsys_kicad_sym:M80-5100842
- removed K1: IM07DTS, Samacsys:IM23TS, symbol Samacsys_kicad_sym:IM07DTS
- removed L1: 10uH, Inductor_SMD:L_1008_2520Metric, symbol Device:L
- removed L2: 68uF/0.3A, Samacsys:LQH3NPN100MMEL, symbol Samacsys:LQH3NPZ680MMEL
- removed PS2: EC5DAW-24D12N, Samacsys:EC5DAW24D12N, symbol Samacsys:EC5DAW-24D12N
- removed Q4: SI2347DS-T1-GE3, Package_TO_SOT_SMD:SOT-23-3, symbol Transistor_FET:Q_PMOS_GSD
- removed R1: 100K, Resistor_SMD:R_0603_1608Metric_Pad0.98x0.95mm_HandSolder, symbol Device:R_Small
- removed R10: 100k, Resistor_SMD:R_0603_1608Metric_Pad0.98x0.95mm_HandSolder, symbol Device:R_Small
- removed R23: 510k, Resistor_SMD:R_0603_1608Metric, symbol Device:R_Small
- removed R28: 100k, Resistor_SMD:R_0603_1608Metric, symbol Device:R_Small
- removed R29: 13.3k, Resistor_SMD:R_0603_1608Metric, symbol Device:R_Small
- removed R55: 649k, Resistor_SMD:R_0603_1608Metric, symbol Device:R_Small
- removed R62: 71.5k, Resistor_SMD:R_0603_1608Metric, symbol Device:R_Small
- removed R71: 10k, Resistor_SMD:R_0603_1608Metric, symbol Device:R_Small
- removed TP3: TestPoint_Small, TestPoint:TestPoint_THTPad_D1.0mm_Drill0.5mm, symbol Connector:TestPoint_Small
- removed U1: ADM3057ExRW, Package_SO:SOIC-20W_7.5x12.8mm_P1.27mm, symbol Interface_CAN_LIN:ADM3057ExRW
- removed U2: FT230XS, Package_SO:SSOP-16_3.9x4.9mm_P0.635mm, symbol Interface_USB:FT230XS
Connections:
- no-connect marks 17 -> 2
Other:
- added sheet Charger Detect (iso-input.kicad_sch)
- added sheet FDCAN CAR (fdcan.kicad_sch)
- added sheet FDCAN CHG (fdcan.kicad_sch)
- added sheet Interface connectors (interface-connectors.kicad_sch)
- added sheet Power (power.kicad_sch)
- added sheet Relay Driver M (relay-driver.kicad_sch)
- added sheet Relay Driver P (relay-driver.kicad_sch)
- added sheet Relay Driver PRE (relay-driver.kicad_sch)
- added sheet SDC Driver (sdc-driver.kicad_sch)
- added sheet Stack Connectors (stack-connectors.kicad_sch)
- added sheet USB (usb.kicad_sch)
- added sheet VDDRLY Detect (iso-input.kicad_sch)
- note added: "jak będzie miejsce to wsadzić duże kondensatory"
- note removed: "1*"
- note removed: "200-PTF10601LD"
- note removed: "200-PTF10801LD"
- note removed: "200-PTF12001LD"
- note removed: "200-PTT10601SD"
- note removed: "200-PTT10801SD"
- note removed: "200-PTT12001SD"
- note removed: "594-2222-021-37221"
- note removed: "595-ISO6740FDWR"
- note removed: "595-ISOUSB111DWXR"
- note removed: "595-ISOW1044BDFMR"
- note removed: "810-ACM55V7012PLTL00"
- note removed: "919-REC5A-0505SW/H2"
- note removed: "967-CCG152412D"
- note removed: "ADD CMC in master on isolated ADC"
- note removed: "TVS, RRP AND DECOUPLING"
- note removed: "add filtration"
- note removed: "idk co z tym zrobic chuj z tym?"
- note removed: "move 5A transisors to the isolated side, fuck it"
- note removed: "reset z płytki"
- note removed: "zmienić na 3.3"

Commit message: pcb finished
Other:
- sheet Interface connectors ports: added FDCAN1+, FDCAN1-, FDCAN2+, FDCAN2-; removed CANFD1+, CANFD1-, CANFD2+, CANFD2-
Changed lines of the file:
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@@
+		)
+	)
+	(label "FDCAN2-"
+		(at 223.52 238.76 0)
+		(effects
+			(font
+				(size 1.27 1.27)
+			)
+			(justify left bottom)
+		)
+	)
+	(label "FDCAN1-"
+		(at 223.52 213.36 0)
+		(effects
+			(font
+				(size 1.27 1.27)
+			)
+			(justify left bottom)
+		)
+	)
+	(label "CHARGER_DETECTION"
+		(at 125.73 184.15 0)
+		(effects
+			(font
+				(size 1.27 1.27)
+			)
+			(justify left bottom)
+		)
+	)
+	(label "CHARGER"
+		(at 224.79 184.15 0)
+		(effects
+			(font
+				(size 1.27 1.27)
+			)
+			(justify left bottom)
+		)
+	)
+	(label "FDCAN1+"
+		(at 223.52 205.74 0)
+		(effects
+			(font
+				(size 1.27 1.27)
+			)
+			(justify left bottom)
+		)
+	)
+	(label "TSMS_DETECTION"
+		(at 125.73 158.75 0)
+		(effects
+			(font
+				(size 1.27 1.27)
+			)
+			(justify left bottom)
+		)
+	)
+	(label "FDCAN2+"
+		(at 223.52 231.14 0)
+		(effects
+			(font
+				(size 1.27 1.27)
+			)
+			(justify left bottom)
 		)
 	)
@@
 			)
 		)
-		(pin "CANFD1+" bidirectional
+		(pin "FDCAN1+" bidirectional
 			(at 241.3 205.74 180)
 			(effects
@@
 			)
 		)
-		(pin "CANFD1-" bidirectional
+		(pin "FDCAN1-" bidirectional
 			(at 241.3 213.36 180)
 			(effects
@@
 			)
 		)
-		(pin "CANFD2+" bidirectional
+		(pin "FDCAN2+" bidirectional
 			(at 241.3 231.14 180)
 			(effects
@@
 			)
 		)
-		(pin "CANFD2-" bidirectional
+		(pin "FDCAN2-" bidirectional
 			(at 241.3 238.76 180)
 			(effects
