File: hardware/isolation/interface-connectors.kicad_sch (KiCad schematic)
At the start: 4 parts, among them J2 M80-5102042, J4 M80-5100642

Commit message: sync
Connections:
- net +5VUSB: now also J2.14; no longer J2.12
- net CANFD1+: now also J2.5; no longer J2.3
- net CANFD1-: now also J2.6; no longer J2.4
- net CANFD2+: now also J2.7; no longer J2.5
- net CANFD2-: now also J2.8; no longer J2.6
- net CHARGER_DETECTION: now also J2.9; no longer J2.13
- net D+: now also J2.4; no longer J2.2
- net D-: now also J2.3; no longer J2.1
- net GND: now also J2.11; no longer J2.7
- net GNDUSB: now also J2.13; no longer J2.11
- net SDC_IN: now also J2.2; no longer J2.8
- net SDC_OUT: now also J2.12; no longer J2.18
- net _VDDRLY: now reaches D17.2 (A)
- net _VDDRLY: now also J2.1; no longer J2.9
Other:
- note removed: "USBGND"

Commit message: pcb finished
Parts:
- added J5: Conn_01x02, Connector_PinHeader_2.00mm:PinHeader_1x02_P2.00mm_Vertical, symbol Connector_Generic:Conn_01x02
Connections:
- net CHARGER_DETECTION: now also J2.11; no longer J2.9
- net D+: now also J2.3; no longer J2.4
- net D-: now also J2.4; no longer J2.3
- net GND: now also J5.2 (Pin_2); no longer J2.11
- net CANFD1+ renamed FDCAN1+
- net CANFD1- renamed FDCAN1-
- net CANFD2+ renamed FDCAN2+
- net CANFD2- renamed FDCAN2-
- new net +24V: J5.1 (Pin_1)
- no-connect marks 4 -> 5
