File: hardware/isolation/stack-connectors.kicad_sch (KiCad schematic)
At the start: 2 parts, among them J1 Conn_02x10_Odd_Even, J3 Conn_02x04_Odd_Even

Commit message: pcb finished
Connections:
- net +3.3VA renamed +3.3VAISO
- net +3.3VIO renamed +3.3VIOISO
- net +5VA renamed +5VAISO
- net +5VIO renamed +5VIOISO
- net GND renamed GNDISO
Changed lines of the file:
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@@
 			)
 		)
-		(property "Value" "+5VIO"
+		(property "Value" "+5VIOISO"
 			(at 163.83 107.95 90)
 			(show_name no)
@@
 			)
 		)
-		(property "Value" "GND"
+		(property "Value" "GNDISO"
 			(at 163.83 90.17 90)
 			(show_name no)
@@
 			)
 		)
-		(property "Value" "GND"
+		(property "Value" "GNDISO"
 			(at 142.24 80.01 0)
 			(show_name no)
@@
 			)
 		)
-		(property "Value" "GND"
+		(property "Value" "GNDISO"
 			(at 160.02 119.38 0)
 			(show_name no)
@@
 			)
 		)
-		(property "Value" "+5VA"
+		(property "Value" "+5VAISO"
 			(at 138.43 107.95 90)
 			(show_name no)
@@
 			)
 		)
-		(property "Value" "+3.3VIO"
+		(property "Value" "+3.3VIOISO"
 			(at 163.83 105.41 90)
 			(show_name no)
@@
 			)
 		)
-		(property "Value" "+3.3VA"
+		(property "Value" "+3.3VAISO"
 			(at 138.43 113.03 90)
 			(show_name no)
