File: hardware/isolation/stack-connectors.kicad_sch (KiCad schematic)
At the start: 2 parts, among them J1 Conn_02x10_Odd_Even, J3 Conn_02x04_Odd_Even

Commit message: bom update
Parts:
- J1: Mouser Part Number (none) -> 200-SQT12001LD
- J3: Mouser Part Number (none) -> 200-SQT10801LD
Changed lines of the file:
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@@
+			)
+		)
+		(property "Mouser Part Number" "200-SQT12001LD "
+			(at 149.86 100.33 0)
+			(hide yes)
+			(show_name no)
+			(do_not_autoplace no)
+			(effects
+				(font
+					(size 1.27 1.27)
+				)
 			)
 		)
@@
 			(at 152.4 68.58 0)
 			(hide yes)
+			(show_name no)
+			(do_not_autoplace no)
+			(effects
+				(font
+					(size 1.27 1.27)
+				)
+			)
+		)
+		(property "Mouser Part Number" "200-SQT10801LD"
+			(at 152.4 68.58 0)
+			(hide yes)
