File: hardware/isolation/fdcan.kicad_sch (KiCad schematic)
At the start: 17 parts, among them U1 ADM3057ExRW

Commit message: sync
Parts:
- C45, C46, C57, C61, C62: footprint Capacitor_SMD:C_0603_1608Metric_Pad1.08x0.95mm_HandSolder -> Capacitor_SMD:C_0805_2012Metric; Mouser Part Number (none) -> 81-GRM21BR61A476ME5L
- FB1, FB2, FB5, FB6: footprint Inductor_SMD:L_0603_1608Metric_Pad1.05x0.95mm_HandSolder -> Inductor_SMD:L_0805_2012Metric; Mouser Part Number (none) -> 623-2508052027Y1
Connections:
- net RS: now reaches R1.2, U1.12 (RS)
- net GNDCANOUT: now reaches C38.1, FB2.2, U1.18 (GNDISO), U1.20 (GNDISO)
- net VDDCANOUT: now reaches C38.2, FB1.2, U1.19 (VISOOUT)
- net VCC: now reaches C61.1, FB6.1, U1.3 (VCC)
- net VIO: now reaches C45.1, FB5.1, U1.4 (VIO)
Changed lines of the file:
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@@
+		)
+	)
+	(wire
+		(pts
+			(xy 128.27 76.2) (xy 135.89 76.2)
+		)
+		(stroke
+			(width 0)
+			(type default)
 		)
 	)
@@
 	(wire
 		(pts
-			(xy 135.89 76.2) (xy 128.27 76.2)
-		)
-		(stroke
-			(width 0)
-			(type default)
-		)
-	)
-	(wire
-		(pts
 			(xy 167.64 78.74) (xy 175.26 78.74)
 		)
@@
 	(wire
 		(pts
-			(xy 135.89 91.44) (xy 128.27 91.44)
-		)
-		(stroke
-			(width 0)
-			(type default)
-		)
-	)
-	(wire
-		(pts
 			(xy 231.14 87.63) (xy 231.14 91.44)
 		)
@@
 			(type solid)
 			(color 132 0 0 1)
+		)
+	)
+	(wire
+		(pts
+			(xy 128.27 91.44) (xy 135.89 91.44)
+		)
+		(stroke
+			(width 0)
+			(type default)
 		)
 	)
@@
 		)
 	)
+	(label "VDDCANOUT"
+		(at 135.89 76.2 180)
+		(effects
+			(font
+				(size 0.508 0.508)
+			)
+			(justify right bottom)
+		)
+	)
+	(label "VCC"
+		(at 167.64 76.2 0)
+		(effects
+			(font
+				(size 0.508 0.508)
+			)
+			(justify left bottom)
+		)
+	)
+	(label "VIO"
+		(at 167.64 78.74 0)
+		(effects
+			(font
+				(size 0.508 0.508)
+			)
+			(justify left bottom)
+		)
+	)
+	(label "RS"
+		(at 135.89 121.92 180)
+		(effects
+			(font
+				(size 0.508 0.508)
+			)
+			(justify right bottom)
+		)
+	)
 	(label "VDDCAN"
 		(at 110.49 76.2 180)
@@
 			(font
 				(size 1.27 1.27)
+			)
+			(justify right bottom)
+		)
+	)
+	(label "GNDCANOUT"
+		(at 135.89 91.44 180)
+		(effects
+			(font
+				(size 0.508 0.508)
 			)
 			(justify right bottom)
@@
 			)
 		)
-		(property "Footprint" "Capacitor_SMD:C_0603_1608Metric_Pad1.08x0.95mm_HandSolder"
+		(property "Footprint" "Capacitor_SMD:C_0805_2012Metric"
 			(at 231.14 85.09 0)
 			(hide yes)
@@
 			)
 		)
-		(property "Datasheet" ""
+		(property "Datasheet" "https://ds.murata.com/simsurfing/mlcc.html?partnumbers=%5B%22GRM21BR61A476ME15%22%5D&oripartnumbers=%5B%22GRM21BR61A476ME15L%22%5D&rgear=suaykx&rgearinfo=com"
 			(at 231.14 85.09 0)
 			(hide yes)
@@
 		)
 		(property "Description" "Unpolarized capacitor, small symbol"
+			(at 231.14 85.09 0)
+			(hide yes)
+			(show_name no)
+			(do_not_autoplace no)
+			(effects
+				(font
+					(size 1.27 1.27)
+				)
+			)
+		)
+		(property "Mouser Part Number" "81-GRM21BR61A476ME5L"
 			(at 231.14 85.09 0)
 			(hide yes)
@@
 			)
 		)
-		(property "Footprint" "Inductor_SMD:L_0603_1608Metric_Pad1.05x0.95mm_HandSolder"
+		(property "Footprint" "Inductor_SMD:L_0805_2012Metric"
 			(at 120.65 93.218 90)
 			(hide yes)
@@
 			)
 		)
-		(property "Datasheet" "https://www.mouser.pl/ProductDetail/Eaton-Electronics/MFBW1V1608-202-R?qs=W%2FMpXkg%252BdQ4ShGRk3jgFwA%3D%3D"
+		(property "Datasheet" "--"
 			(at 120.65 91.44 0)
 			(hide yes)
@@
 		(property "Description" "Ferrite bead, small symbol"
 			(at 120.65 91.44 0)
+			(hide yes)
+			(show_name no)
+			(do_not_autoplace no)
+			(effects
+				(font
+					(size 1.27 1.27)
+				)
+			)
+		)
+		(property "Mouser Part Number" "623-2508052027Y1 "
+			(at 120.65 91.44 90)
 			(hide yes)
 			(show_name no)
@@
 			)
 		)
-		(property "Footprint" "Capacitor_SMD:C_0603_1608Metric_Pad1.08x0.95mm_HandSolder"
+		(property "Footprint" "Capacitor_SMD:C_0805_2012Metric"
 			(at 113.03 83.82 0)
 			(hide yes)
@@
 			)
 		)
-		(property "Datasheet" ""
+		(property "Datasheet" "https://ds.murata.com/simsurfing/mlcc.html?partnumbers=%5B%22GRM21BR61A476ME15%22%5D&oripartnumbers=%5B%22GRM21BR61A476ME15L%22%5D&rgear=suaykx&rgearinfo=com"
 			(at 113.03 83.82 0)
 			(hide yes)
@@
 		)
 		(property "Description" "Unpolarized capacitor, small symbol"
+			(at 113.03 83.82 0)
+			(hide yes)
+			(show_name no)
+			(do_not_autoplace no)
+			(effects
+				(font
+					(size 1.27 1.27)
+				)
+			)
+		)
+		(property "Mouser Part Number" "81-GRM21BR61A476ME5L"
 			(at 113.03 83.82 0)
 			(hide yes)
@@
 			)
 		)
-		(property "Footprint" "Capacitor_SMD:C_0603_1608Metric_Pad1.08x0.95mm_HandSolder"
+		(property "Footprint" "Capacitor_SMD:C_0805_2012Metric"
 			(at 210.82 85.09 0)
 			(hide yes)
@@
 			)
 		)
-		(property "Datasheet" ""
+		(property "Datasheet" "https://ds.murata.com/simsurfing/mlcc.html?partnumbers=%5B%22GRM21BR61A476ME15%22%5D&oripartnumbers=%5B%22GRM21BR61A476ME15L%22%5D&rgear=suaykx&rgearinfo=com"
 			(at 210.82 85.09 0)
 			(hide yes)
@@
 		)
 		(property "Description" "Unpolarized capacitor, small symbol"
+			(at 210.82 85.09 0)
+			(hide yes)
+			(show_name no)
+			(do_not_autoplace no)
+			(effects
+				(font
+					(size 1.27 1.27)
+				)
+			)
+		)
+		(property "Mouser Part Number" "81-GRM21BR61A476ME5L"
 			(at 210.82 85.09 0)
 			(hide yes)
@@
 			)
 		)
-		(property "Footprint" "Inductor_SMD:L_0603_1608Metric_Pad1.05x0.95mm_HandSolder"
+		(property "Footprint" "Inductor_SMD:L_0805_2012Metric"
 			(at 185.42 80.518 90)
 			(hide yes)
@@
 			)
 		)
-		(property "Datasheet" "https://www.mouser.pl/ProductDetail/Eaton-Electronics/MFBW1V1608-202-R?qs=W%2FMpXkg%252BdQ4ShGRk3jgFwA%3D%3D"
+		(property "Datasheet" "--"
 			(at 185.42 78.74 0)
 			(hide yes)
@@
 		(property "Description" "Ferrite bead, small symbol"
 			(at 185.42 78.74 0)
+			(hide yes)
+			(show_name no)
+			(do_not_autoplace no)
+			(effects
+				(font
+					(size 1.27 1.27)
+				)
+			)
+		)
+		(property "Mouser Part Number" "623-2508052027Y1 "
+			(at 185.42 78.74 90)
 			(hide yes)
 			(show_name no)
@@
 			)
 		)
-		(property "Footprint" "Inductor_SMD:L_0603_1608Metric_Pad1.05x0.95mm_HandSolder"
+		(property "Footprint" "Inductor_SMD:L_0805_2012Metric"
 			(at 120.65 77.978 90)
 			(hide yes)
@@
 			)
 		)
-		(property "Datasheet" "https://www.mouser.pl/ProductDetail/Eaton-Electronics/MFBW1V1608-202-R?qs=W%2FMpXkg%252BdQ4ShGRk3jgFwA%3D%3D"
+		(property "Datasheet" "--"
 			(at 120.65 76.2 0)
 			(hide yes)
@@
 		(property "Description" "Ferrite bead, small symbol"
 			(at 120.65 76.2 0)
+			(hide yes)
+			(show_name no)
+			(do_not_autoplace no)
+			(effects
+				(font
+					(size 1.27 1.27)
+				)
+			)
+		)
+		(property "Mouser Part Number" "623-2508052027Y1 "
+			(at 120.65 76.2 90)
 			(hide yes)
 			(show_name no)
@@
 			)
 		)
-		(property "Footprint" "Capacitor_SMD:C_0603_1608Metric_Pad1.08x0.95mm_HandSolder"
+		(property "Footprint" "Capacitor_SMD:C_0805_2012Metric"
 			(at 195.58 85.09 0)
 			(hide yes)
@@
 			)
 		)
-		(property "Datasheet" ""
+		(property "Datasheet" "https://ds.murata.com/simsurfing/mlcc.html?partnumbers=%5B%22GRM21BR61A476ME15%22%5D&oripartnumbers=%5B%22GRM21BR61A476ME15L%22%5D&rgear=suaykx&rgearinfo=com"
 			(at 195.58 85.09 0)
 			(hide yes)
@@
 		)
 		(property "Description" "Unpolarized capacitor, small symbol"
+			(at 195.58 85.09 0)
+			(hide yes)
+			(show_name no)
+			(do_not_autoplace no)
+			(effects
+				(font
+					(size 1.27 1.27)
+				)
+			)
+		)
+		(property "Mouser Part Number" "81-GRM21BR61A476ME5L"
 			(at 195.58 85.09 0)
 			(hide yes)
@@
 			)
 		)
-		(property "Footprint" "Inductor_SMD:L_0603_1608Metric_Pad1.05x0.95mm_HandSolder"
+		(property "Footprint" "Inductor_SMD:L_0805_2012Metric"
 			(at 220.98 77.978 90)
 			(hide yes)
@@
 			)
 		)
-		(property "Datasheet" "https://www.mouser.pl/ProductDetail/Eaton-Electronics/MFBW1V1608-202-R?qs=W%2FMpXkg%252BdQ4ShGRk3jgFwA%3D%3D"
+		(property "Datasheet" "--"
 			(at 220.98 76.2 0)
 			(hide yes)
@@
 		(property "Description" "Ferrite bead, small symbol"
 			(at 220.98 76.2 0)
+			(hide yes)
+			(show_name no)
+			(do_not_autoplace no)
+			(effects
+				(font
+					(size 1.27 1.27)
+				)
+			)
+		)
+		(property "Mouser Part Number" "623-2508052027Y1 "
+			(at 220.98 76.2 90)
 			(hide yes)
 			(show_name no)
@@
 			)
 		)
-		(property "Footprint" "Capacitor_SMD:C_0603_1608Metric_Pad1.08x0.95mm_HandSolder"
+		(property "Footprint" "Capacitor_SMD:C_0805_2012Metric"
 			(at 175.26 85.09 0)
 			(hide yes)
@@
 			)
 		)
-		(property "Datasheet" ""
+		(property "Datasheet" "https://ds.murata.com/simsurfing/mlcc.html?partnumbers=%5B%22GRM21BR61A476ME15%22%5D&oripartnumbers=%5B%22GRM21BR61A476ME15L%22%5D&rgear=suaykx&rgearinfo=com"
 			(at 175.26 85.09 0)
 			(hide yes)
@@
 			(at 175.26 85.09 0)
 			(hide yes)
+			(show_name no)
+			(do_not_autoplace no)
+			(effects
+				(font
+					(size 1.27 1.27)
+				)
+			)
+		)
+		(property "Mouser Part Number" "81-GRM21BR61A476ME5L"
+			(at 175.26 85.09 0)
+			(hide yes)

Commit message: pcb finished
Parts:
- added D19: 5.3V/400W, Package_TO_SOT_SMD:SOT-23-3, symbol Power_Protection:ESDA5V3L
- C29, C32, C38: footprint Capacitor_SMD:C_0603_1608Metric_Pad1.08x0.95mm_HandSolder -> Capacitor_SMD:C_0603_1608Metric
- R1: footprint Resistor_SMD:R_0603_1608Metric_Pad0.98x0.95mm_HandSolder -> Resistor_SMD:R_0603_1608Metric
Connections:
- net CANH: now also D19.1 (K)
- net CANL: now also D19.2 (K)
- no-connect marks 2 -> 3
Changed lines of the file:
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@@
 	)
 	(junction
+		(at 78.74 101.6)
+		(diameter 0)
+		(color 0 0 0 0)
+	)
+	(junction
 		(at 231.14 91.44)
 		(diameter 0)
@@
 	)
 	(junction
-		(at 195.58 91.44)
+		(at 125.73 127)
 		(diameter 0)
 		(color 0 0 0 0)
 	)
 	(junction
-		(at 125.73 127)
+		(at 115.57 114.3)
 		(diameter 0)
 		(color 0 0 0 0)
 	)
 	(junction
-		(at 115.57 114.3)
+		(at 195.58 91.44)
 		(diameter 0)
 		(color 0 0 0 0)
@@
 	)
 	(junction
+		(at 73.66 99.06)
+		(diameter 0)
+		(color 0 0 0 0)
+	)
+	(junction
 		(at 175.26 91.44)
 		(diameter 0)
@@
 		(at 167.64 127)
 	)
+	(no_connect
+		(at 76.2 114.3)
+	)
+	(wire
+		(pts
+			(xy 78.74 101.6) (xy 135.89 101.6)
+		)
+		(stroke
+			(width 0)
+			(type default)
+		)
+	)
 	(wire
 		(pts
@@
 	(wire
 		(pts
+			(xy 167.64 101.6) (xy 170.18 101.6)
+		)
+		(stroke
+			(width 0)
+			(type default)
+		)
+	)
+	(wire
+		(pts
 			(xy 231.14 73.66) (xy 231.14 76.2)
 		)
@@
 	(wire
 		(pts
-			(xy 167.64 101.6) (xy 170.18 101.6)
+			(xy 104.14 114.3) (xy 104.14 118.11)
 		)
 		(stroke
@@
 	(wire
 		(pts
-			(xy 104.14 114.3) (xy 104.14 118.11)
+			(xy 187.96 78.74) (xy 195.58 78.74)
 		)
 		(stroke
@@
 	(wire
 		(pts
-			(xy 187.96 78.74) (xy 195.58 78.74)
+			(xy 167.64 99.06) (xy 170.18 99.06)
 		)
 		(stroke
@@
 		)
 	)
+	(wire
+		(pts
+			(xy 78.74 101.6) (xy 78.74 104.14)
+		)
+		(stroke
+			(width 0)
+			(type default)
+		)
+	)
 	(polyline
 		(pts
@@
 	(wire
 		(pts
+			(xy 73.66 99.06) (xy 73.66 104.14)
+		)
+		(stroke
+			(width 0)
+			(type default)
+		)
+	)
+	(wire
+		(pts
 			(xy 113.03 76.2) (xy 118.11 76.2)
 		)
@@
 	(wire
 		(pts
-			(xy 133.35 101.6) (xy 135.89 101.6)
+			(xy 63.5 101.6) (xy 78.74 101.6)
 		)
 		(stroke
@@
 	(wire
 		(pts
-			(xy 133.35 99.06) (xy 135.89 99.06)
+			(xy 63.5 99.06) (xy 73.66 99.06)
 		)
 		(stroke
@@
 	(wire
 		(pts
-			(xy 231.14 91.44) (xy 231.14 93.98)
+			(xy 231.14 91.44) (xy 231.14 92.71)
 		)
 		(stroke
@@
 		)
 	)
-	(wire
-		(pts
-			(xy 167.64 99.06) (xy 170.18 99.06)
-		)
-		(stroke
-			(width 0)
-			(type default)
-		)
-	)
 	(polyline
 		(pts
@@
 	(wire
 		(pts
-			(xy 195.58 91.44) (xy 195.58 93.98)
+			(xy 195.58 91.44) (xy 195.58 92.71)
 		)
 		(stroke
@@
 	(wire
 		(pts
+			(xy 73.66 99.06) (xy 135.89 99.06)
+		)
+		(stroke
+			(width 0)
+			(type default)
+		)
+	)
+	(wire
+		(pts
 			(xy 123.19 91.44) (xy 128.27 91.44)
 		)
@@
 	(hierarchical_label "CANH"
 		(shape bidirectional)
-		(at 133.35 99.06 180)
+		(at 63.5 99.06 180)
 		(effects
 			(font
@@
 	(hierarchical_label "CANL"
 		(shape bidirectional)
-		(at 133.35 101.6 180)
+		(at 63.5 101.6 180)
 		(effects
 			(font
@@
 	(symbol
 		(lib_id "power:GND")
-		(at 231.14 93.98 0)
+		(at 231.14 92.71 0)
 		(unit 1)
 		(body_style 1)
@@
 		(dnp no)
 		(property "Reference" "#PWR051"
-			(at 231.14 100.33 0)
+			(at 231.14 99.06 0)
 			(hide yes)
 			(show_name no)
@@
 		)
 		(property "Value" "GNDISO"
-			(at 231.14 97.79 0)
+			(at 231.14 96.52 0)
 			(show_name no)
 			(do_not_autoplace no)
@@
 		)
 		(property "Footprint" ""
-			(at 231.14 93.98 0)
+			(at 231.14 92.71 0)
 			(hide yes)
 			(show_name no)
@@
 		)
 		(property "Datasheet" ""
-			(at 231.14 93.98 0)
+			(at 231.14 92.71 0)
 			(hide yes)
 			(show_name no)
@@
 		)
 		(property "Description" "Power symbol creates a global label with name \"GND\" , ground"
-			(at 231.14 93.98 0)
+			(at 231.14 92.71 0)
 			(hide yes)
 			(show_name no)
@@
 			)
 		)
-		(property "Footprint" "Capacitor_SMD:C_0603_1608Metric_Pad1.08x0.95mm_HandSolder"
+		(property "Footprint" "Capacitor_SMD:C_0603_1608Metric"
 			(at 115.57 120.65 0)
 			(hide yes)
@@
 			)
 		)
-		(property "Footprint" "Capacitor_SMD:C_0603_1608Metric_Pad1.08x0.95mm_HandSolder"
+		(property "Footprint" "Capacitor_SMD:C_0603_1608Metric"
 			(at 104.14 120.65 0)
 			(hide yes)
@@
 	)
 	(symbol
+		(lib_id "Power_Protection:ESDA5V3L")
+		(at 76.2 109.22 0)
+		(unit 1)
+		(body_style 1)
+		(exclude_from_sim no)
+		(in_bom yes)
+		(on_board yes)
+		(in_pos_files yes)
+		(dnp no)
+		(property "Reference" "D19"
+			(at 69.85 107.95 0)
+			(show_name no)
+			(do_not_autoplace no)
+			(effects
+				(font
+					(size 1.27 1.27)
+				)
+				(justify right)
+			)
+		)
+		(property "Value" "5.3V/400W"
+			(at 69.85 110.49 0)
+			(show_name no)
+			(do_not_autoplace no)
+			(effects
+				(font
+					(size 1.27 1.27)
+				)
+				(justify right)
+			)
+		)
+		(property "Footprint" "Package_TO_SOT_SMD:SOT-23-3"
+			(at 60.96 119.38 0)
+			(hide yes)
+			(show_name no)
+			(do_not_autoplace no)
+			(effects
+				(font
+					(size 1.27 1.27)
+				)
+				(justify left)
+			)
+		)
+		(property "Datasheet" "https://www.st.com/resource/en/datasheet/esdal.pdf"
+			(at 76.2 124.46 0)
+			(hide yes)
+			(show_name no)
+			(do_not_autoplace no)
+			(effects
+				(font
+					(size 1.27 1.27)
+				)
+			)
+		)
+		(property "Description" "TVS Diode Array, 5.5V Standoff, 2 Channels, SOT23"
+			(at 76.2 121.92 0)
+			(hide yes)
+			(show_name no)
+			(do_not_autoplace no)
+			(effects
+				(font
+					(size 1.27 1.27)
+				)
+			)
+		)
+		(property "Mouser Part Number" "511-ESDA5V3L"
+			(at 76.2 109.22 0)
+			(hide yes)
+			(show_name no)
+			(do_not_autoplace no)
+			(effects
+				(font
+					(size 1.27 1.27)
+				)
+			)
+		)
+		(pin "1"
+		)
+		(pin "2"
+		)
+		(pin "3"
+		)
+		(instances
+			(project "PUTM_AMS_MASTER_ISOLATION"
+				(path "/9b254bae-97c6-45e7-8618-9f461c55b31a/bb7c4aa8-5d23-481b-8672-1d87fa8c6d83"
+					(reference "D19")
+					(unit 1)
+				)
+				(path "/9b254bae-97c6-45e7-8618-9f461c55b31a/c0d62127-a5e4-40e6-9bd1-c5a7f1ecee97"
+					(reference "D20")
+					(unit 1)
+				)
+			)
+		)
+	)
+	(symbol
 		(lib_id "power:GND")
-		(at 195.58 93.98 0)
+		(at 195.58 92.71 0)
 		(unit 1)
 		(body_style 1)
@@
 		(dnp no)
 		(property "Reference" "#PWR027"
-			(at 195.58 100.33 0)
+			(at 195.58 99.06 0)
 			(hide yes)
 			(show_name no)
@@
 		)
 		(property "Value" "GNDISO"
-			(at 195.58 97.79 0)
+			(at 195.58 96.52 0)
 			(show_name no)
 			(do_not_autoplace no)
@@
 		)
 		(property "Footprint" ""
-			(at 195.58 93.98 0)
+			(at 195.58 92.71 0)
 			(hide yes)
 			(show_name no)
@@
 		)
 		(property "Datasheet" ""
-			(at 195.58 93.98 0)
+			(at 195.58 92.71 0)
 			(hide yes)
 			(show_name no)
@@
 		)
 		(property "Description" "Power symbol creates a global label with name \"GND\" , ground"
-			(at 195.58 93.98 0)
+			(at 195.58 92.71 0)
 			(hide yes)
 			(show_name no)
@@
 			)
 		)
-		(property "Footprint" "Capacitor_SMD:C_0603_1608Metric_Pad1.08x0.95mm_HandSolder"
+		(property "Footprint" "Capacitor_SMD:C_0603_1608Metric"
 			(at 128.27 83.82 0)
 			(hide yes)
@@
 			)
 		)
-		(property "Footprint" "Resistor_SMD:R_0603_1608Metric_Pad0.98x0.95mm_HandSolder"
+		(property "Footprint" "Resistor_SMD:R_0603_1608Metric"
 			(at 130.81 121.92 0)
 			(hide yes)

Commit message: made bigger gap span between isolated ground planes
Parts:
- C21, C36: Mouser Part Number 80-CAS21C222KARFC -> 80-CAS26C182KARFC
Changed lines of the file:
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@@
 			)
 		)
-		(property "Mouser Part Number" "80-CAS21C222KARFC "
+		(property "Mouser Part Number" "80-CAS26C182KARFC"
 			(at 165.1 137.16 0)
 			(hide yes)
@@
 			)
 		)
-		(property "Mouser Part Number" "80-CAS21C222KARFC "
+		(property "Mouser Part Number" "80-CAS26C182KARFC"
 			(at 137.16 137.16 0)
 			(hide yes)
