File: hardware/isolation/fdcan.kicad_sch (KiCad schematic)
At the start: 18 parts, among them U1 ADM3057ExRW

Commit message: sync
Parts:
- added R89: 120, Resistor_SMD:R_0603_1608Metric, symbol Device:R_Small
Connections:
- net CANH: now also R89.1
- net CANL: now also R89.2
Changed lines of the file:
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@@
+	)
+	(junction
+		(at 57.15 88.9)
+		(diameter 0)
+		(color 0 0 0 0)
 	)
 	(junction
@@
 	)
 	(junction
+		(at 78.74 101.6)
+		(diameter 0)
+		(color 0 0 0 0)
+	)
+	(junction
 		(at 210.82 76.2)
 		(diameter 0)
@@
 	)
 	(junction
-		(at 78.74 101.6)
-		(diameter 0)
-		(color 0 0 0 0)
-	)
-	(junction
 		(at 231.14 91.44)
 		(diameter 0)
@@
 	)
 	(junction
+		(at 73.66 99.06)
+		(diameter 0)
+		(color 0 0 0 0)
+	)
+	(junction
 		(at 175.26 78.74)
 		(diameter 0)
@@
 	)
 	(junction
+		(at 57.15 101.6)
+		(diameter 0)
+		(color 0 0 0 0)
+	)
+	(junction
 		(at 104.14 127)
 		(diameter 0)
@@
 	(junction
 		(at 151.13 152.4)
-		(diameter 0)
-		(color 0 0 0 0)
-	)
-	(junction
-		(at 73.66 99.06)
 		(diameter 0)
 		(color 0 0 0 0)
@@
 	(wire
 		(pts
+			(xy 73.66 88.9) (xy 73.66 99.06)
+		)
+		(stroke
+			(width 0)
+			(type default)
+		)
+	)
+	(wire
+		(pts
 			(xy 170.18 106.68) (xy 170.18 109.22)
 		)
@@
 	(wire
 		(pts
+			(xy 57.15 88.9) (xy 73.66 88.9)
+		)
+		(stroke
+			(width 0)
+			(type default)
+		)
+	)
+	(wire
+		(pts
 			(xy 128.27 76.2) (xy 135.89 76.2)
 		)
@@
 	(wire
 		(pts
+			(xy 57.15 97.79) (xy 57.15 101.6)
+		)
+		(stroke
+			(width 0)
+			(type default)
+		)
+	)
+	(wire
+		(pts
 			(xy 115.57 127) (xy 125.73 127)
 		)
@@
 	(wire
 		(pts
+			(xy 57.15 101.6) (xy 78.74 101.6)
+		)
+		(stroke
+			(width 0)
+			(type default)
+		)
+	)
+	(wire
+		(pts
 			(xy 167.64 78.74) (xy 175.26 78.74)
 		)
@@
 	(wire
 		(pts
-			(xy 63.5 101.6) (xy 78.74 101.6)
+			(xy 50.8 101.6) (xy 57.15 101.6)
 		)
 		(stroke
@@
 	(wire
 		(pts
-			(xy 63.5 99.06) (xy 73.66 99.06)
+			(xy 50.8 88.9) (xy 57.15 88.9)
 		)
 		(stroke
@@
 		(pts
 			(xy 101.6 127) (xy 104.14 127)
+		)
+		(stroke
+			(width 0)
+			(type default)
+		)
+	)
+	(wire
+		(pts
+			(xy 57.15 88.9) (xy 57.15 92.71)
 		)
 		(stroke
@@
 	(hierarchical_label "CANH"
 		(shape bidirectional)
-		(at 63.5 99.06 180)
+		(at 50.8 88.9 180)
 		(effects
 			(font
@@
 	(hierarchical_label "CANL"
 		(shape bidirectional)
-		(at 63.5 101.6 180)
+		(at 50.8 101.6 180)
 		(effects
 			(font
@@
 					(unit 1)
 				)
+			)
+		)
+	)
+	(symbol
+		(lib_id "Device:R_Small")
+		(at 57.15 95.25 0)
+		(mirror y)
+		(unit 1)
+		(body_style 1)
+		(exclude_from_sim no)
+		(in_bom yes)
+		(on_board yes)
+		(in_pos_files yes)
+		(dnp no)
+		(property "Reference" "R89"
+			(at 59.69 93.98 0)
+			(show_name no)
+			(do_not_autoplace no)
+			(effects
+				(font
+					(size 1.27 1.27)
+				)
+				(justify right)
+			)
+		)
+		(property "Value" "120"
+			(at 59.69 96.52 0)
+			(show_name no)
+			(do_not_autoplace no)
+			(effects
+				(font
+					(size 1.27 1.27)
+				)
+				(justify right)
+			)
+		)
+		(property "Footprint" "Resistor_SMD:R_0603_1608Metric"
+			(at 57.15 95.25 0)
+			(hide yes)
+			(show_name no)
+			(do_not_autoplace no)
+			(effects
+				(font
+					(size 1.27 1.27)
+				)
+			)
+		)
+		(property "Datasheet" ""
+			(at 57.15 95.25 0)
+			(hide yes)
+			(show_name no)
+			(do_not_autoplace no)
+			(effects
+				(font
+					(size 1.27 1.27)
+				)
+			)
+		)
+		(property "Description" ""
+			(at 57.15 95.25 0)
+			(hide yes)
+			(show_name no)
+			(do_not_autoplace no)
+			(effects
+				(font
+					(size 1.27 1.27)
+				)
+			)
+		)
+		(property "Manufacturer_Name" "--"
+			(at 57.15 95.25 0)
+			(hide yes)
+			(show_name no)
+			(do_not_autoplace no)
+			(effects
+				(font
+					(size 1.27 1.27)
+				)
+			)
+		)
+		(property "Manufacturer_Part_Number" "--"
+			(at 57.15 95.25 0)
+			(hide yes)
+			(show_name no)
+			(do_not_autoplace no)
+			(effects
+				(font
+					(size 1.27 1.27)
+				)
+			)
+		)
+		(property "Arrow Part Number" ""
+			(at 57.15 95.25 0)
+			(hide yes)
+			(show_name no)
+			(do_not_autoplace no)
+			(effects
+				(font
+					(size 1.27 1.27)
+				)
+			)
+		)
+		(property "Arrow Price/Stock" ""
+			(at 57.15 95.25 0)
+			(hide yes)
+			(show_name no)
+			(do_not_autoplace no)
+			(effects
+				(font
+					(size 1.27 1.27)
+				)
+			)
+		)
+		(property "Mouser Part Number" "--"
+			(at 57.15 95.25 0)
+			(hide yes)
+			(show_name no)
+			(do_not_autoplace no)
+			(effects
+				(font
+					(size 1.27 1.27)
+				)
+			)
+		)
+		(property "DigiKey Part Number" ""
+			(at 57.15 95.25 0)
+			(show_name no)
+			(do_not_autoplace no)
+			(effects
+				(font
+					(size 1.27 1.27)
+				)
+			)
+		)
+		(pin "1"
+		)
+		(pin "2"
+		)
+		(instances
+			(project "PUTM_AMS_MASTER_ISOLATION"
+				(path "/9b254bae-97c6-45e7-8618-9f461c55b31a/bb7c4aa8-5d23-481b-8672-1d87fa8c6d83"
+					(reference "R89")
+					(unit 1)
+				)
+				(path "/9b254bae-97c6-45e7-8618-9f461c55b31a/c0d62127-a5e4-40e6-9bd1-c5a7f1ecee97"
+					(reference "R90")
+					(unit 1)
+				)
