File: hardware/isolation/power.kicad_sch (KiCad schematic)
At the start: 50 parts, among them IC4 LMZM23601V5SILT, IC6 3.3V/0.5A, IC7 3.3V/0.5A, Q4 SI2347DS-T1-GE3, U4 TPS2113PWR

Commit message: sync
Connections:
- net PS_GND: now reaches C2.2, C3.2, C6.2, FL1.3, PS2.1 (-VIN)
- net PS_+24V: now reaches C2.1, C3.1, C7.2, FL1.4, PS2.16 (+VIN)
Changed lines of the file:
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@@
+		)
+	)
+	(label "PS_+24V"
+		(at 196.85 53.34 180)
+		(effects
+			(font
+				(size 0.5 0.5)
+			)
+			(justify right bottom)
+		)
+	)
+	(label "PS_GND"
+		(at 196.85 63.5 180)
+		(effects
+			(font
+				(size 0.5 0.5)
+			)
+			(justify right bottom)
 		)
 	)

Commit message: pcb finished
Parts:
- removed TP10, TP11, TP12, TP3, TP9: TestPoint_Small, TestPoint:TestPoint_THTPad_D1.0mm_Drill0.5mm, symbol Connector:TestPoint_Small
- R10, R11: footprint Resistor_SMD:R_0603_1608Metric_Pad0.98x0.95mm_HandSolder -> Resistor_SMD:R_0603_1608Metric
Connections:
- net F_24V: now also D1.1 (A1); no longer D1.2 (A2)
- net GND: now also D1.2 (A2); no longer D1.1 (A1)
- net F_+3.3V renamed F_+3.3VA
- net F_+3.3VA: no longer C14.2, F5.1, IC6.5 (VO)
- new net F_+3.3VIO: C14.2, F5.1, IC6.5 (VO)

Commit message: made bigger gap span between isolated ground planes
Parts:
- C1, C6, C7, C8: Mouser Part Number 80-CAS21C222KARFC -> 80-CAS26C182KARFC
Changed lines of the file:
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@@
 			)
 		)
-		(property "Mouser Part Number" "80-CAS21C222KARFC "
+		(property "Mouser Part Number" "80-CAS26C182KARFC"
 			(at 227.33 17.78 0)
 			(hide yes)
@@
 			)
 		)
-		(property "Mouser Part Number" "80-CAS21C222KARFC "
+		(property "Mouser Part Number" "80-CAS26C182KARFC"
 			(at 227.33 78.74 0)
 			(hide yes)
@@
 			)
 		)
-		(property "Mouser Part Number" "80-CAS21C222KARFC "
+		(property "Mouser Part Number" "80-CAS26C182KARFC"
 			(at 199.39 17.78 0)
 			(hide yes)
@@
 			)
 		)
-		(property "Mouser Part Number" "80-CAS21C222KARFC "
+		(property "Mouser Part Number" "80-CAS26C182KARFC"
 			(at 199.39 78.74 0)
 			(hide yes)
