File: hardware/isolation/usb.kicad_sch (KiCad schematic)
At the start: 28 parts, among them IC1 ISO6542DBQR, Q3 Si2365EDS, U2 FT230XS, U3 RI3-0505S

Commit message: made bigger gap span between isolated ground planes
Parts:
- C10, C26: Mouser Part Number 80-CAS21C222KARFC -> 80-CAS26C182KARFC
Changed lines of the file:
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@@
 			)
 		)
-		(property "Mouser Part Number" "80-CAS21C222KARFC "
+		(property "Mouser Part Number" "80-CAS26C182KARFC"
 			(at 62.23 81.28 0)
 			(hide yes)
@@
 			)
 		)
-		(property "Mouser Part Number" "80-CAS21C222KARFC "
+		(property "Mouser Part Number" "80-CAS26C182KARFC"
 			(at 90.17 81.28 0)
 			(hide yes)
