File: hardware/isolation/relay-driver.kicad_sch (KiCad schematic)
At the start: 7 parts, among them K1 IM07DTS, Q1 BSS316NH6327XTSA1

Commit message: sync
Parts:
- removed Q1: BSS316NH6327XTSA1, Package_TO_SOT_SMD:TSOT-23, symbol Device:Q_NMOS
- added Q8: 2N7002, Package_TO_SOT_SMD:SOT-23, symbol Transistor_FET:2N7002
Connections:
- net EN: now also Q8.1 (G)
- net GNDISO: now also Q8.2 (S)
- net at D2.2 (A), K1.8 (COIL_2): now also Q8.3 (D)
Changed lines of the file:
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@@
 	)
 	(symbol
-		(lib_id "Device:Q_NMOS")
+		(lib_id "Transistor_FET:2N7002")
 		(at 135.89 138.43 0)
 		(unit 1)
@@
 		(in_pos_files yes)
 		(dnp no)
-		(property "Reference" "Q1"
-			(at 134.62 132.08 0)
+		(property "Reference" "Q8"
+			(at 141.0716 137.2616 0)
 			(show_name no)
 			(do_not_autoplace no)
@@
 					(size 1.27 1.27)
 				)
-				(justify right)
+				(justify left)
 			)
 		)
-		(property "Value" "BSS316NH6327XTSA1"
-			(at 134.62 134.62 0)
+		(property "Value" "2N7002"
+			(at 141.0716 139.573 0)
 			(show_name no)
 			(do_not_autoplace no)
@@
 					(size 1.27 1.27)
 				)
-				(justify right)
+				(justify left)
 			)
 		)
-		(property "Footprint" "Package_TO_SOT_SMD:TSOT-23"
-			(at 140.97 135.89 0)
+		(property "Footprint" "Package_TO_SOT_SMD:SOT-23"
+			(at 140.97 140.335 0)
+			(hide yes)
+			(show_name no)
+			(do_not_autoplace no)
+			(effects
+				(font
+					(size 1.27 1.27)
+					(italic yes)
+				)
+				(justify left)
+			)
+		)
+		(property "Datasheet" "https://www.onsemi.com/pub/Collateral/NDS7002A-D.PDF"
+			(at 135.89 138.43 0)
 			(hide yes)
 			(show_name no)
@@
 					(size 1.27 1.27)
 				)
+				(justify left)
 			)
 		)
-		(property "Datasheet" "https://www.mouser.pl/datasheet/3/70/1/Infineon_BSS316N_DS_v02_03_EN.pdf"
+		(property "Description" ""
 			(at 135.89 138.43 0)
 			(hide yes)
@@
 			)
 		)
-		(property "Description" "MOSFETs N-Ch 30V 1.4A SOT-23-3"
+		(property "Manufacturer_Name" "--"
 			(at 135.89 138.43 0)
 			(hide yes)
@@
 			)
 		)
-		(property "Mouser Part Number" "726-BSS316NH6327"
+		(property "Manufacturer_Part_Number" "--"
 			(at 135.89 138.43 0)
 			(hide yes)
@@
 			)
 		)
-		(pin "G"
+		(property "Mouser Part Number" "621-DMN65D8L-7"
+			(at 135.89 138.43 0)
+			(hide yes)
+			(show_name no)
+			(do_not_autoplace no)
+			(effects
+				(font
+					(size 1.27 1.27)
+				)
+			)
 		)
-		(pin "D"
+		(property "DigiKey Part Number" ""
+			(at 135.89 138.43 0)
+			(show_name no)
+			(do_not_autoplace no)
+			(effects
+				(font
+					(size 1.27 1.27)
+				)
+			)
 		)
-		(pin "S"
+		(pin "1"
+		)
+		(pin "2"
+		)
+		(pin "3"
 		)
 		(instances
 			(project "PUTM_AMS_MASTER_ISOLATION"
 				(path "/9b254bae-97c6-45e7-8618-9f461c55b31a/27672bac-fee4-4e98-a9bd-03760133f34d"
-					(reference "Q5")
+					(reference "Q10")
 					(unit 1)
 				)
 				(path "/9b254bae-97c6-45e7-8618-9f461c55b31a/51b19b7d-5029-4e68-a889-ab95c2ea105b"
-					(reference "Q1")
+					(reference "Q8")
 					(unit 1)
 				)
 				(path "/9b254bae-97c6-45e7-8618-9f461c55b31a/52eeafc6-1d9f-461b-ab5d-05873b4b2dbb"
-					(reference "Q2")
+					(reference "Q9")
 					(unit 1)
 				)

Commit message: sync
Connections:
- net +24V is gone; now on net VDDSDC: R72.2
Changed lines of the file:
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@@
-		)
-	)
-	(wire
-		(pts
-			(xy 168.91 133.35) (xy 168.91 130.81)
-		)
-		(stroke
-			(width 0)
-			(type default)
 		)
 	)
@@
 			)
 			(justify right)
+		)
+	)
+	(hierarchical_label "VDDSDC"
+		(shape output)
+		(at 168.91 133.35 0)
+		(effects
+			(font
+				(size 1.27 1.27)
+			)
+			(justify left)
 		)
 	)
@@
 					(unit 1)
 				)
-			)
-		)
-	)
-	(symbol
-		(lib_id "power:+24V")
-		(at 168.91 130.81 0)
-		(unit 1)
-		(body_style 1)
-		(exclude_from_sim no)
-		(in_bom yes)
-		(on_board yes)
-		(in_pos_files yes)
-		(dnp no)
-		(fields_autoplaced yes)
-		(property "Reference" "#PWR011"
-			(at 168.91 134.62 0)
-			(hide yes)
-			(show_name no)
-			(do_not_autoplace no)
-			(effects
-				(font
-					(size 1.27 1.27)
-				)
-			)
-		)
-		(property "Value" "+24V"
-			(at 168.91 125.73 0)
-			(show_name no)
-			(do_not_autoplace no)
-			(effects
-				(font
-					(size 1.27 1.27)
-				)
-			)
-		)
-		(property "Footprint" ""
-			(at 168.91 130.81 0)
-			(hide yes)
-			(show_name no)
-			(do_not_autoplace no)
-			(effects
-				(font
-					(size 1.27 1.27)
-				)
-			)
-		)
-		(property "Datasheet" ""
-			(at 168.91 130.81 0)
-			(hide yes)
-			(show_name no)
-			(do_not_autoplace no)
-			(effects
-				(font
-					(size 1.27 1.27)
-				)
-			)
-		)
-		(property "Description" "Power symbol creates a global label with name \"+24V\""
-			(at 168.91 130.81 0)
-			(hide yes)
-			(show_name no)
-			(do_not_autoplace no)
-			(effects
-				(font
-					(size 1.27 1.27)
-				)
-			)
-		)
-		(pin "1"
-		)
-		(instances
-			(project "PUTM_AMS_MASTER_ISOLATION"
-				(path "/9b254bae-97c6-45e7-8618-9f461c55b31a/27672bac-fee4-4e98-a9bd-03760133f34d"
-					(reference "#PWR069")
-					(unit 1)
-				)
-				(path "/9b254bae-97c6-45e7-8618-9f461c55b31a/51b19b7d-5029-4e68-a889-ab95c2ea105b"
-					(reference "#PWR011")
-					(unit 1)
-				)
-				(path "/9b254bae-97c6-45e7-8618-9f461c55b31a/52eeafc6-1d9f-461b-ab5d-05873b4b2dbb"
-					(reference "#PWR056")
-					(unit 1)
-				)

Commit message: pcb finished
Connections:
- net +24ISO renamed +24VISO
Changed lines of the file:
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@@
 		(in_pos_files yes)
 		(dnp no)
-		(fields_autoplaced yes)
 		(property "Reference" "#PWR04"
 			(at 138.43 86.36 0)
@@
 			)
 		)
-		(property "Value" "+24ISO"
-			(at 138.43 77.47 0)
+		(property "Value" "+24VISO"
+			(at 138.43 78.74 0)
 			(show_name no)
 			(do_not_autoplace no)

Commit message: relay fix and changed ic PN for isolated rx/tx for usb to a type with standard output low instead of high
Connections:
- net DRV_H: now also K1.4 (NO_1); no longer K1.2 (NC_1)
Changed lines of the file:
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@@
 	)
 	(no_connect
-		(at 156.21 105.41)
+		(at 151.13 105.41)
 	)
 	(wire
@@
 	(wire
 		(pts
-			(xy 151.13 118.11) (xy 166.37 118.11)
-		)
-		(stroke
-			(width 0)
-			(type default)
-		)
-	)
-	(wire
-		(pts
 			(xy 163.83 107.95) (xy 166.37 107.95)
-		)
-		(stroke
-			(width 0)
-			(type default)
-		)
-	)
-	(wire
-		(pts
-			(xy 151.13 105.41) (xy 151.13 118.11)
 		)
 		(stroke
@@
 	(wire
 		(pts
+			(xy 156.21 118.11) (xy 166.37 118.11)
+		)
+		(stroke
+			(width 0)
+			(type default)
+		)
+	)
+	(wire
+		(pts
 			(xy 138.43 107.95) (xy 138.43 133.35)
 		)
@@
 		)
 		(stroke
+			(width 0)
+			(type default)
+		)
+	)
+	(wire
+		(pts
+			(xy 156.21 105.41) (xy 156.21 118.11)
+		)
+		(stroke

Commit message: sync
Parts:
- R72: value 1k -> 10k
Changed lines of the file:
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@@
 			)
 		)
-		(property "Value" "1k"
+		(property "Value" "10k"
 			(at 163.83 130.81 90)
 			(show_name no)
