File: hardware/isolation/relay-driver.kicad_sch (KiCad schematic)
At the start: 7 parts, among them K1 IM07DTS, Q8 2N7002

Commit message: bom update
Parts:
- D2, D4: value 30V/4A -> 1000V/1A; Mouser Part Number 78-BAT42W-E3-18 -> 863-NRVS1MFL
Changed lines of the file:
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@@
 			)
 		)
-		(property "Value" "30V/4A"
+		(property "Value" "1000V/1A"
 			(at 168.91 114.3 90)
 			(show_name no)
@@
 			)
 		)
-		(property "Datasheet" "https://www.vishay.com/docs/86404/bat42w.pdf"
+		(property "Datasheet" ""
 			(at 166.37 113.03 90)
 			(hide yes)
@@
 			)
 		)
-		(property "Description" "Schottky Diodes & Rectifiers 30Volt 200mA 4A IFSM"
+		(property "Description" "1000V/1A"
 			(at 166.37 113.03 0)
 			(hide yes)
@@
 			)
 		)
-		(property "Mouser Part Number" "78-BAT42W-E3-18"
+		(property "Mouser Part Number" "863-NRVS1MFL "
 			(at 166.37 113.03 90)
 			(hide yes)
@@
 			)
 		)
-		(property "Value" "30V/4A"
+		(property "Value" "1000V/1A"
 			(at 135.89 97.5359 90)
 			(show_name no)
@@
 			)
 		)
-		(property "Datasheet" "https://www.vishay.com/docs/86404/bat42w.pdf"
+		(property "Datasheet" ""
 			(at 138.43 96.52 90)
 			(hide yes)
@@
 			)
 		)
-		(property "Mouser Part Number" "78-BAT42W-E3-18"
+		(property "Mouser Part Number" "863-NRVS1MFL "
 			(at 138.43 96.52 90)
 			(hide yes)
