File: hardware/isolation/sdc-driver.kicad_sch (KiCad schematic)
At the start: 4 parts, among them K2 IM07DTS

Commit message: pcb finished
Connections:
- net +24ISO renamed +24VISO
Changed lines of the file:
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@@
 		(in_pos_files yes)
 		(dnp no)
-		(fields_autoplaced yes)
 		(property "Reference" "#PWR05"
 			(at 140.97 86.36 0)
@@
 			)
 		)
-		(property "Value" "+24ISO"
-			(at 140.97 77.47 0)
+		(property "Value" "+24VISO"
+			(at 140.97 78.74 0)
 			(show_name no)
 			(do_not_autoplace no)

Commit message: sync
Parts:
- R75: value 1k -> 10k
Changed lines of the file:
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@@
 			)
 		)
-		(property "Value" "1k"
+		(property "Value" "10k"
 			(at 184.15 93.98 0)
 			(show_name no)
