File: hardware/isolation/sdc-driver.kicad_sch (KiCad schematic)
At the start: 4 parts, among them K2 IM07DTS

Commit message: bom update
Parts:
- D7: value 30V/4A -> 1000V/1A; Mouser Part Number 78-BAT42W-E3-18 -> 863-NRVS1MFL
Changed lines of the file:
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@@
 			)
 		)
-		(property "Value" "30V/4A"
+		(property "Value" "1000V/1A"
 			(at 138.43 97.5359 90)
 			(show_name no)
@@
 			)
 		)
-		(property "Datasheet" "https://www.vishay.com/docs/86404/bat42w.pdf"
+		(property "Datasheet" ""
 			(at 140.97 96.52 90)
 			(hide yes)
@@
 			)
 		)
-		(property "Mouser Part Number" "78-BAT42W-E3-18"
+		(property "Mouser Part Number" "863-NRVS1MFL "
 			(at 140.97 96.52 90)
 			(hide yes)
