File: hardware/isolation/iso-input.kicad_sch (KiCad schematic)
At the start: 3 parts, among them U6 ISOM8710DFFR

Commit message: pcb finished
Parts:
- C60: footprint Capacitor_SMD:C_0603_1608Metric_Pad1.08x0.95mm_HandSolder -> Capacitor_SMD:C_0603_1608Metric
Changed lines of the file:
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@@
 			)
 		)
-		(property "Footprint" "Capacitor_SMD:C_0603_1608Metric_Pad1.08x0.95mm_HandSolder"
+		(property "Footprint" "Capacitor_SMD:C_0603_1608Metric"
 			(at 166.37 92.71 0)
 			(hide yes)

Commit message: sync
Parts:
- R86: value 1k -> 10k
Changed lines of the file:
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@@
 			)
 		)
-		(property "Value" "1k"
+		(property "Value" "10k"
 			(at 133.35 97.79 90)
 			(show_name no)

Commit message: sync
Changed lines of the file:
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@@
 		(instances
 			(project "PUTM_AMS_MASTER_ISOLATION"
+				(path "/9b254bae-97c6-45e7-8618-9f461c55b31a"
+					(reference "U7")
+					(unit 1)
+				)
 				(path "/9b254bae-97c6-45e7-8618-9f461c55b31a/577357ca-978a-4aab-a7a4-e0cbcaa1ed5b"
 					(reference "U7")

Commit message: kek
Parts:
- R86: value 10k -> 4.7k
Changed lines of the file:
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@@
 			)
 		)
-		(property "Value" "10k"
+		(property "Value" "4.7k"
 			(at 133.35 97.79 90)
 			(show_name no)
@@
 		(instances
 			(project "PUTM_AMS_MASTER_ISOLATION"
-				(path "/9b254bae-97c6-45e7-8618-9f461c55b31a"
-					(reference "U7")
-					(unit 1)
-				)
 				(path "/9b254bae-97c6-45e7-8618-9f461c55b31a/577357ca-978a-4aab-a7a4-e0cbcaa1ed5b"
 					(reference "U7")
